Commit message: Added stl/obj mesh fallback from cli
Added stl & obj files to meshes, updated xacro files to build a specific file type using arg:mesh:=mesh_type (defaulted to dae)

File: urdf/arm/openarm_arm.xacro (robot description, xacro)
@@ -2,5 +2,5 @@
 <robot xmlns:xacro="http://www.ros.org/wiki/xacro" name="openarm">
   <xacro:include filename="$(find openarm_description)/urdf/arm/openarm_macro.xacro" />
-  <xacro:macro name="openarm_arm" params="arm_type arm_prefix:='' no_prefix:=false description_pkg:='openarm_description' connected_to:='base' xyz:='0 0 0' rpy:='0 0 0' joint_limits inertials kinematics kinematics_link kinematics_offset:=none " >
+  <xacro:macro name="openarm_arm" params="arm_type arm_prefix:='' no_prefix:=false description_pkg:='openarm_description' connected_to:='base' xyz:='0 0 0' rpy:='0 0 0' joint_limits inertials kinematics kinematics_link kinematics_offset:=none mesh_ext:='dae'" >
     <xacro:property name="prefix" value="${'' if no_prefix else 'openarm' + '_' + arm_prefix}" />
     <xacro:if value="${arm_prefix == 'right_'}">

File: urdf/arm/openarm_macro.xacro (robot description, xacro)
@@ -27,5 +27,5 @@
         <xacro:openarm-kinematics-link config="${kinematics_link}" name="${name}" />
         <geometry>
-          <mesh filename="package://${description_pkg}/meshes/arm/${arm_type}/visual/${name}.dae" scale="0.001 ${0.001*reflect} 0.001" />
+          <mesh filename="package://${description_pkg}/meshes/arm/${arm_type}/visual/${name}.${mesh_ext}" scale="0.001 ${0.001*reflect} 0.001" />
         </geometry>
       </visual>

File: urdf/body/openarm_body.xacro (robot description, xacro)
@@ -12,5 +12,7 @@
               inertials
               kinematics
-              kinematics_link">
+              kinematics_link
+              mesh_ext:='dae'
+              ">
     <!-- <xacro:property name="prefix" value="${'' if no_prefix else body_prefix + 'body_'}" /> -->
     <xacro:property name="prefix" value="${'' if no_prefix else 'openarm_' + 'body_'}" />

File: urdf/body/openarm_body_macro.xacro (robot description, xacro)
@@ -23,5 +23,5 @@
         <xacro:openarm-body-kinematics config="${kinematics_link}" name="${name}" />
         <geometry>
-          <mesh filename="package://${description_pkg}/meshes/body/${body_type}/visual/${name}.dae" scale="0.001 0.001 0.001" />
+          <mesh filename="package://${description_pkg}/meshes/body/${body_type}/visual/${name}.${mesh_ext}" scale="0.001 0.001 0.001" />
         </geometry>
       </visual>

File: urdf/ee/ee_with_one_link.xacro (robot description, xacro)
@@ -2,5 +2,5 @@
 <robot xmlns:xacro="http://www.ros.org/wiki/xacro" name="ee_with_one_link">
   <!-- safety_distance: Minimum safety distance in [m] by which the collision volumes are expanded and which is enforced during robot motions -->
-  <xacro:macro name="ee_with_one_link" params="connected_to:='' arm_type arm_prefix:='' ee_type ee_inertials rpy_ee:='0 0 0' xyz_ee:='0 0 0' tcp_xyz:='0 0 0' tcp_rpy:='0 0 0' description_pkg:=openarm_description with_sc:=false">
+  <xacro:macro name="ee_with_one_link" params="connected_to:='' arm_type arm_prefix:='' ee_type ee_inertials rpy_ee:='0 0 0' xyz_ee:='0 0 0' tcp_xyz:='0 0 0' tcp_rpy:='0 0 0' description_pkg:=openarm_description with_sc:=false mesh_ext:='dae'">
     <xacro:property name="ee_prefix" default="robot_"/>
     <xacro:unless value="${arm_type == ''}">

File: urdf/ee/openarm_hand.xacro (robot description, xacro)
@@ -2,5 +2,5 @@
 <robot xmlns:xacro="http://www.ros.org/wiki/xacro" name="hand">
   <!-- safety_distance: Minimum safety distance in [m] by which the collision volumes are expanded and which is enforced during robot motions -->
-  <xacro:macro name="openarm_hand" params="connected_to:='' arm_type arm_prefix:='' ee_type ee_inertials ee_kinematics_link rpy_ee:='0 0 0' xyz_ee:='0 0 0' tcp_xyz:='0 0 0' tcp_rpy:='0 0 0' description_pkg:=openarm_description">
+  <xacro:macro name="openarm_hand" params="connected_to:='' arm_type arm_prefix:='' ee_type ee_inertials ee_kinematics_link rpy_ee:='0 0 0' xyz_ee:='0 0 0' tcp_xyz:='0 0 0' tcp_rpy:='0 0 0' description_pkg:=openarm_description mesh_ext:='dae'">
     <xacro:property name="ee_prefix" default=""/>
     <xacro:unless value="${arm_type == ''}">
@@ -29,5 +29,5 @@
         <xacro:openarm-ee-kinematics-link config="${ee_kinematics_link}" name="left_finger" />
         <geometry>
-          <mesh filename="package://${description_pkg}/meshes/ee/${ee_type}/visual/finger.dae" scale="0.001 0.001 0.001"/>
+          <mesh filename="package://${description_pkg}/meshes/ee/${ee_type}/visual/finger.${mesh_ext}" scale="0.001 0.001 0.001"/>
         </geometry>
       </visual>
@@ -44,5 +44,5 @@
         <xacro:openarm-ee-kinematics-link config="${ee_kinematics_link}" name="right_finger" />
         <geometry>
-          <mesh filename="package://${description_pkg}/meshes/ee/${ee_type}/visual/finger.dae" scale="0.001 -0.001 0.001"/>
+          <mesh filename="package://${description_pkg}/meshes/ee/${ee_type}/visual/finger.${mesh_ext}" scale="0.001 -0.001 0.001"/>
         </geometry>
       </visual>

File: urdf/ee/openarm_hand_macro.xacro (robot description, xacro)
@@ -25,5 +25,5 @@
         <xacro:openarm-ee-kinematics-link config="${ee_kinematics_link}" name="${name}" />
         <geometry>
-          <mesh filename="package://${description_pkg}/meshes/ee/${ee_type}/visual/${name}.dae" scale="0.001 0.001 0.001" />
+          <mesh filename="package://${description_pkg}/meshes/ee/${ee_type}/visual/${name}.${mesh_ext}" scale="0.001 0.001 0.001" />
         </geometry>
       </visual>

File: urdf/robot/openarm_robot.xacro (robot description, xacro)
@@ -36,6 +36,6 @@
             left_arm_prefix:='left_'
             right_arm_prefix:='right_'
-            "
-            >
+            mesh_ext:='dae'
+            ">
     <xacro:include filename="$(find openarm_description)/urdf/arm/openarm_macro.xacro" />
     <xacro:include filename="$(find openarm_description)/urdf/arm/openarm_arm.xacro" />
@@ -62,5 +62,6 @@
         inertials="${body_inertials}"
         kinematics="${body_kinematics}"
-        kinematics_link="${body_kinematics_link}" />
+        kinematics_link="${body_kinematics_link}"
+        mesh_ext="${mesh_ext}" />
         <!-- left arm -->
         <xacro:openarm_arm
@@ -76,5 +77,6 @@
         kinematics="${kinematics}"
         kinematics_link="${kinematics_link}"
-        kinematics_offset="${kinematics_offset}" />
+        kinematics_offset="${kinematics_offset}"
+        mesh_ext="${mesh_ext}" />
         <!-- right arm -->
         <xacro:openarm_arm
@@ -90,5 +92,6 @@
         kinematics="${kinematics}"
         kinematics_link="${kinematics_link}"
-        kinematics_offset="${kinematics_offset}" />
+        kinematics_offset="${kinematics_offset}"
+        mesh_ext="${mesh_ext}" />
         <!-- ros2_control hardware interfaces for bimanual setup -->
         <xacro:if value="${ros2_control}">
@@ -101,5 +104,6 @@
             left_arm_prefix="${left_arm_prefix}"
             right_arm_prefix="${right_arm_prefix}"
-            hand="${hand}"/>
+            hand="${hand}"
+            mesh_ext="${mesh_ext}"/>
         </xacro:if>
         <xacro:if value="$(eval hand and ee_type == 'openarm_hand')">
@@ -116,4 +120,5 @@
                 tcp_rpy="$(arg tcp_rpy)"
                 description_pkg="$(arg description_pkg)"
+                mesh_ext="${mesh_ext}"
             />
             <xacro:openarm_hand
@@ -129,4 +134,5 @@
                 tcp_rpy="$(arg tcp_rpy)"
                 description_pkg="$(arg description_pkg)"
+                mesh_ext="${mesh_ext}"
             />
           </xacro:if>
@@ -144,4 +150,5 @@
         inertials="${inertials}"
         connected_to=""
+        mesh_ext="${mesh_ext}"
         />
         <xacro:if value="${ros2_control}">
@@ -153,5 +160,6 @@
             fake_sensor_commands="${fake_sensor_commands}"
             hand="${hand}"
-            bimanual="false"/>
+            bimanual="false"
+            mesh_ext="${mesh_ext}"/>
         </xacro:if>
         <xacro:if value="${hand and ee_type == 'openarm_hand'}">
@@ -171,5 +179,6 @@
             tcp_xyz="$(arg tcp_xyz)"
             tcp_rpy="$(arg tcp_rpy)"
-            description_pkg="$(arg description_pkg)"/>
+            description_pkg="$(arg description_pkg)"
+            mesh_ext="${mesh_ext}"/>
         </xacro:if>
         </xacro:if>

File: urdf/robot/v10.urdf.xacro (robot description, xacro)
@@ -22,4 +22,5 @@
   <xacro:arg name="fake_sensor_commands" default="false" />
   <xacro:arg name="bimanual" default="false" />
+  <xacro:arg name="mesh_ext" default="dae" />
   <xacro:arg name="right_arm_base_xyz" default="0.0 -0.031 0.698" />
   <xacro:arg name="right_arm_base_rpy" default="1.5708 0 0" />
@@ -54,4 +55,5 @@
   body_connected_to="world"
   bimanual="$(arg bimanual)"
+  mesh_ext="$(arg mesh_ext)"
   right_arm_base_xyz="$(arg right_arm_base_xyz)"
   left_arm_base_xyz="$(arg left_arm_base_xyz)"
