Commit message: fix mesh path

File: assets/robot/openarm_v1.0/urdf/ee/openarm_ee_macro.xacro (robot description, xacro)
@@ -33,5 +33,5 @@
   </xacro:macro>
   <xacro:macro name="ee_link_with_sc" params="name prefix rpy:='0 0 0' ee_kinematics_link reflect:=1">
-    <xacro:property name="ee_mesh_root" value="${'package://' + description_pkg + '/assets/end_effector/parallel_link/mesh' if ee_type == 'parallel_link' else 'package://' + description_pkg + '/assets/end_effector/pinch_gripper/meshes/old'}" />
+    <xacro:property name="ee_mesh_root" value="${'package://' + description_pkg + '/assets/end_effector/parallel_link/meshes' if ee_type == 'parallel_link' else 'package://' + description_pkg + '/assets/end_effector/pinch_gripper/meshes'}" />
     <link name="${prefix}${name}">
       <visual name="${prefix}${name}_visual">
@@ -61,5 +61,5 @@
   </xacro:macro>
   <xacro:macro name="ee_finger_link_with_sc" params="name prefix ee_kinematics_link arm_reflect:=1 finger_reflect:=1">
-    <xacro:property name="ee_mesh_root" value="${'package://' + description_pkg + '/assets/end_effector/parallel_link/mesh' if ee_type == 'parallel_link' else 'package://' + description_pkg + '/assets/end_effector/pinch_gripper/meshes/old'}" />
+    <xacro:property name="ee_mesh_root" value="${'package://' + description_pkg + '/assets/end_effector/parallel_link/meshes' if ee_type == 'parallel_link' else 'package://' + description_pkg + '/assets/end_effector/pinch_gripper/meshes'}" />
     <link name="${prefix}${name}">
       <visual name="${prefix}${name}_visual">
