Commit message: Keep V1 TCP defaults in the gripper macro

File: assets/robot/openarm_v1.0/urdf/ee/ee_dispatcher.xacro (robot description, xacro)
@@ -14,5 +14,5 @@
 <robot xmlns:xacro="http://www.ros.org/wiki/xacro">
   <xacro:include filename="$(find openarm_description)/assets/robot/openarm_v1.0/urdf/ee/parallel_link/openarm_parallel_gripper.xacro" />
-  <xacro:macro name="openarm_ee" params="ee_type connected_to arm_type arm_prefix ee_kinematics ee_kinematics_link ee_inertials ee_joints_limits rpy_ee:='0 0 0' xyz_ee:='0 0 0' tcp_xyz:='0 0 0.093' tcp_rpy:='0 0 0' description_pkg:=openarm_description no_prefix:=false">
+  <xacro:macro name="openarm_ee" params="ee_type connected_to arm_type arm_prefix ee_kinematics ee_kinematics_link ee_inertials ee_joints_limits rpy_ee:='0 0 0' xyz_ee:='0 0 0' tcp_xyz:='0 0 0' tcp_rpy:='0 0 0' description_pkg:=openarm_description no_prefix:=false">
     <xacro:if value="${ee_type == 'parallel_link'}">
       <xacro:openarm_parallel_gripper
@@ -25,6 +25,4 @@
         ee_inertials="${ee_inertials}"
         ee_joints_limits="${ee_joints_limits}"
-        tcp_xyz="${tcp_xyz}"
-        tcp_rpy="${tcp_rpy}"
         description_pkg="${description_pkg}"
         no_prefix="${no_prefix}"

Commit message: Fix V1 link and control names with no_prefix

File: assets/robot/openarm_v1.0/urdf/ee/ee_dispatcher.xacro (robot description, xacro)
@@ -14,5 +14,5 @@
 <robot xmlns:xacro="http://www.ros.org/wiki/xacro">
   <xacro:include filename="$(find openarm_description)/assets/robot/openarm_v1.0/urdf/ee/parallel_link/openarm_parallel_gripper.xacro" />
-  <xacro:macro name="openarm_ee" params="ee_type connected_to arm_type arm_prefix ee_kinematics ee_kinematics_link ee_inertials ee_joints_limits rpy_ee:='0 0 0' xyz_ee:='0 0 0' tcp_xyz:='0 0 0' tcp_rpy:='0 0 0' description_pkg:=openarm_description">
+  <xacro:macro name="openarm_ee" params="ee_type connected_to arm_type arm_prefix ee_kinematics ee_kinematics_link ee_inertials ee_joints_limits rpy_ee:='0 0 0' xyz_ee:='0 0 0' tcp_xyz:='0 0 0' tcp_rpy:='0 0 0' description_pkg:=openarm_description no_prefix:=false">
     <xacro:if value="${ee_type == 'parallel_link'}">
       <xacro:openarm_parallel_gripper
@@ -25,4 +25,6 @@
         ee_inertials="${ee_inertials}"
         ee_joints_limits="${ee_joints_limits}"
+        description_pkg="${description_pkg}"
+        no_prefix="${no_prefix}"
       />
     </xacro:if>

File: assets/robot/openarm_v1.0/urdf/ee/parallel_link/openarm_parallel_gripper.xacro (robot description, xacro)
@@ -18,9 +18,6 @@
     parallel-link gripper — measured from the hand frame origin.
   -->
-  <xacro:macro name="openarm_parallel_gripper" params="connected_to:='' arm_type arm_prefix:='' ee_type ee_inertials ee_kinematics ee_kinematics_link ee_joints_limits rpy_ee:='0 0 0' xyz_ee:='0 0 0' tcp_xyz:='0 0 0.0835' tcp_rpy:='0 0 0' description_pkg:=openarm_description">
-    <xacro:property name="ee_prefix" default=""/>
-    <xacro:unless value="${arm_type == ''}">
-      <xacro:property name="ee_prefix" value="openarm_${arm_prefix}" />
-    </xacro:unless>
+  <xacro:macro name="openarm_parallel_gripper" params="connected_to:='' arm_type arm_prefix:='' ee_type ee_inertials ee_kinematics ee_kinematics_link ee_joints_limits rpy_ee:='0 0 0' xyz_ee:='0 0 0' tcp_xyz:='0 0 0.0835' tcp_rpy:='0 0 0' description_pkg:=openarm_description no_prefix:=false">
+    <xacro:property name="ee_prefix" value="${'' if no_prefix or arm_type == '' else 'openarm_' + arm_prefix}" />
     <link name="${ee_prefix}hand">
       <visual name="${ee_prefix}hand_visual">
