Commit message: Remove commented-out finger joints from the V1 gripper macro
openarm_parallel_gripper.xacro kept an old, commented-out definition of
finger_joint1 and finger_joint2 (z = 0.115, 333 N, 10 m/s) after the
real joints. xacro preserves comments, so this block was emitted
verbatim, with unexpanded ${ee_prefix}, into every generated V1 URDF and,
since #89, into the standalone gripper URDF as well.

Remove the block and regenerate the V1 example URDF.

Co-Authored-By: Claude Opus 5.5 <noreply@anthropic.com>

File: assets/robot/openarm_v1.0/urdf/ee/parallel_link/openarm_parallel_gripper.xacro (robot description, xacro)
@@ -95,17 +95,4 @@
         <mimic joint="${ee_prefix}finger_joint1" />
     </joint>
-    <!-- <joint name="${ee_prefix}finger_joint1" type="prismatic">
-      <parent link="${connected_to}" /> <child link="${ee_prefix}right_finger" />
-      <origin xyz="0 -0.006 0.115" rpy="0 0 0" />
-      <axis xyz="0 -1 0" />
-      <limit effort="333" lower="0.0" upper="0.044" velocity="10.0" />
-    </joint>
-    <joint name="${ee_prefix}finger_joint2" type="prismatic">
-      <parent link="${connected_to}" /> <child link="${ee_prefix}left_finger" />
-      <origin xyz="0 0.006 0.115" rpy="0 0 0" />
-      <axis xyz="0 1 0" />
-      <limit effort="333" lower="0.0" upper="0.044" velocity="10.0" />
-      <mimic joint="${ee_prefix}finger_joint1" />
-    </joint> -->
   </xacro:macro>
 </robot>
