Commit message: Keep V1 finger frames aligned and rotate opposing meshes

File: assets/robot/openarm_v1.0/urdf/ee/parallel_link/openarm_parallel_gripper.xacro (robot description, xacro)
@@ -77,5 +77,5 @@
         <child link="${ee_prefix}right_finger" />
         <xacro:openarm-ee-kinematics config="${ee_kinematics}" name="finger_joint" />
-        <axis xyz="0 1 0" />
+        <axis xyz="0 -1 0" />
         <limit effort="${finger_limits.effort}" lower="${finger_limits.lower}"
                upper="${finger_limits.upper}" velocity="${finger_limits.velocity}" />

File: assets/robot/openarm_v1.0/urdf/example/v1.urdf (robot description, URDF)
Before this commit: robot openarm, 26 links, 25 joints
Joints:
- joint openarm_left_finger_joint1: axis 0 1 0 -> 0 -1 0; origin xyz=0.0 -0.005 0.015 rpy=0 0 3.141592653589793 -> xyz=0.0 -0.005 0.015 rpy=0 0 0
- joint openarm_right_finger_joint1: axis 0 1 0 -> 0 -1 0; origin xyz=0.0 -0.005 0.015 rpy=0 0 3.141592653589793 -> xyz=0.0 -0.005 0.015 rpy=0 0 0

Commit message: Use shared V1 gripper force and velocity limits

File: assets/robot/openarm_v1.0/urdf/ee/parallel_link/openarm_parallel_gripper.xacro (robot description, xacro)
@@ -20,4 +20,5 @@
   <xacro:macro name="openarm_parallel_gripper" params="connected_to:='' arm_type arm_prefix:='' ee_type ee_inertials ee_kinematics ee_kinematics_link ee_joints_limits rpy_ee:='0 0 0' xyz_ee:='0 0 0' tcp_xyz:='0 0 0.0835' tcp_rpy:='0 0 0' description_pkg:=openarm_description no_prefix:=false">
     <xacro:property name="ee_prefix" value="${'' if no_prefix or arm_type == '' else 'openarm_' + arm_prefix}" />
+    <xacro:property name="finger_limits" value="${ee_joints_limits['finger_joint']['limit']}" />
     <link name="${ee_prefix}hand">
       <visual name="${ee_prefix}hand_visual">
@@ -80,5 +81,6 @@
         <xacro:openarm-ee-kinematics config="${ee_kinematics}" name="finger_joint" />
         <axis xyz="0 -1 0" />
-        <limit effort="333" lower="0.0" upper="0.044" velocity="10.0" />
+        <limit effort="${finger_limits.effort}" lower="${finger_limits.lower}"
+               upper="${finger_limits.upper}" velocity="${finger_limits.velocity}" />
     </joint>
     <joint name="${ee_prefix}finger_joint2" type="prismatic">
@@ -88,5 +90,6 @@
         <origin xyz="${fj.x} ${-fj.y} ${fj.z}" rpy="0 0 0" />
         <axis xyz="0 1 0" />
-        <limit effort="333" lower="0.0" upper="0.044" velocity="10.0" />
+        <limit effort="${finger_limits.effort}" lower="${finger_limits.lower}"
+               upper="${finger_limits.upper}" velocity="${finger_limits.velocity}" />
         <mimic joint="${ee_prefix}finger_joint1" />
     </joint>

File: assets/robot/openarm_v1.0/urdf/example/v1.urdf (robot description, URDF)
Before this commit: robot openarm, 26 links, 25 joints
Joints:
- joint openarm_left_finger_joint1: limit lower=0.0 upper=0.044 effort=333 velocity=10.0 -> lower=0.0 upper=0.044 effort=150.75 velocity=0.661
- joint openarm_left_finger_joint2: limit lower=0.0 upper=0.044 effort=333 velocity=10.0 -> lower=0.0 upper=0.044 effort=150.75 velocity=0.661
- joint openarm_right_finger_joint1: limit lower=0.0 upper=0.044 effort=333 velocity=10.0 -> lower=0.0 upper=0.044 effort=150.75 velocity=0.661
- joint openarm_right_finger_joint2: limit lower=0.0 upper=0.044 effort=333 velocity=10.0 -> lower=0.0 upper=0.044 effort=150.75 velocity=0.661

Commit message: Preserve the V1 gripper hierarchy while correcting origins

File: assets/robot/openarm_v1.0/urdf/ee/parallel_link/openarm_parallel_gripper.xacro (robot description, xacro)
@@ -74,5 +74,5 @@
     </link>
     <joint name="${ee_prefix}finger_joint1" type="prismatic">
-        <parent link="${ee_prefix}hand" />
+        <parent link="${connected_to}" />
         <child link="${ee_prefix}right_finger" />
         <xacro:openarm-ee-kinematics config="${ee_kinematics}" name="finger_joint" />
@@ -82,5 +82,5 @@
     </joint>
     <joint name="${ee_prefix}finger_joint2" type="prismatic">
-        <parent link="${ee_prefix}hand" />
+        <parent link="${connected_to}" />
         <child link="${ee_prefix}left_finger" />
         <xacro:property name="fj" value="${ee_kinematics['finger_joint']['kinematic']}" />

File: assets/robot/openarm_v1.0/urdf/example/v1.urdf (robot description, URDF)
Before this commit: robot openarm, 26 links, 25 joints
Joints:
- joint openarm_left_finger_joint1: origin xyz=0.0 -0.005 0.015 rpy=0 0 0 -> xyz=0.0 -0.005 0.1151 rpy=0 0 0; parent openarm_left_hand -> openarm_left_link7
- joint openarm_left_finger_joint2: origin xyz=0.0 0.005 0.015 rpy=0 0 0 -> xyz=0.0 0.005 0.1151 rpy=0 0 0; parent openarm_left_hand -> openarm_left_link7
- joint openarm_right_finger_joint1: origin xyz=0.0 -0.005 0.015 rpy=0 0 0 -> xyz=0.0 -0.005 0.1151 rpy=0 0 0; parent openarm_right_hand -> openarm_right_link7
- joint openarm_right_finger_joint2: origin xyz=0.0 0.005 0.015 rpy=0 0 0 -> xyz=0.0 0.005 0.1151 rpy=0 0 0; parent openarm_right_hand -> openarm_right_link7

Commit message: Use measured V1 end-effector inertias and hand-parent fingers

File: assets/robot/openarm_v1.0/urdf/ee/parallel_link/openarm_parallel_gripper.xacro (robot description, xacro)
@@ -74,5 +74,5 @@
     </link>
     <joint name="${ee_prefix}finger_joint1" type="prismatic">
-        <parent link="${connected_to}" />
+        <parent link="${ee_prefix}hand" />
         <child link="${ee_prefix}right_finger" />
         <xacro:openarm-ee-kinematics config="${ee_kinematics}" name="finger_joint" />
@@ -82,5 +82,5 @@
     </joint>
     <joint name="${ee_prefix}finger_joint2" type="prismatic">
-        <parent link="${connected_to}" />
+        <parent link="${ee_prefix}hand" />
         <child link="${ee_prefix}left_finger" />
         <xacro:property name="fj" value="${ee_kinematics['finger_joint']['kinematic']}" />

File: assets/robot/openarm_v1.0/urdf/example/v1.urdf (robot description, URDF)
Before this commit: robot openarm, 26 links, 25 joints
Links:
- link openarm_left_hand: mass 0.127 -> 0.1723111736408497
- link openarm_left_left_finger: mass 0.03602545343277134 -> 0.07444998664008126
- link openarm_left_link7: mass 0.4659771327380578 -> 0.4054971268153967
- link openarm_left_right_finger: mass 0.03602545343277134 -> 0.07444998664008126
- link openarm_right_hand: mass 0.127 -> 0.1723111736408497
- link openarm_right_left_finger: mass 0.03602545343277134 -> 0.07444998664008126
- link openarm_right_link7: mass 0.4659771327380578 -> 0.4054971268153967
- link openarm_right_right_finger: mass 0.03602545343277134 -> 0.07444998664008126
Joints:
- joint openarm_left_finger_joint1: origin xyz=0.0 -0.005 0.1151 rpy=0 0 0 -> xyz=0.0 -0.005 0.015 rpy=0 0 0; parent openarm_left_link7 -> openarm_left_hand
- joint openarm_left_finger_joint2: origin xyz=0.0 0.005 0.1151 rpy=0 0 0 -> xyz=0.0 0.005 0.015 rpy=0 0 0; parent openarm_left_link7 -> openarm_left_hand
- joint openarm_right_finger_joint1: origin xyz=0.0 -0.005 0.1151 rpy=0 0 0 -> xyz=0.0 -0.005 0.015 rpy=0 0 0; parent openarm_right_link7 -> openarm_right_hand
- joint openarm_right_finger_joint2: origin xyz=0.0 0.005 0.1151 rpy=0 0 0 -> xyz=0.0 0.005 0.015 rpy=0 0 0; parent openarm_right_link7 -> openarm_right_hand

Commit message: Set the V1 TCP 90 mm from hand (#92)
Change the V1 hand-local TCP default from **85.9 mm to 90 mm**, placing
it **190.1 mm from link7**. Update the robot gripper macro, standalone
gripper and example URDF together.

Rationale:

This aligns the V1 TCP with openarm_isaac_lab, so that
openarm_description, openarm_mujoco and openarm_isaac_lab use the same
TCP.

- The [V1
USD](https://github.com/enactic/openarm_isaac_lab/blob/cb7ff7547bdb81f290591edb9302b4845b1d49a7/source/openarm/openarm/tasks/manager_based/openarm_manipulation/usds/openarm_unimanual/openarm_unimanual.usd)
in openarm_isaac_lab places `openarm_ee_tcp` 193.1 mm from link7.
- The [cabinet
task](https://github.com/enactic/openarm_isaac_lab/blob/cb7ff7547bdb81f290591edb9302b4845b1d49a7/source/openarm/openarm/tasks/manager_based/openarm_manipulation/unimanual/cabinet/config/joint_pos_env_cfg.py#L65)
applies a −3 mm Z offset to it, so the TCP that the task uses is 190.1
mm from link7.
- `hand` is 100.1 mm from link7, so the TCP is 190.1 − 100.1 = **90 mm**
from `hand`.
- openarm_mujoco uses the same value since enactic/openarm_mujoco#95.

Impact on users:

This moves the `*_hand_tcp` frame 4.1 mm further along the hand Z axis
(from 186.0 mm to 190.1 mm from link7). Joints, link frames, meshes and
inertias don't change.

- If you use `*_hand_tcp` as the target or tip frame for IK, motion
planning or Cartesian control, the same target pose now puts the gripper
4.1 mm further back from the target. For example, the fingertips stop
4.1 mm shorter of a grasp point. To keep the previous behavior, pass
`tcp_xyz:='0 0 0.0859'` explicitly.
- If you recorded or trained poses relative to `*_hand_tcp`, they're now
4.1 mm off. This includes datasets, calibrations and policies.
- The default MoveIt configuration in openarm_ros2 isn't affected: its
arm groups end at joint7, and its end effectors are attached to
`*_hand`. The `*_hand_tcp` frame only appears in its RViz
configurations.


Validation: single-arm and bimanual TCP poses match MuJoCo at 103
configurations each. Prefix modes, ROS2 control, standalone expansion
and custom TCP overrides pass.

File: assets/robot/openarm_v1.0/urdf/ee/parallel_link/openarm_parallel_gripper.xacro (robot description, xacro)
@@ -14,5 +14,5 @@
 <robot xmlns:xacro="http://www.ros.org/wiki/xacro" name="parallel_gripper">
   <!-- tcp_xyz: offset from hand to hand_tcp (metres). -->
-  <xacro:macro name="openarm_parallel_gripper" params="connected_to:='' arm_type arm_prefix:='' ee_type ee_inertials ee_kinematics ee_kinematics_link ee_joints_limits rpy_ee:='0 0 0' xyz_ee:='0 0 0' tcp_xyz:='0 0 0.0859' tcp_rpy:='0 0 0' description_pkg:=openarm_description no_prefix:=false mesh_root:=''">
+  <xacro:macro name="openarm_parallel_gripper" params="connected_to:='' arm_type arm_prefix:='' ee_type ee_inertials ee_kinematics ee_kinematics_link ee_joints_limits rpy_ee:='0 0 0' xyz_ee:='0 0 0' tcp_xyz:='0 0 0.09' tcp_rpy:='0 0 0' description_pkg:=openarm_description no_prefix:=false mesh_root:=''">
     <xacro:property name="ee_prefix" value="${'' if no_prefix or arm_type == '' else 'openarm_' + arm_prefix}" />
     <xacro:property name="ee_mesh_root" value="${mesh_root if mesh_root != '' else 'package://' + description_pkg + '/assets/end_effector/parallel_link/meshes'}" />

File: assets/robot/openarm_v1.0/urdf/example/v1.urdf (robot description, URDF)
Before this commit: robot openarm, 26 links, 25 joints
Joints:
- joint openarm_left_hand_tcp_joint: origin xyz=0 0 0.0859 rpy=0 0 0 -> xyz=0 0 0.09 rpy=0 0 0
- joint openarm_right_hand_tcp_joint: origin xyz=0 0 0.0859 rpy=0 0 0 -> xyz=0 0 0.09 rpy=0 0 0
