Commit message: Align V1 TCP with the Isaac 193.1 mm reference

File: assets/end_effector/parallel_link/urdf/parallel_link_standalone.urdf.xacro (robot description, xacro)
@@ -17,5 +17,5 @@
   <xacro:arg name="ee_config_dir" default="$(find openarm_description)/assets/end_effector/parallel_link/config" />
   <xacro:arg name="mesh_root" default="$(find openarm_description)/assets/end_effector/parallel_link/meshes" />
-  <xacro:arg name="tcp_xyz" default="0 0 0.0859" />
+  <xacro:arg name="tcp_xyz" default="0 0 0.093" />
   <xacro:arg name="tcp_rpy" default="0 0 0" />
   <link name="base_link" />

File: assets/robot/openarm_v1.0/urdf/ee/ee_dispatcher.xacro (robot description, xacro)
@@ -14,5 +14,5 @@
 <robot xmlns:xacro="http://www.ros.org/wiki/xacro">
   <xacro:include filename="$(find openarm_description)/assets/robot/openarm_v1.0/urdf/ee/parallel_link/openarm_parallel_gripper.xacro" />
-  <xacro:macro name="openarm_ee" params="ee_type connected_to arm_type arm_prefix ee_kinematics ee_kinematics_link ee_inertials ee_joints_limits rpy_ee:='0 0 0' xyz_ee:='0 0 0' tcp_xyz:='0 0 0.0859' tcp_rpy:='0 0 0' description_pkg:=openarm_description no_prefix:=false">
+  <xacro:macro name="openarm_ee" params="ee_type connected_to arm_type arm_prefix ee_kinematics ee_kinematics_link ee_inertials ee_joints_limits rpy_ee:='0 0 0' xyz_ee:='0 0 0' tcp_xyz:='0 0 0.093' tcp_rpy:='0 0 0' description_pkg:=openarm_description no_prefix:=false">
     <xacro:if value="${ee_type == 'parallel_link'}">
       <xacro:openarm_parallel_gripper

File: assets/robot/openarm_v1.0/urdf/ee/parallel_link/openarm_parallel_gripper.xacro (robot description, xacro)
@@ -14,5 +14,5 @@
 <robot xmlns:xacro="http://www.ros.org/wiki/xacro" name="parallel_gripper">
   <!-- tcp_xyz: offset from hand to hand_tcp (metres). -->
-  <xacro:macro name="openarm_parallel_gripper" params="connected_to:='' arm_type arm_prefix:='' ee_type ee_inertials ee_kinematics ee_kinematics_link ee_joints_limits rpy_ee:='0 0 0' xyz_ee:='0 0 0' tcp_xyz:='0 0 0.0859' tcp_rpy:='0 0 0' description_pkg:=openarm_description no_prefix:=false mesh_root:=''">
+  <xacro:macro name="openarm_parallel_gripper" params="connected_to:='' arm_type arm_prefix:='' ee_type ee_inertials ee_kinematics ee_kinematics_link ee_joints_limits rpy_ee:='0 0 0' xyz_ee:='0 0 0' tcp_xyz:='0 0 0.093' tcp_rpy:='0 0 0' description_pkg:=openarm_description no_prefix:=false mesh_root:=''">
     <xacro:property name="ee_prefix" value="${'' if no_prefix or arm_type == '' else 'openarm_' + arm_prefix}" />
     <xacro:property name="ee_mesh_root" value="${mesh_root if mesh_root != '' else 'package://' + description_pkg + '/assets/end_effector/parallel_link/meshes'}" />

File: assets/robot/openarm_v1.0/urdf/example/v1.urdf (robot description, URDF)
Before this commit: robot openarm, 26 links, 25 joints
Joints:
- joint openarm_left_hand_tcp_joint: origin xyz=0 0 0.0859 rpy=0 0 0 -> xyz=0 0 0.093 rpy=0 0 0
- joint openarm_right_hand_tcp_joint: origin xyz=0 0 0.0859 rpy=0 0 0 -> xyz=0 0 0.093 rpy=0 0 0

Commit message: Generate the standalone V1 gripper with the shared macro

File: assets/end_effector/parallel_link/urdf/parallel_link_standalone.urdf.xacro (robot description, xacro)
@@ -13,90 +13,22 @@
 -->
 <robot xmlns:xacro="http://www.ros.org/wiki/xacro" name="parallel_link">
+  <xacro:include filename="$(find openarm_description)/assets/robot/openarm_v1.0/urdf/ee/openarm_ee_macro.xacro" />
+  <xacro:include filename="$(find openarm_description)/assets/robot/openarm_v1.0/urdf/ee/parallel_link/openarm_parallel_gripper.xacro" />
   <xacro:arg name="ee_config_dir" default="$(find openarm_description)/assets/end_effector/parallel_link/config" />
   <xacro:arg name="mesh_root" default="$(find openarm_description)/assets/end_effector/parallel_link/meshes" />
-  <xacro:arg name="tcp_xyz" default="0 0 0" />
+  <xacro:arg name="tcp_xyz" default="0 0 0.0835" />
   <xacro:arg name="tcp_rpy" default="0 0 0" />
-  <xacro:property name="ee_inertials" value="${xacro.load_yaml('$(arg ee_config_dir)/inertials.yaml')}" />
-  <xacro:property name="ee_kinematics" value="${xacro.load_yaml('$(arg ee_config_dir)/kinematics.yaml')}" />
-  <xacro:property name="ee_kinematics_link" value="${xacro.load_yaml('$(arg ee_config_dir)/kinematics_link.yaml')}" />
-  <xacro:property name="ee_joint_limits" value="${xacro.load_yaml('$(arg ee_config_dir)/joint_limits.yaml')}" />
-  <xacro:macro name="parallel_link_inertial" params="name">
-    <xacro:property name="I" value="${ee_inertials[name]}" lazy_eval="false" />
-    <inertial>
-      <origin
-        xyz="${I.origin.x} ${I.origin.y} ${I.origin.z}"
-        rpy="${I.origin.roll} ${I.origin.pitch} ${I.origin.yaw}" />
-      <mass value="${I.mass}" />
-      <inertia ixx="${I.inertia.xx}" ixy="${I.inertia.xy}" ixz="${I.inertia.xz}"
-               iyy="${I.inertia.yy}" iyz="${I.inertia.yz}" izz="${I.inertia.zz}" />
-    </inertial>
-  </xacro:macro>
-  <xacro:macro name="parallel_link_visual_collision" params="name mesh_name mesh_scale">
-    <xacro:property name="K" value="${ee_kinematics_link[name]['kinematic']}" lazy_eval="false" />
-    <visual name="${name}_visual">
-      <origin xyz="${K.x} ${K.y} ${K.z}" rpy="${K.roll} ${K.pitch} ${K.yaw}" />
-      <geometry>
-        <mesh filename="$(arg mesh_root)/visual/${mesh_name}.dae" scale="${mesh_scale}" />
-      </geometry>
-    </visual>
-    <collision name="${name}_collision">
-      <origin xyz="${K.x} ${K.y} ${K.z}" rpy="${K.roll} ${K.pitch} ${K.yaw}" />
-      <geometry>
-        <mesh filename="$(arg mesh_root)/collision/${mesh_name}.stl" scale="${mesh_scale}" />
-      </geometry>
-    </collision>
-  </xacro:macro>
-  <link name="base_link">
-    <visual name="base_link_visual">
-      <origin xyz="0 0 0" rpy="0 0 0" />
-      <geometry>
-        <mesh filename="$(arg mesh_root)/visual/hand.dae" scale="0.001 0.001 0.001" />
-      </geometry>
-    </visual>
-    <collision name="base_link_collision">
-      <origin xyz="0 0 0" rpy="0 0 0" />
-      <geometry>
-        <mesh filename="$(arg mesh_root)/collision/hand.stl" scale="0.001 0.001 0.001" />
-      </geometry>
-    </collision>
-  </link>
-  <link name="hand_tcp" />
-  <joint name="hand_tcp_joint" type="fixed">
-    <origin xyz="$(arg tcp_xyz)" rpy="$(arg tcp_rpy)" />
-    <parent link="base_link" />
-    <child link="hand_tcp" />
-  </joint>
-  <link name="right_finger">
-    <xacro:parallel_link_visual_collision name="right_finger" mesh_name="finger" mesh_scale="-0.001 0.001 0.001" />
-    <xacro:parallel_link_inertial name="right_finger" />
-  </link>
-  <link name="left_finger">
-    <xacro:parallel_link_visual_collision name="left_finger" mesh_name="finger" mesh_scale="0.001 0.001 0.001" />
-    <xacro:parallel_link_inertial name="left_finger" />
-  </link>
-  <joint name="finger_joint1" type="prismatic">
-    <parent link="base_link" />
-    <child link="right_finger" />
-    <xacro:property name="fj" value="${ee_kinematics['finger_joint']['kinematic']}" />
-    <origin xyz="${fj.x} ${fj.y} ${fj.z}" rpy="${fj.roll} ${fj.pitch} ${fj.yaw}" />
-    <axis xyz="0 -1 0" />
-    <limit
-      effort="${ee_joint_limits['finger_joint']['limit']['effort']}"
-      lower="${ee_joint_limits['finger_joint']['limit']['lower']}"
-      upper="${ee_joint_limits['finger_joint']['limit']['upper']}"
-      velocity="${ee_joint_limits['finger_joint']['limit']['velocity']}" />
-  </joint>
-  <joint name="finger_joint2" type="prismatic">
-    <parent link="base_link" />
-    <child link="left_finger" />
-    <xacro:property name="fj" value="${ee_kinematics['finger_joint']['kinematic']}" />
-    <origin xyz="${fj.x} ${-fj.y} ${fj.z}" rpy="${fj.roll} ${fj.pitch} ${fj.yaw}" />
-    <axis xyz="0 1 0" />
-    <limit
-      effort="${ee_joint_limits['finger_joint']['limit']['effort']}"
-      lower="${ee_joint_limits['finger_joint']['limit']['lower']}"
-      upper="${ee_joint_limits['finger_joint']['limit']['upper']}"
-      velocity="${ee_joint_limits['finger_joint']['limit']['velocity']}" />
-    <mimic joint="finger_joint1" />
-  </joint>
+  <link name="base_link" />
+  <xacro:openarm_parallel_gripper
+    connected_to="base_link"
+    arm_type=""
+    ee_type="parallel_link"
+    no_prefix="true"
+    mesh_root="$(arg mesh_root)"
+    tcp_xyz="$(arg tcp_xyz)"
+    tcp_rpy="$(arg tcp_rpy)"
+    ee_inertials="${xacro.load_yaml('$(arg ee_config_dir)/inertials.yaml')}"
+    ee_kinematics="${xacro.load_yaml('$(arg ee_config_dir)/kinematics.yaml')}"
+    ee_kinematics_link="${xacro.load_yaml('$(arg ee_config_dir)/kinematics_link.yaml')}"
+    ee_joints_limits="${xacro.load_yaml('$(arg ee_config_dir)/joint_limits.yaml')}" />
 </robot>

File: assets/robot/openarm_v1.0/urdf/ee/parallel_link/openarm_parallel_gripper.xacro (robot description, xacro)
@@ -18,6 +18,7 @@
     parallel-link gripper — measured from the hand frame origin.
   -->
-  <xacro:macro name="openarm_parallel_gripper" params="connected_to:='' arm_type arm_prefix:='' ee_type ee_inertials ee_kinematics ee_kinematics_link ee_joints_limits rpy_ee:='0 0 0' xyz_ee:='0 0 0' tcp_xyz:='0 0 0.0835' tcp_rpy:='0 0 0' description_pkg:=openarm_description no_prefix:=false">
+  <xacro:macro name="openarm_parallel_gripper" params="connected_to:='' arm_type arm_prefix:='' ee_type ee_inertials ee_kinematics ee_kinematics_link ee_joints_limits rpy_ee:='0 0 0' xyz_ee:='0 0 0' tcp_xyz:='0 0 0.0835' tcp_rpy:='0 0 0' description_pkg:=openarm_description no_prefix:=false mesh_root:=''">
     <xacro:property name="ee_prefix" value="${'' if no_prefix or arm_type == '' else 'openarm_' + arm_prefix}" />
+    <xacro:property name="ee_mesh_root" value="${mesh_root if mesh_root != '' else 'package://' + description_pkg + '/assets/end_effector/parallel_link/meshes'}" />
     <xacro:property name="finger_limits" value="${ee_joints_limits['finger_joint']['limit']}" />
     <link name="${ee_prefix}hand">
@@ -25,5 +26,5 @@
         <xacro:openarm-ee-kinematics-link config="${ee_kinematics_link}" name="hand" />
         <geometry>
-          <mesh filename="package://${description_pkg}/assets/end_effector/parallel_link/meshes/visual/hand.dae" scale="0.001 0.001 0.001"/>
+          <mesh filename="${ee_mesh_root}/visual/hand.dae" scale="0.001 0.001 0.001"/>
         </geometry>
       </visual>
@@ -31,5 +32,5 @@
         <xacro:openarm-ee-kinematics-link config="${ee_kinematics_link}" name="hand" />
         <geometry>
-          <mesh filename="package://${description_pkg}/assets/end_effector/parallel_link/meshes/collision/hand.stl" scale="0.001 0.001 0.001" />
+          <mesh filename="${ee_mesh_root}/collision/hand.stl" scale="0.001 0.001 0.001" />
         </geometry>
       </collision>
@@ -50,5 +51,5 @@
         <xacro:openarm-ee-kinematics-link config="${ee_kinematics_link}" name="left_finger" />
         <geometry>
-          <mesh filename="package://${description_pkg}/assets/end_effector/parallel_link/meshes/visual/finger.dae" scale="0.001 0.001 0.001"/>
+          <mesh filename="${ee_mesh_root}/visual/finger.dae" scale="0.001 0.001 0.001"/>
         </geometry>
       </visual>
@@ -56,5 +57,5 @@
         <xacro:openarm-ee-kinematics-link config="${ee_kinematics_link}" name="left_finger" />
         <geometry>
-          <mesh filename="package://${description_pkg}/assets/end_effector/parallel_link/meshes/collision/finger.stl" scale="0.001 0.001 0.001" />
+          <mesh filename="${ee_mesh_root}/collision/finger.stl" scale="0.001 0.001 0.001" />
         </geometry>
       </collision>
@@ -65,5 +66,5 @@
         <xacro:openarm-ee-kinematics-link config="${ee_kinematics_link}" name="right_finger" />
         <geometry>
-          <mesh filename="package://${description_pkg}/assets/end_effector/parallel_link/meshes/visual/finger.dae" scale="0.001 -0.001 0.001"/>
+          <mesh filename="${ee_mesh_root}/visual/finger.dae" scale="0.001 -0.001 0.001"/>
         </geometry>
       </visual>
@@ -71,5 +72,5 @@
         <xacro:openarm-ee-kinematics-link config="${ee_kinematics_link}" name="right_finger" />
         <geometry>
-          <mesh filename="package://${description_pkg}/assets/end_effector/parallel_link/meshes/collision/finger.stl" scale="0.001 -0.001 0.001" />
+          <mesh filename="${ee_mesh_root}/collision/finger.stl" scale="0.001 -0.001 0.001" />
         </geometry>
       </collision>

Commit message: Attach V1 fingers to hand and correct gripper origins

File: assets/end_effector/parallel_link/urdf/parallel_link_standalone.urdf.xacro (robot description, xacro)
@@ -17,5 +17,5 @@
   <xacro:arg name="ee_config_dir" default="$(find openarm_description)/assets/end_effector/parallel_link/config" />
   <xacro:arg name="mesh_root" default="$(find openarm_description)/assets/end_effector/parallel_link/meshes" />
-  <xacro:arg name="tcp_xyz" default="0 0 0.0835" />
+  <xacro:arg name="tcp_xyz" default="0 0 0.0859" />
   <xacro:arg name="tcp_rpy" default="0 0 0" />
   <link name="base_link" />

File: assets/robot/openarm_v1.0/urdf/ee/parallel_link/openarm_parallel_gripper.xacro (robot description, xacro)
@@ -13,10 +13,6 @@
 -->
 <robot xmlns:xacro="http://www.ros.org/wiki/xacro" name="parallel_gripper">
-  <!--
-    tcp_xyz: offset from hand link to hand_tcp along +Z of hand (metres).
-    Default 0 0 0.0835 is the calibrated fingertip-centre offset for the
-    parallel-link gripper — measured from the hand frame origin.
-  -->
-  <xacro:macro name="openarm_parallel_gripper" params="connected_to:='' arm_type arm_prefix:='' ee_type ee_inertials ee_kinematics ee_kinematics_link ee_joints_limits rpy_ee:='0 0 0' xyz_ee:='0 0 0' tcp_xyz:='0 0 0.0835' tcp_rpy:='0 0 0' description_pkg:=openarm_description no_prefix:=false mesh_root:=''">
+  <!-- tcp_xyz: offset from hand to hand_tcp (metres). -->
+  <xacro:macro name="openarm_parallel_gripper" params="connected_to:='' arm_type arm_prefix:='' ee_type ee_inertials ee_kinematics ee_kinematics_link ee_joints_limits rpy_ee:='0 0 0' xyz_ee:='0 0 0' tcp_xyz:='0 0 0.0859' tcp_rpy:='0 0 0' description_pkg:=openarm_description no_prefix:=false mesh_root:=''">
     <xacro:property name="ee_prefix" value="${'' if no_prefix or arm_type == '' else 'openarm_' + arm_prefix}" />
     <xacro:property name="ee_mesh_root" value="${mesh_root if mesh_root != '' else 'package://' + description_pkg + '/assets/end_effector/parallel_link/meshes'}" />
@@ -78,5 +74,5 @@
     </link>
     <joint name="${ee_prefix}finger_joint1" type="prismatic">
-        <parent link="${connected_to}" />
+        <parent link="${ee_prefix}hand" />
         <child link="${ee_prefix}right_finger" />
         <xacro:openarm-ee-kinematics config="${ee_kinematics}" name="finger_joint" />
@@ -86,5 +82,5 @@
     </joint>
     <joint name="${ee_prefix}finger_joint2" type="prismatic">
-        <parent link="${connected_to}" />
+        <parent link="${ee_prefix}hand" />
         <child link="${ee_prefix}left_finger" />
         <xacro:property name="fj" value="${ee_kinematics['finger_joint']['kinematic']}" />
@@ -95,17 +91,4 @@
         <mimic joint="${ee_prefix}finger_joint1" />
     </joint>
-    <!-- <joint name="${ee_prefix}finger_joint1" type="prismatic">
-      <parent link="${connected_to}" /> <child link="${ee_prefix}right_finger" />
-      <origin xyz="0 -0.006 0.115" rpy="0 0 0" />
-      <axis xyz="0 -1 0" />
-      <limit effort="333" lower="0.0" upper="0.044" velocity="10.0" />
-    </joint>
-    <joint name="${ee_prefix}finger_joint2" type="prismatic">
-      <parent link="${connected_to}" /> <child link="${ee_prefix}left_finger" />
-      <origin xyz="0 0.006 0.115" rpy="0 0 0" />
-      <axis xyz="0 1 0" />
-      <limit effort="333" lower="0.0" upper="0.044" velocity="10.0" />
-      <mimic joint="${ee_prefix}finger_joint1" />
-    </joint> -->
   </xacro:macro>
 </robot>

File: assets/robot/openarm_v1.0/urdf/example/v1.urdf (robot description, URDF)
Before this commit: robot openarm, 26 links, 25 joints
Joints:
- joint openarm_left_finger_joint1: origin xyz=0.0 -0.005 0.1025 rpy=0 0 0 -> xyz=0.0 -0.005 0.015 rpy=0 0 0; parent openarm_left_link7 -> openarm_left_hand
- joint openarm_left_finger_joint2: origin xyz=0.0 0.005 0.1025 rpy=0 0 0 -> xyz=0.0 0.005 0.015 rpy=0 0 0; parent openarm_left_link7 -> openarm_left_hand
- joint openarm_left_hand_joint: origin xyz=0.0 0.0 0.1025 rpy=0 0 0 -> xyz=0.0 0.0 0.1001 rpy=0 0 0
- joint openarm_left_hand_tcp_joint: origin xyz=0 0 0.0835 rpy=0 0 0 -> xyz=0 0 0.0859 rpy=0 0 0
- joint openarm_right_finger_joint1: origin xyz=0.0 -0.005 0.1025 rpy=0 0 0 -> xyz=0.0 -0.005 0.015 rpy=0 0 0; parent openarm_right_link7 -> openarm_right_hand
- joint openarm_right_finger_joint2: origin xyz=0.0 0.005 0.1025 rpy=0 0 0 -> xyz=0.0 0.005 0.015 rpy=0 0 0; parent openarm_right_link7 -> openarm_right_hand
- joint openarm_right_hand_joint: origin xyz=0.0 0.0 0.1025 rpy=0 0 0 -> xyz=0.0 0.0 0.1001 rpy=0 0 0
- joint openarm_right_hand_tcp_joint: origin xyz=0 0 0.0835 rpy=0 0 0 -> xyz=0 0 0.0859 rpy=0 0 0
