Commit message: Correct V1 parallel gripper force and velocity limits

File: assets/robot/openarm_v1.0/urdf/example/v1.urdf (robot description, URDF)
Before this commit: robot openarm, 26 links, 25 joints
Joints:
- joint openarm_left_finger_joint1: limit lower=0.0 upper=0.044 effort=333 velocity=10.0 -> lower=0.0 upper=0.044 effort=150.75 velocity=0.661
- joint openarm_left_finger_joint2: limit lower=0.0 upper=0.044 effort=333 velocity=10.0 -> lower=0.0 upper=0.044 effort=150.75 velocity=0.661
- joint openarm_right_finger_joint1: limit lower=0.0 upper=0.044 effort=333 velocity=10.0 -> lower=0.0 upper=0.044 effort=150.75 velocity=0.661
- joint openarm_right_finger_joint2: limit lower=0.0 upper=0.044 effort=333 velocity=10.0 -> lower=0.0 upper=0.044 effort=150.75 velocity=0.661

Commit message: Refresh the V1 example URDF from its Xacro source

File: assets/robot/openarm_v1.0/urdf/example/v1.urdf (robot description, URDF)
Before this commit: robot openarm, 24 links, 23 joints
Links:
- added link openarm_left_hand, mass 0.127; collision mesh filename=package://openarm_description/assets/end_effector/parallel_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 scale=0.001 0.001 0.001; visual mesh filename=package://openarm_description/assets/end_effector/parallel_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 scale=0.001 0.001 0.001
- added link openarm_right_hand, mass 0.127; collision mesh filename=package://openarm_description/assets/end_effector/parallel_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 scale=0.001 0.001 0.001; visual mesh filename=package://openarm_description/assets/end_effector/parallel_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 scale=0.001 0.001 0.001
Joints:
- added joint openarm_left_hand_joint: type fixed, parent openarm_left_link7, child openarm_left_hand, origin xyz=0.0 0.0 0.1025 rpy=0 0 0
- added joint openarm_right_hand_joint: type fixed, parent openarm_right_link7, child openarm_right_hand, origin xyz=0.0 0.0 0.1025 rpy=0 0 0
- joint openarm_left_finger_joint1: origin xyz=0.0 0.0 0.1025 rpy=0 0 0 -> xyz=0.0 -0.005 0.1025 rpy=0 0 0
- joint openarm_left_finger_joint2: origin xyz=0.0 -0.0 0.1025 rpy=0 0 0 -> xyz=0.0 0.005 0.1025 rpy=0 0 0
- joint openarm_left_hand_tcp_joint: origin xyz=0 0 0 rpy=0 0 0 -> xyz=0 0 0.0835 rpy=0 0 0; parent openarm_left_link7 -> openarm_left_hand
- joint openarm_right_finger_joint1: origin xyz=0.0 0.0 0.1025 rpy=0 0 0 -> xyz=0.0 -0.005 0.1025 rpy=0 0 0
- joint openarm_right_finger_joint2: origin xyz=0.0 -0.0 0.1025 rpy=0 0 0 -> xyz=0.0 0.005 0.1025 rpy=0 0 0
- joint openarm_right_hand_tcp_joint: origin xyz=0 0 0 rpy=0 0 0 -> xyz=0 0 0.0835 rpy=0 0 0; parent openarm_right_link7 -> openarm_right_hand

Commit message: Update V1 link7, hand and finger inertial allocation

File: assets/robot/openarm_v1.0/urdf/example/v1.urdf (robot description, URDF)
Before this commit: robot openarm, 26 links, 25 joints
Links:
- link openarm_left_hand: mass 0.127 -> 0.1723111736408497
- link openarm_left_left_finger: mass 0.03602545343277134 -> 0.07444998664008126
- link openarm_left_link7: mass 0.4659771327380578 -> 0.4054971268153967
- link openarm_left_right_finger: mass 0.03602545343277134 -> 0.07444998664008126
- link openarm_right_hand: mass 0.127 -> 0.1723111736408497
- link openarm_right_left_finger: mass 0.03602545343277134 -> 0.07444998664008126
- link openarm_right_link7: mass 0.4659771327380578 -> 0.4054971268153967
- link openarm_right_right_finger: mass 0.03602545343277134 -> 0.07444998664008126

Commit message: Update V1 and V2 base mass and diagonal inertia

File: assets/robot/openarm_v1.0/urdf/example/v1.urdf (robot description, URDF)
Before this commit: robot openarm, 26 links, 25 joints
Links:
- link openarm_body_link0: mass 13.89 -> 3.74

File: assets/robot/openarm_v2.0/urdf/example/v2.urdf (robot description, URDF)
Before this commit: robot openarm_v20, 22 links, 21 joints
Links:
- link openarm_body_link0: mass 13.89 -> 3.74

Commit message: Update V1 and V2 base mass and diagonal inertia

File: assets/robot/openarm_v1.0/urdf/example/v1.urdf (robot description, URDF)
Before this commit: robot openarm, 26 links, 25 joints
Links:
- link openarm_body_link0: mass 13.89 -> 3.74

Commit message: Fix V1 and V2 bimanual mounting origins

File: assets/robot/openarm_v1.0/urdf/example/v1.urdf (robot description, URDF)
Before this commit: robot openarm, 26 links, 25 joints
Joints:
- joint openarm_left_openarm_body_link0_joint: origin xyz=0.0 0.031 0.698 rpy=-1.5708 0 0 -> xyz=0.0 0.030 0.697 rpy=-1.5708 0 0
- joint openarm_right_openarm_body_link0_joint: origin xyz=0.0 -0.031 0.698 rpy=1.5708 0 0 -> xyz=0.0 -0.030 0.697 rpy=1.5708 0 0

File: assets/robot/openarm_v1.0/urdf/openarm_v10.urdf.xacro (robot description, xacro)
@@ -29,7 +29,7 @@
   <xacro:arg name="fake_sensor_commands" default="false" />
   <xacro:arg name="bimanual" default="true" />
-  <xacro:arg name="right_arm_base_xyz" default="0.0 -0.031 0.698" />
+  <xacro:arg name="right_arm_base_xyz" default="0.0 -0.030 0.697" />
   <xacro:arg name="right_arm_base_rpy" default="1.5708 0 0" />
-  <xacro:arg name="left_arm_base_xyz" default="0.0 0.031 0.698" />
+  <xacro:arg name="left_arm_base_xyz" default="0.0 0.030 0.697" />
   <xacro:arg name="left_arm_base_rpy" default="-1.5708 0 0" />
   <xacro:arg name="can_fd" default="true" />

File: assets/robot/openarm_v2.0/urdf/example/v2.urdf (robot description, URDF)
Before this commit: robot openarm_v20, 22 links, 21 joints
Joints:
- joint openarm_left_base_link_mount_joint: origin xyz=0.0 0.031 0.698 rpy=0.0 0.0 0.0 -> xyz=0.0 0.03 0.697 rpy=0.0 0.0 0.0
- joint openarm_right_base_link_mount_joint: origin xyz=0.0 -0.031 0.698 rpy=0.0 0.0 0.0 -> xyz=0.0 -0.03 0.697 rpy=0.0 0.0 0.0
