Commit message: fix: preserve embedded DAE materials in v2.0

File: assets/robot/openarm_v2.0/urdf/utils/openarm_v20_ee.xacro (robot description, xacro)
@@ -51,4 +51,5 @@
             <xacro:openarm_v20_emit_origin origin="${base_visual_cfg.origin}" reflect_x="${reflect_x if base_link_reflects else 1}" reflect_y="${reflect_y if base_link_reflects else 1}" reflect_z="${reflect_z if base_link_reflects else 1}" />
           </xacro:unless>
+          <!-- Preserve the mesh's embedded materials. -->
           <geometry>
             <mesh
@@ -56,7 +57,4 @@
               scale="${(reflect_x if base_link_reflects else 1) * base_visual_cfg.geometry.scale.x} ${(reflect_y if base_link_reflects else 1) * base_visual_cfg.geometry.scale.y} ${(reflect_z if base_link_reflects else 1) * base_visual_cfg.geometry.scale.z}" />
           </geometry>
-          <material name="${base_link_full_name}_material">
-            <color rgba="0.752941176470588 0.752941176470588 0.752941176470588 1" />
-          </material>
         </visual>
       </xacro:if>

File: assets/robot/openarm_v2.0/urdf/utils/openarm_v20_utils.xacro (robot description, xacro)
@@ -94,4 +94,5 @@
             <xacro:openarm_v20_emit_origin origin="${visual_cfg.origin}" reflect_x="${reflect_x}" reflect_y="${reflect_y}" reflect_z="${reflect_z}" />
           </xacro:unless>
+          <!-- Preserve the mesh's embedded materials. -->
           <geometry>
             <mesh
@@ -99,7 +100,4 @@
               scale="${reflect_x * visual_cfg.geometry.scale.x} ${reflect_y * visual_cfg.geometry.scale.y} ${reflect_z * visual_cfg.geometry.scale.z}" />
           </geometry>
-          <material name="${link_name}_material">
-            <color rgba="0.752941176470588 0.752941176470588 0.752941176470588 1" />
-          </material>
         </visual>
       </xacro:if>

Commit message: Keep V2 mounting poses independent of reference frame emission

File: assets/robot/openarm_v2.0/urdf/utils/openarm_v20_ee.xacro (robot description, xacro)
@@ -116,5 +116,5 @@
     <xacro:unless value="${skip_mount_joint}">
       <joint name="${prefix}ee_mount_joint" type="fixed">
-        <xacro:openarm_v20_emit_origin origin="${resolved_mount_origin}" reflect_x="${reflect_x}" reflect_y="${reflect_y}" reflect_z="${reflect_z}" />
+        <xacro:openarm_v20_emit_origin origin="${resolved_mount_origin}" />
         <parent link="${connected_to}" />
         <child link="${base_link_full_name}" />
@@ -196,20 +196,7 @@
       </xacro:if>
     </joint>
-    <!-- Optionally expose a grasp helper frame from EE reference_points.yaml. -->
-    <xacro:if value="${emit_grasp_frame and grasp_reference_point in ee_reference_points}">
-      <xacro:property name="grasp_ref" value="${ee_reference_points[grasp_reference_point]}" lazy_eval="false" />
-      <xacro:property name="grasp_ref_parent" value="${prefix + 'ee_' + grasp_ref['parent']}" lazy_eval="false" />
-      <xacro:property name="grasp_ref_reflects" value="${component_reflects and grasp_reference_point in reflect_include_reference_points}" lazy_eval="false" />
-      <xacro:openarm_v20_emit_reference_link
-        link_name="${prefix + grasp_reference_point}"
-        parent_link="${grasp_ref_parent}"
-        origin="${grasp_ref['origin']}"
-        reflect_x="${reflect_x if grasp_ref_reflects else 1}"
-        reflect_y="${reflect_y if grasp_ref_reflects else 1}"
-        reflect_z="${reflect_z if grasp_ref_reflects else 1}"
-        frame_shift="${resolved_base_frame_shift if use_base_frame_shift else 'none'}" />
-    </xacro:if>
     <xacro:openarm_v20_emit_reference_frames
       reference_points="${ee_reference_points}"
+      force_emit_reference="${grasp_reference_point if emit_grasp_frame else ''}"
       prefix="${prefix}" link_prefix="${prefix + 'ee_'}"
       base_link_name="${base_link_name}"

File: assets/robot/openarm_v2.0/urdf/utils/openarm_v20_robot.xacro (robot description, xacro)
@@ -256,5 +256,5 @@
   <!-- Resolve runtime assembly data from a static descriptor plus preset overrides. -->
   <xacro:macro name="openarm_v20_resolve_component_runtime"
-    params="component_name components robot_preset config_root root_frame component_cfg component_desc parent_desc:=none collapse_internal_empty_links:=false out_name">
+    params="component_name components robot_preset config_root root_frame component_cfg component_desc parent_desc:=none collapse_internal_empty_links:=false emit_grasp_frame:=false out_name">
     <xacro:property name="none_value" value="${'none'}" lazy_eval="false" />
     <xacro:property name="zero_origin" value="${dict(x=0.0, y=0.0, z=0.0, roll=0.0, pitch=0.0, yaw=0.0)}" lazy_eval="false" />
@@ -285,5 +285,12 @@
     <xacro:property name="has_parent_override" value="${'parent' in connection and connection['parent'] != None}" lazy_eval="false" />
     <xacro:property name="has_origin_override" value="${'origin' in connection and connection['origin'] != None}" lazy_eval="false" />
-    <!-- Start from defaults, then let reference-point lookup and explicit overrides refine the mount. -->
+    <xacro:openarm_v20_require
+      condition="${not (has_parent_reference_key and has_parent_override)}"
+      message="${'Component `%s` must choose parent or parent_reference_point, not both.' % component_name}" />
+    <xacro:property name="origin_cfg" value="${connection['origin'] if has_origin_override else zero_origin}" lazy_eval="false" />
+    <xacro:property name="connection_origin"
+      value="${dict(x=origin_cfg.get('x') or 0.0, y=origin_cfg.get('y') or 0.0, z=origin_cfg.get('z') or 0.0, roll=origin_cfg.get('roll') or 0.0, pitch=origin_cfg.get('pitch') or 0.0, yaw=origin_cfg.get('yaw') or 0.0)}"
+      lazy_eval="false" />
+    <xacro:property name="resolved_mount_origin" value="${connection_origin}" lazy_eval="false" />
     <xacro:if value="${has_parent_reference_key}">
       <xacro:openarm_v20_require
@@ -302,37 +309,21 @@
       <xacro:property name="parent_ref_should_reflect" value="${parent_component_reflects and parent_ref_name in parent_reflect_include_reference_points}" lazy_eval="false" />
       <xacro:property name="parent_ref_canonical_link" value="${parent_ref['parent']}" lazy_eval="false" />
-      <xacro:property
-        name="resolved_connected_to"
-        value="${parent_desc['link_name_map'][parent_ref_canonical_link] if parent_ref_canonical_link in parent_desc['link_name_map'] else parent_desc['link_prefix'] + parent_ref_canonical_link}"
-        lazy_eval="false" />
-      <xacro:property
-        name="resolved_mount_origin"
-        value="${dict(x=((parent_reflect_cfg['x'] * parent_ref['origin']['x']) if parent_ref_should_reflect else parent_ref['origin']['x']),
-                     y=((parent_reflect_cfg['y'] * parent_ref['origin']['y']) if parent_ref_should_reflect else parent_ref['origin']['y']),
-                     z=((parent_reflect_cfg['z'] * parent_ref['origin']['z']) if parent_ref_should_reflect else parent_ref['origin']['z']),
-                     roll=parent_ref['origin']['roll'],
-                     pitch=parent_ref['origin']['pitch'],
-                     yaw=parent_ref['origin']['yaw'])}"
-        lazy_eval="false" />
-      <xacro:if value="${parent_ref.get('emit', False)}">
+      <xacro:property name="resolved_connected_to"
+        value="${parent_desc['link_name_map'][parent_ref_canonical_link] if parent_ref_canonical_link in parent_desc['link_name_map'] else parent_desc['link_prefix'] + parent_ref_canonical_link}" lazy_eval="false" />
+      <xacro:property name="reference_origin" value="${parent_ref['origin']}" lazy_eval="false" />
+      <xacro:if value="${parent_ref_canonical_link == parent_desc['topology']['links'][0] and parent_desc.get('base_frame_shift', 'none') != 'none'}">
+        <xacro:openarm_v20_compose_pose first="${parent_desc['base_frame_shift']}" second="${reference_origin}" out_name="reference_origin" />
+      </xacro:if>
+      <xacro:if value="${parent_ref_should_reflect}">
+        <xacro:openarm_v20_reflect_pose origin="${reference_origin}" reflect_x="${parent_reflect_cfg['x']}" reflect_y="${parent_reflect_cfg['y']}" reflect_z="${parent_reflect_cfg['z']}" out_name="reference_origin" />
+      </xacro:if>
+      <xacro:openarm_v20_compose_pose first="${reference_origin}" second="${connection_origin}" out_name="reference_mount_origin" />
+      <xacro:property name="resolved_mount_origin" value="${reference_mount_origin}" lazy_eval="false" />
+      <xacro:property name="parent_reference_emitted" value="${parent_ref.get('emit', False) or (emit_grasp_frame and parent_desc['component_type'] == 'end_effector' and parent_ref_name == 'grasp_frame')}" lazy_eval="false" />
+      <xacro:if value="${parent_reference_emitted}">
         <xacro:property name="reference_prefix" value="${parent_desc['root_link_actual'] + '_' if parent_desc['component_type'] == 'body' else parent_desc['prefix']}" lazy_eval="false" />
         <xacro:property name="resolved_connected_to" value="${reference_prefix + parent_ref_name}" lazy_eval="false" />
-        <xacro:property name="resolved_mount_origin" value="${zero_origin}" lazy_eval="false" />
-      </xacro:if>
-    </xacro:if>
-    <xacro:if value="${has_parent_override}">
-      <xacro:property name="resolved_connected_to" value="${connection['parent']}" lazy_eval="false" />
-    </xacro:if>
-    <xacro:if value="${has_origin_override}">
-      <xacro:property name="origin_override" value="${connection['origin']}" lazy_eval="false" />
-      <xacro:property
-        name="resolved_mount_origin"
-        value="${dict(x=(origin_override['x'] if origin_override['x'] != None else resolved_mount_origin['x']),
-                     y=(origin_override['y'] if origin_override['y'] != None else resolved_mount_origin['y']),
-                     z=(origin_override['z'] if origin_override['z'] != None else resolved_mount_origin['z']),
-                     roll=(origin_override['roll'] if origin_override['roll'] != None else resolved_mount_origin['roll']),
-                     pitch=(origin_override['pitch'] if origin_override['pitch'] != None else resolved_mount_origin['pitch']),
-                     yaw=(origin_override['yaw'] if origin_override['yaw'] != None else resolved_mount_origin['yaw']))}"
-        lazy_eval="false" />
+        <xacro:property name="resolved_mount_origin" value="${connection_origin}" lazy_eval="false" />
+      </xacro:if>
     </xacro:if>
     <!-- reference point child empty links are already absorbed into config; runtime collapse only targets the parent's terminal empty link -->
@@ -343,5 +334,5 @@
     <xacro:if value="${has_parent_reference_key and not has_parent_override and collapse_internal_empty_links and parent_terminal_link_empty and parent_ref_canonical_link == parent_desc['topology']['links'][-1]}">
       <xacro:property name="skip_mount_joint" value="${True}" lazy_eval="false" />
-      <xacro:property name="base_frame_shift" value="${resolved_mount_origin}" lazy_eval="false" />
+      <xacro:openarm_v20_reflect_pose origin="${reference_mount_origin}" reflect_x="${reflect_x}" reflect_y="${reflect_y}" reflect_z="${reflect_z}" out_name="base_frame_shift" />
     </xacro:if>
     <!-- A parent can expose at most one child that consumes its terminal empty link. -->
@@ -511,5 +502,9 @@
       parent_desc="${parent_desc}"
       collapse_internal_empty_links="${collapse_internal_empty_links}"
+      emit_grasp_frame="${emit_grasp_frame}"
       out_name="component_runtime" />
+    <xacro:property name="runtime_link_name_map"
+      value="${dict(list(component_desc['link_name_map'].items()) + ([(component_runtime['collapse_source_link'], component_runtime['collapse_child_link'])] if component_runtime['collapse_source_link'] != 'none' else []))}" lazy_eval="false" />
+    <xacro:property name="component_desc" value="${dict(component_desc, link_name_map=runtime_link_name_map, base_frame_shift=component_runtime['base_frame_shift'])}" lazy_eval="false" />
     <xacro:openarm_v20_emit_component_from_runtime
       component_desc="${component_desc}"

File: assets/robot/openarm_v2.0/urdf/utils/openarm_v20_utils.xacro (robot description, xacro)
@@ -20,5 +20,5 @@
   </xacro:macro>
   <!-- Compose two poses in xacro so mount transforms can be absorbed into geometry or joints. -->
-  <xacro:macro name="openarm_v20_emit_composed_origin" params="first second reflect_x:=1 reflect_y:=1 reflect_z:=1 reflect_position:=true reflect_rotation:=${False}">
+  <xacro:macro name="openarm_v20_compose_pose" params="first second out_name">
     <xacro:property name="a_r" value="${first['roll']}" />
     <xacro:property name="a_p" value="${first['pitch']}" />
@@ -71,7 +71,14 @@
     <xacro:property name="rp" value="${atan2(-c31, cy_norm)}" />
     <xacro:property name="ry" value="${atan2(c21, c11) if cy_norm > 1e-9 else 0.0}" />
-    <origin
-      xyz="${(reflect_x * tx) if reflect_position else tx} ${(reflect_y * ty) if reflect_position else ty} ${(reflect_z * tz) if reflect_position else tz}"
-      rpy="${reflect_y * reflect_z * rr if reflect_rotation else rr} ${reflect_x * reflect_z * rp if reflect_rotation else rp} ${reflect_x * reflect_y * ry if reflect_rotation else ry}" />
+    <xacro:property name="${out_name}" value="${dict(x=tx, y=ty, z=tz, roll=rr, pitch=rp, yaw=ry)}" scope="parent" lazy_eval="false" />
+  </xacro:macro>
+  <xacro:macro name="openarm_v20_reflect_pose" params="origin reflect_x:=1 reflect_y:=1 reflect_z:=1 out_name">
+    <xacro:property name="${out_name}"
+      value="${dict(x=reflect_x * origin['x'], y=reflect_y * origin['y'], z=reflect_z * origin['z'], roll=reflect_y * reflect_z * origin['roll'], pitch=reflect_x * reflect_z * origin['pitch'], yaw=reflect_x * reflect_y * origin['yaw'])}"
+      scope="parent" lazy_eval="false" />
+  </xacro:macro>
+  <xacro:macro name="openarm_v20_emit_composed_origin" params="first second reflect_x:=1 reflect_y:=1 reflect_z:=1 reflect_position:=true reflect_rotation:=${False}">
+    <xacro:openarm_v20_compose_pose first="${first}" second="${second}" out_name="composed_origin" />
+    <xacro:openarm_v20_emit_origin origin="${composed_origin}" reflect_x="${reflect_x}" reflect_y="${reflect_y}" reflect_z="${reflect_z}" reflect_position="${reflect_position}" reflect_rotation="${reflect_rotation}" />
   </xacro:macro>
   <xacro:macro name="openarm_v20_emit_limit" params="limit">
@@ -201,10 +208,10 @@
   </xacro:macro>
   <xacro:macro name="openarm_v20_emit_reference_frames"
-    params="reference_points prefix link_prefix link_name_map:=${dict()} base_link_name:='' reflect_x:=1 reflect_y:=1 reflect_z:=1 reflect_include_reference_points:=^ frame_shift:=none index:=0">
+    params="reference_points prefix link_prefix link_name_map:=${dict()} base_link_name:='' reflect_x:=1 reflect_y:=1 reflect_z:=1 reflect_include_reference_points:=^ frame_shift:=none force_emit_reference:='' index:=0">
     <xacro:property name="reference_names" value="${list(reference_points.keys())}" lazy_eval="false" />
     <xacro:if value="${index &lt; len(reference_names)}">
       <xacro:property name="reference_name" value="${reference_names[index]}" lazy_eval="false" />
       <xacro:property name="reference" value="${reference_points[reference_name]}" lazy_eval="false" />
-      <xacro:if value="${reference.get('emit', False)}">
+      <xacro:if value="${reference.get('emit', False) or reference_name == force_emit_reference}">
         <xacro:property name="reference_parent" value="${reference['parent']}" lazy_eval="false" />
         <xacro:property name="reference_reflects" value="${reference_name in reflect_include_reference_points}" lazy_eval="false" />
@@ -223,5 +230,5 @@
         reflect_x="${reflect_x}" reflect_y="${reflect_y}" reflect_z="${reflect_z}"
         reflect_include_reference_points="${reflect_include_reference_points}"
-        frame_shift="${frame_shift}" index="${index + 1}" />
+        frame_shift="${frame_shift}" force_emit_reference="${force_emit_reference}" index="${index + 1}" />
     </xacro:if>
   </xacro:macro>
