Commit message: Generate V2 control interfaces from enabled preset components

File: assets/robot/openarm_v2.0/urdf/openarm_v20.urdf.xacro (robot description, xacro)
@@ -14,8 +14,10 @@
 <robot xmlns:xacro="http://www.ros.org/wiki/xacro" name="openarm_v20">
   <xacro:include filename="$(find openarm_description)/assets/robot/openarm_v2.0/urdf/utils/openarm_v20_robot.xacro" />
-  <xacro:include filename="$(find openarm_description)/assets/robot/openarm_v2.0/urdf/ros2_control/openarm.bimanual.ros2_control.xacro" />
+  <xacro:include filename="$(find openarm_description)/assets/robot/openarm_v2.0/urdf/ros2_control/openarm_robot.ros2_control.xacro" />
   <xacro:arg name="robot_preset" default="default_bimanual" />
   <xacro:arg name="collapse_internal_empty_links" default="true" />
   <xacro:arg name="emit_grasp_frame" default="false" />
+  <xacro:arg name="ros2_control" default="true" />
+  <xacro:arg name="fake_sensor_commands" default="false" />
   <xacro:arg name="use_fake_hardware" default="true" />
   <xacro:arg name="left_can_interface" default="can1" />
@@ -30,20 +32,8 @@
     collapse_internal_empty_links="$(arg collapse_internal_empty_links)"
     emit_grasp_frame="$(arg emit_grasp_frame)" />
-  <xacro:property name="gains_file" value="${config_root}/arm/control/control_gains.yaml" />
-  <xacro:property name="gains_dict" value="${xacro.load_yaml(gains_file)}" />
-  <xacro:property name="pinch_mimics_file" value="$(find openarm_description)/assets/end_effector/pinch_gripper/config/joint/joint_mimics.yaml" />
-  <xacro:property name="pinch_mimics_dict" value="${xacro.load_yaml(pinch_mimics_file)}" />
-  <xacro:property name="pinch_finger_mimic_multiplier" value="${pinch_mimics_dict['joint2']['multiplier'] if 'joint2' in pinch_mimics_dict else 1.0}" />
-  <xacro:openarm_bimanual_ros2_control
-    arm_type="v20"
-    control_gains="${gains_dict}"
-    use_fake_hardware="$(arg use_fake_hardware)"
-    left_can_interface="$(arg left_can_interface)"
-    right_can_interface="$(arg right_can_interface)"
-    can_fd="$(arg can_fd)"
-    ee_type="pinch_gripper"
-    left_arm_prefix="left_"
-    right_arm_prefix="right_"
-    left_finger_mimic_multiplier="${pinch_finger_mimic_multiplier}"
-    right_finger_mimic_multiplier="${pinch_finger_mimic_multiplier}" />
+  <xacro:if value="$(arg ros2_control)">
+    <xacro:openarm_v20_ros2_control robot_preset="${robot_preset_cfg}" config_root="${config_root}"
+      can_interfaces="${dict(left='$(arg left_can_interface)', right='$(arg right_can_interface)')}"
+      use_fake_hardware="$(arg use_fake_hardware)" fake_sensor_commands="$(arg fake_sensor_commands)" can_fd="$(arg can_fd)" />
+  </xacro:if>
 </robot>

File: assets/robot/openarm_v2.0/urdf/ros2_control/openarm.ros2_control.xacro (robot description, xacro)
@@ -13,20 +13,25 @@
 -->
 <robot xmlns:xacro="http://www.ros.org/wiki/xacro">
-<xacro:macro name="openarm_arm_ros2_control"
-         params="arm_type
-             control_gains
-             can_interface
-             use_fake_hardware:=^|false
-             fake_sensor_commands:=^|false
-             hand:=^|false
-             ee_type:=^|parallel_link
-             gazebo_effort:=^|false
-             arm_prefix:=''
-             bimanual:=false
-             can_fd:=^|true">
-    <ros2_control name="openarm_hardware_interface" type="system">
+  <xacro:macro name="openarm_v20_control_joint" params="joint_name">
+    <joint name="${joint_name}">
+      <command_interface name="position" />
+      <command_interface name="velocity" />
+      <command_interface name="effort" />
+      <state_interface name="position"><param name="initial_value">0.0</param></state_interface>
+      <state_interface name="velocity"><param name="initial_value">0.0</param></state_interface>
+      <state_interface name="effort"><param name="initial_value">0.0</param></state_interface>
+    </joint>
+  </xacro:macro>
+  <xacro:macro name="openarm_v20_control_joints" params="joint_names index:=0">
+    <xacro:if value="${index &lt; len(joint_names)}">
+      <xacro:openarm_v20_control_joint joint_name="${joint_names[index]}" />
+      <xacro:openarm_v20_control_joints joint_names="${joint_names}" index="${index + 1}" />
+    </xacro:if>
+  </xacro:macro>
+  <xacro:macro name="openarm_v20_arm_ros2_control"
+    params="system_name joint_names hardware_prefix can_interface control_gains ee_type:='' arm_type:=v20 use_fake_hardware:=true fake_sensor_commands:=false can_fd:=true">
+    <ros2_control name="${system_name}" type="system">
         <hardware>
           <param name="arm_type">${arm_type}</param>
-          <param name="prefix">${arm_prefix}</param>
           <xacro:if value="${use_fake_hardware}">
             <plugin>mock_components/GenericSystem</plugin>
@@ -34,9 +39,8 @@
             <param name="state_following_offset">0.0</param>
           </xacro:if>
-          <xacro:if value="${use_fake_hardware == 0}">
+          <xacro:unless value="${use_fake_hardware}">
             <plugin>openarm_hardware/OpenArmHW</plugin>
             <param name="can_interface">${can_interface}</param>
-            <param name="arm_prefix">${arm_prefix}</param>
-            <param name="hand">${hand}</param>
+            <param name="arm_prefix">${hardware_prefix}</param>
             <param name="can_fd">${can_fd}</param>
             <param name="ee_type">${ee_type}</param>
@@ -55,37 +59,7 @@
             <param name="kd6">${control_gains['joint6']['kd']}</param>
             <param name="kd7">${control_gains['joint7']['kd']}</param>
-          </xacro:if>
+          </xacro:unless>
         </hardware>
-      <xacro:macro name="configure_joint" params="joint_name initial_position">
-        <joint name="${joint_name}">
-          <!--
-            deactivated for gazebo velocity and position interface due to a bug
-            https://github.com/ros-controls/gz_ros2_control/issues/343
-            Command Interfaces -->
-            <command_interface name="position"/>
-            <command_interface name="velocity"/>
-            <command_interface name="effort"/>
-          <!-- State Interfaces -->
-          <state_interface name="position">
-            <param name="initial_value">${initial_position}</param>
-          </state_interface>
-          <state_interface name="velocity">
-            <param name="initial_value">0.0</param>
-          </state_interface>
-          <state_interface name="effort">
-            <param name="initial_value">0.0</param>
-          </state_interface>
-        </joint>
-      </xacro:macro>
-      <xacro:configure_joint joint_name="openarm_${arm_prefix}joint1" initial_position="0.0"/>
-      <xacro:configure_joint joint_name="openarm_${arm_prefix}joint2" initial_position="0.0"/>
-      <xacro:configure_joint joint_name="openarm_${arm_prefix}joint3" initial_position="0.0"/>
-      <xacro:configure_joint joint_name="openarm_${arm_prefix}joint4" initial_position="0.0"/>
-      <xacro:configure_joint joint_name="openarm_${arm_prefix}joint5" initial_position="0.0"/>
-      <xacro:configure_joint joint_name="openarm_${arm_prefix}joint6" initial_position="0.0"/>
-      <xacro:configure_joint joint_name="openarm_${arm_prefix}joint7" initial_position="0.0"/>
-      <xacro:if value="${hand}">
-        <xacro:configure_joint joint_name="openarm_${arm_prefix}finger_joint1" initial_position="0.0" />
-      </xacro:if>
+      <xacro:openarm_v20_control_joints joint_names="${joint_names}" />
     </ros2_control>
   </xacro:macro>
