Commit message: Separate shared assembly from V2 arm and gripper definitions

File: assets/end_effector/pinch_gripper/urdf/pinch_gripper_macro.xacro (robot description, xacro)
@@ -13,7 +13,8 @@
 -->
 <robot xmlns:xacro="http://www.ros.org/wiki/xacro">
-  <xacro:include filename="$(find openarm_description)/assets/robot/openarm_v2.0/urdf/utils/openarm_v20_utils.xacro" />
-  <!-- Current EE implementation targets the two-finger gripper topology. -->
-  <xacro:macro name="openarm_v20_ee"
+  <xacro:include filename="$(find openarm_description)/assets/common/links.xacro" />
+  <xacro:include filename="$(find openarm_description)/assets/common/reference_frames.xacro" />
+  <xacro:include filename="$(find openarm_description)/assets/common/validation.xacro" />
+  <xacro:macro name="openarm_pinch_gripper"
     params="prefix connected_to mount_origin:=none topology joint_origins joint_axes joint_limits joint_mimics inertials visuals collisions reflect_x:=1 reflect_y:=1 reflect_z:=1 component_reflects:=false reflect_include_links:=^ reflect_include_joints:=^ reflect_include_reference_points:=^ limit_override_joints:=^ ee_reference_points:=^ emit_grasp_frame:=false grasp_reference_point:=grasp_frame skip_mount_joint:=false base_frame_shift:=none">
     <xacro:property name="base_link_name" value="${topology['links'][0]}" />
@@ -46,8 +47,8 @@
           <xacro:property name="base_visual_cfg" value="${visuals[base_link_name]}" lazy_eval="false" />
           <xacro:if value="${use_base_frame_shift}">
-            <xacro:openarm_v20_emit_composed_origin first="${resolved_base_frame_shift}" second="${base_visual_cfg.origin}" reflect_x="${reflect_x if base_link_reflects else 1}" reflect_y="${reflect_y if base_link_reflects else 1}" reflect_z="${reflect_z if base_link_reflects else 1}" />
+            <xacro:openarm_emit_composed_origin first="${resolved_base_frame_shift}" second="${base_visual_cfg.origin}" reflect_x="${reflect_x if base_link_reflects else 1}" reflect_y="${reflect_y if base_link_reflects else 1}" reflect_z="${reflect_z if base_link_reflects else 1}" />
           </xacro:if>
           <xacro:unless value="${use_base_frame_shift}">
-            <xacro:openarm_v20_emit_origin origin="${base_visual_cfg.origin}" reflect_x="${reflect_x if base_link_reflects else 1}" reflect_y="${reflect_y if base_link_reflects else 1}" reflect_z="${reflect_z if base_link_reflects else 1}" />
+            <xacro:openarm_emit_origin origin="${base_visual_cfg.origin}" reflect_x="${reflect_x if base_link_reflects else 1}" reflect_y="${reflect_y if base_link_reflects else 1}" reflect_z="${reflect_z if base_link_reflects else 1}" />
           </xacro:unless>
           <!-- Preserve the mesh's embedded materials. -->
@@ -63,8 +64,8 @@
           <xacro:property name="base_collision_cfg" value="${collisions[base_link_name]}" lazy_eval="false" />
           <xacro:if value="${use_base_frame_shift}">
-            <xacro:openarm_v20_emit_composed_origin first="${resolved_base_frame_shift}" second="${base_collision_cfg.origin}" reflect_x="${reflect_x if base_link_reflects else 1}" reflect_y="${reflect_y if base_link_reflects else 1}" reflect_z="${reflect_z if base_link_reflects else 1}" />
+            <xacro:openarm_emit_composed_origin first="${resolved_base_frame_shift}" second="${base_collision_cfg.origin}" reflect_x="${reflect_x if base_link_reflects else 1}" reflect_y="${reflect_y if base_link_reflects else 1}" reflect_z="${reflect_z if base_link_reflects else 1}" />
           </xacro:if>
           <xacro:unless value="${use_base_frame_shift}">
-            <xacro:openarm_v20_emit_origin origin="${base_collision_cfg.origin}" reflect_x="${reflect_x if base_link_reflects else 1}" reflect_y="${reflect_y if base_link_reflects else 1}" reflect_z="${reflect_z if base_link_reflects else 1}" />
+            <xacro:openarm_emit_origin origin="${base_collision_cfg.origin}" reflect_x="${reflect_x if base_link_reflects else 1}" reflect_y="${reflect_y if base_link_reflects else 1}" reflect_z="${reflect_z if base_link_reflects else 1}" />
           </xacro:unless>
           <geometry>
@@ -80,8 +81,8 @@
         <inertial>
           <xacro:if value="${use_base_frame_shift}">
-            <xacro:openarm_v20_emit_composed_origin first="${resolved_base_frame_shift}" second="${base_inertial_cfg.origin}" reflect_x="${reflect_x if base_link_reflects else 1}" reflect_y="${reflect_y if base_link_reflects else 1}" reflect_z="${reflect_z if base_link_reflects else 1}" />
+            <xacro:openarm_emit_composed_origin first="${resolved_base_frame_shift}" second="${base_inertial_cfg.origin}" reflect_x="${reflect_x if base_link_reflects else 1}" reflect_y="${reflect_y if base_link_reflects else 1}" reflect_z="${reflect_z if base_link_reflects else 1}" />
           </xacro:if>
           <xacro:unless value="${use_base_frame_shift}">
-            <xacro:openarm_v20_emit_origin origin="${base_inertial_cfg.origin}" reflect_x="${reflect_x if base_link_reflects else 1}" reflect_y="${reflect_y if base_link_reflects else 1}" reflect_z="${reflect_z if base_link_reflects else 1}" />
+            <xacro:openarm_emit_origin origin="${base_inertial_cfg.origin}" reflect_x="${reflect_x if base_link_reflects else 1}" reflect_y="${reflect_y if base_link_reflects else 1}" reflect_z="${reflect_z if base_link_reflects else 1}" />
           </xacro:unless>
           <mass value="${base_inertial_cfg.mass}" />
@@ -96,5 +97,5 @@
       </xacro:if>
     </link>
-    <xacro:openarm_v20_emit_link
+    <xacro:openarm_emit_link
       link_name="${prefix}ee_link1"
       source_name="${finger1_source}"
@@ -105,5 +106,5 @@
       reflect_y="${reflect_y if finger1_link_reflects else 1}"
       reflect_z="${reflect_z if finger1_link_reflects else 1}" />
-    <xacro:openarm_v20_emit_link
+    <xacro:openarm_emit_link
       link_name="${prefix}ee_link2"
       source_name="${finger2_source}"
@@ -116,5 +117,5 @@
     <xacro:unless value="${skip_mount_joint}">
       <joint name="${prefix}ee_mount_joint" type="fixed">
-        <xacro:openarm_v20_emit_origin origin="${resolved_mount_origin}" />
+        <xacro:openarm_emit_origin origin="${resolved_mount_origin}" />
         <parent link="${connected_to}" />
         <child link="${base_link_full_name}" />
@@ -162,13 +163,13 @@
     <joint name="${prefix}finger_joint1" type="revolute">
       <xacro:if value="${use_base_frame_shift}">
-        <xacro:openarm_v20_emit_composed_origin first="${resolved_base_frame_shift}" second="${finger1_joint_origin_cfg}" reflect_x="${reflect_x if finger1_joint_reflects else 1}" reflect_y="${reflect_y if finger1_joint_reflects else 1}" reflect_z="${reflect_z if finger1_joint_reflects else 1}" />
+        <xacro:openarm_emit_composed_origin first="${resolved_base_frame_shift}" second="${finger1_joint_origin_cfg}" reflect_x="${reflect_x if finger1_joint_reflects else 1}" reflect_y="${reflect_y if finger1_joint_reflects else 1}" reflect_z="${reflect_z if finger1_joint_reflects else 1}" />
       </xacro:if>
       <xacro:unless value="${use_base_frame_shift}">
-        <xacro:openarm_v20_emit_origin origin="${finger1_joint_origin_cfg}" reflect_x="${reflect_x if finger1_joint_reflects else 1}" reflect_y="${reflect_y if finger1_joint_reflects else 1}" reflect_z="${reflect_z if finger1_joint_reflects else 1}" />
+        <xacro:openarm_emit_origin origin="${finger1_joint_origin_cfg}" reflect_x="${reflect_x if finger1_joint_reflects else 1}" reflect_y="${reflect_y if finger1_joint_reflects else 1}" reflect_z="${reflect_z if finger1_joint_reflects else 1}" />
       </xacro:unless>
       <parent link="${base_link_full_name}" />
       <child link="${prefix}ee_link1" />
       <axis xyz="${finger1_joint_axis_reflect_sign * finger1_joint_axis_cfg.x} ${finger1_joint_axis_reflect_sign * finger1_joint_axis_cfg.y} ${finger1_joint_axis_reflect_sign * finger1_joint_axis_cfg.z}" />
-      <xacro:openarm_v20_emit_limit limit="${finger1_joint_limit_effective}" />
+      <xacro:openarm_emit_limit limit="${finger1_joint_limit_effective}" />
       <xacro:if value="${finger1_mimic_override != 'none'}">
         <mimic
@@ -180,13 +181,13 @@
     <joint name="${prefix}finger_joint2" type="revolute">
       <xacro:if value="${use_base_frame_shift}">
-        <xacro:openarm_v20_emit_composed_origin first="${resolved_base_frame_shift}" second="${finger2_joint_origin_cfg}" reflect_x="${reflect_x if finger2_joint_reflects else 1}" reflect_y="${reflect_y if finger2_joint_reflects else 1}" reflect_z="${reflect_z if finger2_joint_reflects else 1}" />
+        <xacro:openarm_emit_composed_origin first="${resolved_base_frame_shift}" second="${finger2_joint_origin_cfg}" reflect_x="${reflect_x if finger2_joint_reflects else 1}" reflect_y="${reflect_y if finger2_joint_reflects else 1}" reflect_z="${reflect_z if finger2_joint_reflects else 1}" />
       </xacro:if>
       <xacro:unless value="${use_base_frame_shift}">
-        <xacro:openarm_v20_emit_origin origin="${finger2_joint_origin_cfg}" reflect_x="${reflect_x if finger2_joint_reflects else 1}" reflect_y="${reflect_y if finger2_joint_reflects else 1}" reflect_z="${reflect_z if finger2_joint_reflects else 1}" />
+        <xacro:openarm_emit_origin origin="${finger2_joint_origin_cfg}" reflect_x="${reflect_x if finger2_joint_reflects else 1}" reflect_y="${reflect_y if finger2_joint_reflects else 1}" reflect_z="${reflect_z if finger2_joint_reflects else 1}" />
       </xacro:unless>
       <parent link="${base_link_full_name}" />
       <child link="${prefix}ee_link2" />
       <axis xyz="${finger2_joint_axis_reflect_sign * finger2_joint_axis_cfg.x} ${finger2_joint_axis_reflect_sign * finger2_joint_axis_cfg.y} ${finger2_joint_axis_reflect_sign * finger2_joint_axis_cfg.z}" />
-      <xacro:openarm_v20_emit_limit limit="${finger2_joint_limit_effective}" />
+      <xacro:openarm_emit_limit limit="${finger2_joint_limit_effective}" />
       <xacro:if value="${finger2_mimic_override != 'none'}">
         <mimic
@@ -196,5 +197,5 @@
       </xacro:if>
     </joint>
-    <xacro:openarm_v20_emit_reference_frames
+    <xacro:openarm_emit_reference_frames
       reference_points="${ee_reference_points}"
       force_emit_reference="${grasp_reference_point if emit_grasp_frame else ''}"

File: assets/end_effector/pinch_gripper/urdf/pinch_gripper_standalone.urdf.xacro (robot description, xacro)
@@ -13,11 +13,5 @@
 -->
 <robot xmlns:xacro="http://www.ros.org/wiki/xacro" name="pinch_gripper">
-  <xacro:include filename="$(find openarm_description)/assets/robot/openarm_v2.0/urdf/utils/openarm_v20_utils.xacro" />
-  <xacro:include filename="$(find openarm_description)/assets/robot/openarm_v2.0/urdf/utils/openarm_v20_ee.xacro" />
-  <xacro:macro name="openarm_v20_require" params="condition message">
-    <xacro:unless value="${condition}">
-      <xacro:property name="openarm_v20_requirement_failed" value="${xacro.fatal(message)}" lazy_eval="false" />
-    </xacro:unless>
-  </xacro:macro>
+  <xacro:include filename="$(find openarm_description)/assets/end_effector/pinch_gripper/urdf/pinch_gripper_macro.xacro" />
   <xacro:arg name="ee_config_dir" default="$(find openarm_description)/assets/end_effector/pinch_gripper/config" />
   <xacro:arg name="ee_inertials_name" default="nominal" />
@@ -29,8 +23,8 @@
   <xacro:property name="reflect_y_value" value="${float('$(arg reflect_y)')}" lazy_eval="false" />
   <xacro:property name="reflect_z_value" value="${float('$(arg reflect_z)')}" lazy_eval="false" />
-  <xacro:openarm_v20_require
+  <xacro:openarm_require
     condition="${reflect_x_value in [-1.0, 1.0] and reflect_y_value in [-1.0, 1.0] and reflect_z_value in [-1.0, 1.0]}"
     message="${'Invalid standalone gripper reflection: each reflect axis must be either 1 or -1.'}" />
-  <xacro:openarm_v20_require
+  <xacro:openarm_require
     condition="${(1 if reflect_x_value == -1.0 else 0) + (1 if reflect_y_value == -1.0 else 0) + (1 if reflect_z_value == -1.0 else 0) &lt;= 1}"
     message="${'Invalid standalone gripper reflection: combined x/y/z reflections are not currently supported.'}" />
@@ -38,5 +32,5 @@
   <xacro:property name="ee_topology" value="${xacro.load_yaml('$(arg ee_config_dir)/struct/topology.yaml')}" lazy_eval="false" />
   <xacro:property name="ee_reference_points" value="${xacro.load_yaml('$(arg ee_config_dir)/struct/reference_points.yaml')}" lazy_eval="false" />
-  <xacro:openarm_v20_ee
+  <xacro:openarm_pinch_gripper
     prefix=""
     connected_to="world"

File: assets/robot/openarm_v2.0/urdf/arm/openarm_arm.xacro (robot description, xacro)
@@ -13,6 +13,5 @@
 -->
 <robot xmlns:xacro="http://www.ros.org/wiki/xacro">
-  <xacro:include filename="$(find openarm_description)/assets/robot/openarm_v2.0/urdf/utils/openarm_v20_utils.xacro" />
-  <!-- Recursively emit the arm chain after the base link has been mounted. -->
+  <xacro:include filename="$(find openarm_description)/assets/common/links.xacro" />
   <xacro:macro name="openarm_v20_emit_arm_chain"
     params="index links prefix joint_origins joint_axes joint_limits inertials visuals collisions reflect_x:=1 reflect_y:=1 reflect_z:=1 component_reflects:=false reflect_include_links:=^ reflect_include_joints:=^ limit_override_joints:=^ tip_collapse_source_link:=none tip_collapse_child_link:=none base_frame_shift:=none">
@@ -30,5 +29,5 @@
         lazy_eval="false" />
       <xacro:unless value="${collapse_tip_child}">
-        <xacro:openarm_v20_emit_link
+        <xacro:openarm_emit_link
           link_name="${prefix}${child_name}"
           source_name="${child_name}"
@@ -40,5 +39,5 @@
           reflect_z="${reflect_z if child_link_reflects else 1}" />
       </xacro:unless>
-      <xacro:openarm_v20_emit_joint
+      <xacro:openarm_emit_joint
         joint_name="${prefix}${joint_name}"
         joint_type="revolute"
@@ -77,5 +76,4 @@
     </xacro:if>
   </xacro:macro>
-  <!-- Emit one arm component: base link, optional mount joint, then the internal joint chain. -->
   <xacro:macro name="openarm_v20_arm"
     params="prefix connected_to mount_origin topology joint_origins joint_axes joint_limits inertials visuals collisions reflect_x:=1 reflect_y:=1 reflect_z:=1 component_reflects:=false reflect_include_links:=^ reflect_include_joints:=^ limit_override_joints:=^ tip_collapse_source_link:=none tip_collapse_child_link:=none skip_mount_joint:=false base_frame_shift:=none">
@@ -84,5 +82,5 @@
     <xacro:property name="resolved_base_frame_shift" value="${base_frame_shift if base_frame_shift != 'none' else 'none'}" lazy_eval="false" />
     <xacro:property name="base_link_reflects" value="${component_reflects and base_link_name in reflect_include_links}" lazy_eval="false" />
-    <xacro:openarm_v20_emit_link
+    <xacro:openarm_emit_link
       link_name="${prefix}${base_link_name}"
       source_name="${base_link_name}"
@@ -96,5 +94,5 @@
     <xacro:unless value="${skip_mount_joint}">
       <joint name="${prefix}${base_link_name}_mount_joint" type="fixed">
-        <xacro:openarm_v20_emit_origin origin="${mount_origin}" reflect_x="1" reflect_y="1" reflect_z="1" reflect_position="false" />
+        <xacro:openarm_emit_origin origin="${mount_origin}" reflect_x="1" reflect_y="1" reflect_z="1" reflect_position="false" />
         <parent link="${connected_to}" />
         <child link="${prefix}${base_link_name}" />

File: assets/robot/openarm_v2.0/urdf/openarm_v20.urdf.xacro (robot description, xacro)
@@ -13,5 +13,5 @@
 -->
 <robot xmlns:xacro="http://www.ros.org/wiki/xacro" name="openarm_v20">
-  <xacro:include filename="$(find openarm_description)/assets/robot/openarm_v2.0/urdf/utils/openarm_v20_robot.xacro" />
+  <xacro:include filename="$(find openarm_description)/assets/common/assembly.xacro" />
   <xacro:include filename="$(find openarm_description)/assets/robot/openarm_v2.0/urdf/ros2_control/openarm_robot.ros2_control.xacro" />
   <xacro:arg name="robot_preset" default="default_bimanual" />
@@ -27,5 +27,5 @@
   <xacro:property name="config_root" value="${robot_root + '/config'}" />
   <xacro:property name="robot_preset_cfg" value="${xacro.load_yaml(config_root + '/robot_presets/' + '$(arg robot_preset)' + '.yaml')}" />
-  <xacro:openarm_v20_robot
+  <xacro:openarm_assemble_robot
     config_root="${config_root}"
     robot_preset="${robot_preset_cfg}"

File: assets/robot/openarm_v2.0/urdf/ros2_control/openarm_robot.ros2_control.xacro (robot description, xacro)
@@ -22,7 +22,7 @@
       <xacro:if value="${component['enabled'] and component['type'] == 'robot' and component['config'] == 'arm'}">
         <xacro:property name="side" value="${component['control']['side']}" lazy_eval="false" />
-        <xacro:openarm_v20_require condition="${side in can_interfaces}" message="${'Unknown control side `%s` on `%s`.' % (side, name)}" />
+        <xacro:openarm_require condition="${side in can_interfaces}" message="${'Unknown control side `%s` on `%s`.' % (side, name)}" />
         <xacro:property name="controlled_arms" value="${[c for c in components if robot_preset[c]['enabled'] and robot_preset[c]['type'] == 'robot' and robot_preset[c]['config'] == 'arm']}" lazy_eval="false" />
-        <xacro:openarm_v20_require condition="${len([c for c in controlled_arms if robot_preset[c]['control']['side'] == side]) == 1}" message="${'Multiple arms select the `%s` hardware interface.' % side}" />
+        <xacro:openarm_require condition="${len([c for c in controlled_arms if robot_preset[c]['control']['side'] == side]) == 1}" message="${'Multiple arms select the `%s` hardware interface.' % side}" />
         <xacro:property name="prefix" value="${component.get('prefix', '')}" lazy_eval="false" />
         <xacro:property name="arm_topology" value="${xacro.load_yaml(config_root + '/arm/struct/topology.yaml')}" lazy_eval="false" />
@@ -30,5 +30,5 @@
         <xacro:property name="joint_names" value="${[prefix + joint for joint in arm_topology['joints'] if arm_topology['joints'][joint]['type'] != 'fixed']}" lazy_eval="false" />
         <xacro:property name="grippers" value="${[c for c in components if robot_preset[c]['enabled'] and robot_preset[c]['type'] == 'end_effector' and robot_preset[c].get('connection', dict()).get('attach_to') == name]}" lazy_eval="false" />
-        <xacro:openarm_v20_require condition="${len(grippers) &lt;= 1}" message="${'Arm `%s` supports one controlled gripper.' % name}" />
+        <xacro:openarm_require condition="${len(grippers) &lt;= 1}" message="${'Arm `%s` supports one controlled gripper.' % name}" />
         <xacro:property name="ee_type" value="${''}" lazy_eval="false" />
         <xacro:if value="${len(grippers) == 1}">
