Commit message: Configure empty arm-tip collapse in topology

File: assets/common/assembly.xacro (robot description, xacro)
@@ -15,5 +15,5 @@
   <xacro:include filename="$(find openarm_description)/assets/common/components.xacro" />
   <xacro:macro name="openarm_resolve_component_runtime"
-    params="component_name components robot_preset config_root root_frame component_cfg component_desc parent_desc:=none collapse_internal_empty_links:=false emit_grasp_frame:=false out_name">
+    params="component_name components robot_preset config_root root_frame component_cfg component_desc parent_desc:=none emit_grasp_frame:=false out_name">
     <xacro:property name="none_value" value="${'none'}" lazy_eval="false" />
     <xacro:property name="zero_origin" value="${dict(x=0.0, y=0.0, z=0.0, roll=0.0, pitch=0.0, yaw=0.0)}" lazy_eval="false" />
@@ -89,7 +89,7 @@
     <xacro:property
       name="parent_terminal_link_empty"
-      value="${has_parent_desc and parent_desc['supports_tip_collapse'] and parent_desc['topology']['links'][-1] not in parent_desc['inertials'] and parent_desc['topology']['links'][-1] not in parent_desc['visuals'] and parent_desc['topology']['links'][-1] not in parent_desc['collisions']}"
-      lazy_eval="false" />
-    <xacro:if value="${has_parent_reference_key and not has_parent_override and collapse_internal_empty_links and parent_terminal_link_empty and parent_ref_canonical_link == parent_desc['topology']['links'][-1]}">
+      value="${has_parent_desc and parent_desc['collapse_empty_end'] and parent_desc['topology']['links'][-1] not in parent_desc['inertials'] and parent_desc['topology']['links'][-1] not in parent_desc['visuals'] and parent_desc['topology']['links'][-1] not in parent_desc['collisions']}"
+      lazy_eval="false" />
+    <xacro:if value="${has_parent_reference_key and not has_parent_override and parent_terminal_link_empty and parent_ref_canonical_link == parent_desc['topology']['links'][-1]}">
       <xacro:property name="skip_mount_joint" value="${True}" lazy_eval="false" />
       <xacro:openarm_reflect_pose origin="${reference_mount_origin}" reflect_x="${reflect_x}" reflect_y="${reflect_y}" reflect_z="${reflect_z}" out_name="base_frame_shift" />
@@ -103,9 +103,9 @@
     <xacro:property
       name="component_terminal_link_empty"
-      value="${component_desc['supports_tip_collapse'] and component_terminal_link not in component_desc['inertials'] and component_terminal_link not in component_desc['visuals'] and component_terminal_link not in component_desc['collisions']}"
+      value="${component_desc['collapse_empty_end'] and component_terminal_link not in component_desc['inertials'] and component_terminal_link not in component_desc['visuals'] and component_terminal_link not in component_desc['collisions']}"
       lazy_eval="false" />
     <xacro:property
       name="collapse_candidate_names"
-      value="${[name for name in attached_children if collapse_internal_empty_links and component_terminal_link_empty and 'parent_reference_point' in robot_preset[name]['connection'] and robot_preset[name]['connection']['parent_reference_point'] != None and ('parent' not in robot_preset[name]['connection'] or robot_preset[name]['connection']['parent'] == None) and robot_preset[name]['connection']['parent_reference_point'] in component_desc['reference_points'] and component_desc['reference_points'][robot_preset[name]['connection']['parent_reference_point']]['parent'] == component_terminal_link]}"
+      value="${[name for name in attached_children if component_terminal_link_empty and 'parent_reference_point' in robot_preset[name]['connection'] and robot_preset[name]['connection']['parent_reference_point'] != None and ('parent' not in robot_preset[name]['connection'] or robot_preset[name]['connection']['parent'] == None) and robot_preset[name]['connection']['parent_reference_point'] in component_desc['reference_points'] and component_desc['reference_points'][robot_preset[name]['connection']['parent_reference_point']]['parent'] == component_terminal_link]}"
       lazy_eval="false" />
     <xacro:openarm_require
@@ -147,5 +147,5 @@
   </xacro:macro>
   <xacro:macro name="openarm_emit_component_tree"
-    params="component_name components robot_preset config_root root_frame parent_desc:=none preloaded_desc:=none collapse_internal_empty_links:=false emit_grasp_frame:=false">
+    params="component_name components robot_preset config_root root_frame parent_desc:=none preloaded_desc:=none emit_grasp_frame:=false">
     <xacro:property name="none_value" value="${'none'}" lazy_eval="false" />
     <xacro:property name="component_cfg" value="${robot_preset[component_name]}" lazy_eval="false" />
@@ -167,5 +167,4 @@
       component_desc="${component_desc}"
       parent_desc="${parent_desc}"
-      collapse_internal_empty_links="${collapse_internal_empty_links}"
       emit_grasp_frame="${emit_grasp_frame}"
       out_name="component_runtime" />
@@ -187,9 +186,8 @@
       preloaded_component_name="${component_runtime['collapse_child_name']}"
       preloaded_component_desc="${component_runtime['collapse_child_desc']}"
-      collapse_internal_empty_links="${collapse_internal_empty_links}"
       emit_grasp_frame="${emit_grasp_frame}" />
   </xacro:macro>
   <xacro:macro name="openarm_emit_attached_components"
-    params="index components parent_component_name robot_preset config_root root_frame parent_desc:=none preloaded_component_name:=none preloaded_component_desc:=none collapse_internal_empty_links:=false emit_grasp_frame:=false">
+    params="index components parent_component_name robot_preset config_root root_frame parent_desc:=none preloaded_component_name:=none preloaded_component_desc:=none emit_grasp_frame:=false">
     <xacro:if value="${index &lt; len(components)}">
       <xacro:property name="none_value" value="${'none'}" lazy_eval="false" />
@@ -212,5 +210,4 @@
           parent_desc="${none_value if is_root_component else parent_desc}"
           preloaded_desc="${component_desc_override}"
-          collapse_internal_empty_links="${collapse_internal_empty_links}"
           emit_grasp_frame="${emit_grasp_frame}" />
       </xacro:if>
@@ -225,10 +222,9 @@
         preloaded_component_name="${preloaded_component_name}"
         preloaded_component_desc="${preloaded_component_desc}"
-        collapse_internal_empty_links="${collapse_internal_empty_links}"
         emit_grasp_frame="${emit_grasp_frame}" />
     </xacro:if>
   </xacro:macro>
   <xacro:macro name="openarm_assemble_robot"
-    params="config_root robot_preset collapse_internal_empty_links:=false emit_grasp_frame:=false">
+    params="config_root robot_preset emit_grasp_frame:=false">
     <xacro:property name="robot_cfg" value="${robot_preset['robot']}" lazy_eval="false" />
     <xacro:property name="root_frame" value="${robot_cfg['root_frame']}" lazy_eval="false" />
@@ -245,5 +241,4 @@
       config_root="${config_root}"
       root_frame="${root_frame}"
-      collapse_internal_empty_links="${collapse_internal_empty_links}"
       emit_grasp_frame="${emit_grasp_frame}" />
   </xacro:macro>

File: assets/common/components.xacro (robot description, xacro)
@@ -50,5 +50,5 @@
                      link_name_map=empty_dict,
                      default_mount_parent=sensor_root_link,
-                     supports_tip_collapse=False)}"
+                     collapse_empty_end=False)}"
         scope="parent"
         lazy_eval="false" />
@@ -89,5 +89,5 @@
       <xacro:property name="component_root_link_actual" value="${component_cfg['link_name'] if component_type == 'body' else (component_link_prefix + component_topology['links'][0])}" lazy_eval="false" />
       <xacro:property name="component_default_mount_parent" value="${component_cfg['link_name'] if component_type == 'body' else (component_link_prefix + component_topology['links'][-1])}" lazy_eval="false" />
-      <xacro:property name="component_supports_tip_collapse" value="${component_type == 'arm' and len([j for j in component_topology['joints'] if component_topology['joints'][j]['parent'] == component_topology['links'][-1]]) == 0}" lazy_eval="false" />
+      <xacro:property name="component_collapse_empty_end" value="${component_type == 'arm' and component_topology.get('collapse_empty_end', False) and len([j for j in component_topology['joints'] if component_topology['joints'][j]['parent'] == component_topology['links'][-1]]) == 0}" lazy_eval="false" />
       <xacro:property
         name="${out_name}"
@@ -112,5 +112,5 @@
                      link_name_map=component_link_name_map,
                      default_mount_parent=component_default_mount_parent,
-                     supports_tip_collapse=component_supports_tip_collapse)}"
+                     collapse_empty_end=component_collapse_empty_end)}"
         scope="parent"
         lazy_eval="false" />

File: assets/robot/openarm_v2.0/urdf/openarm_v20.urdf.xacro (robot description, xacro)
@@ -16,5 +16,4 @@
   <xacro:include filename="$(find openarm_description)/assets/robot/openarm_v2.0/urdf/ros2_control/openarm_robot.ros2_control.xacro" />
   <xacro:arg name="robot_preset" default="default_bimanual" />
-  <xacro:arg name="collapse_internal_empty_links" default="true" />
   <xacro:arg name="emit_grasp_frame" default="false" />
   <xacro:arg name="ros2_control" default="true" />
@@ -30,5 +29,4 @@
     config_root="${config_root}"
     robot_preset="${robot_preset_cfg}"
-    collapse_internal_empty_links="$(arg collapse_internal_empty_links)"
     emit_grasp_frame="$(arg emit_grasp_frame)" />
   <xacro:if value="$(arg ros2_control)">
