Commit message: Generate V2 joints from topology and reuse shared link emission

File: assets/common/components.xacro (robot description, xacro)
@@ -72,4 +72,5 @@
       <xacro:property name="component_link_prefix" value="${component_prefix + ('ee_' if component_type == 'end_effector' else '')}" lazy_eval="false" />
       <xacro:property name="component_topology" value="${xacro.load_yaml(component_cfg_root + '/struct/topology.yaml')}" lazy_eval="false" />
+      <xacro:openarm_validate_topology topology="${component_topology}" component="${component_name}" />
       <xacro:property name="component_reference_points" value="${xacro.load_yaml(component_cfg_root + '/struct/reference_points.yaml')}" lazy_eval="false" />
       <xacro:if value="${component_type == 'accessory'}">
@@ -88,5 +89,5 @@
       <xacro:property name="component_root_link_actual" value="${component_cfg['link_name'] if component_type == 'body' else (component_link_prefix + component_topology['links'][0])}" lazy_eval="false" />
       <xacro:property name="component_default_mount_parent" value="${component_cfg['link_name'] if component_type == 'body' else (component_link_prefix + component_topology['links'][-1])}" lazy_eval="false" />
-      <xacro:property name="component_supports_tip_collapse" value="${component_type == 'arm'}" lazy_eval="false" />
+      <xacro:property name="component_supports_tip_collapse" value="${component_type == 'arm' and len([j for j in component_topology['joints'] if component_topology['joints'][j]['parent'] == component_topology['links'][-1]]) == 0}" lazy_eval="false" />
       <xacro:property
         name="${out_name}"

File: assets/common/validation.xacro (robot description, xacro)
@@ -124,3 +124,25 @@
       robot_preset="${robot_preset}" />
   </xacro:macro>
+  <xacro:macro name="openarm_validate_link_ancestry" params="name topology component depth:=0">
+    <xacro:if value="${name != topology['links'][0]}">
+      <xacro:openarm_require condition="${depth &lt; len(topology['links'])}" message="${'Component `%s` has a cycle at link `%s`.' % (component, name)}" />
+      <xacro:property name="incoming" value="${[j for j in topology['joints'] if topology['joints'][j]['child'] == name]}" lazy_eval="false" />
+      <xacro:openarm_require condition="${len(incoming) == 1}" message="${'Link `%s` in `%s` must have one parent joint.' % (name, component)}" />
+      <xacro:openarm_validate_link_ancestry name="${topology['joints'][incoming[0]]['parent']}" topology="${topology}" component="${component}" depth="${depth + 1}" />
+    </xacro:if>
+  </xacro:macro>
+  <xacro:macro name="openarm_validate_topology" params="topology component index:=0">
+    <xacro:property name="links" value="${topology['links']}" lazy_eval="false" />
+    <xacro:property name="joints" value="${topology['joints']}" lazy_eval="false" />
+    <xacro:if value="${index == 0}">
+      <xacro:openarm_require condition="${len(links) > 0 and len([link for link in links if links.count(link) != 1]) == 0}" message="${'Component `%s` must have nonempty, unique links.' % component}" />
+      <xacro:openarm_require condition="${len([j for j in joints if joints[j]['parent'] not in links or joints[j]['child'] not in links]) == 0}" message="${'Component `%s` has a joint referencing an unknown link.' % component}" />
+      <xacro:openarm_require condition="${len([j for j in joints if joints[j]['child'] == links[0]]) == 0}" message="${'Root link of `%s` cannot have an internal parent joint.' % component}" />
+      <xacro:openarm_require condition="${len([j for j in joints if joints[j]['type'] not in ['fixed', 'revolute', 'continuous', 'prismatic']]) == 0}" message="${'Component `%s` has an unsupported joint type.' % component}" />
+    </xacro:if>
+    <xacro:if value="${index &lt; len(links)}">
+      <xacro:openarm_validate_link_ancestry name="${links[index]}" topology="${topology}" component="${component}" />
+      <xacro:openarm_validate_topology topology="${topology}" component="${component}" index="${index + 1}" />
+    </xacro:if>
+  </xacro:macro>
 </robot>

File: assets/end_effector/pinch_gripper/urdf/pinch_gripper_macro.xacro (robot description, xacro)
@@ -25,6 +25,6 @@
     <xacro:property name="base_link_reflects" value="${component_reflects and base_link_name in reflect_include_links}" lazy_eval="false" />
     <!-- Finger numbering stays semantic; handedness is handled by reflect_* and the joint config. -->
-    <xacro:property name="finger1_source" value="link1" />
-    <xacro:property name="finger2_source" value="link2" />
+    <xacro:property name="finger1_source" value="${topology['joints']['joint1']['child']}" />
+    <xacro:property name="finger2_source" value="${topology['joints']['joint2']['child']}" />
     <xacro:property name="finger1_joint_source" value="joint1" />
     <xacro:property name="finger2_joint_source" value="joint2" />
@@ -41,62 +41,13 @@
     <xacro:property name="finger1_mimic_override" value="${dict(joint=finger1_mimic_target_name, multiplier=joint_mimics[finger1_joint_source]['multiplier'], offset=joint_mimics[finger1_joint_source]['offset']) if finger1_has_mimic else 'none'}" />
     <xacro:property name="finger2_mimic_override" value="${dict(joint=finger2_mimic_target_name, multiplier=joint_mimics[finger2_joint_source]['multiplier'], offset=joint_mimics[finger2_joint_source]['offset']) if finger2_has_mimic else 'none'}" />
-    <!-- The base link is emitted inline because its naming and frame-shift behavior differ from the finger links. -->
-    <link name="${base_link_full_name}">
-      <xacro:if value="${base_link_name in visuals}">
-        <visual name="${base_link_full_name}_visual">
-          <xacro:property name="base_visual_cfg" value="${visuals[base_link_name]}" lazy_eval="false" />
-          <xacro:if value="${use_base_frame_shift}">
-            <xacro:openarm_emit_composed_origin first="${resolved_base_frame_shift}" second="${base_visual_cfg.origin}" reflect_x="${reflect_x if base_link_reflects else 1}" reflect_y="${reflect_y if base_link_reflects else 1}" reflect_z="${reflect_z if base_link_reflects else 1}" />
-          </xacro:if>
-          <xacro:unless value="${use_base_frame_shift}">
-            <xacro:openarm_emit_origin origin="${base_visual_cfg.origin}" reflect_x="${reflect_x if base_link_reflects else 1}" reflect_y="${reflect_y if base_link_reflects else 1}" reflect_z="${reflect_z if base_link_reflects else 1}" />
-          </xacro:unless>
-          <!-- Preserve the mesh's embedded materials. -->
-          <geometry>
-            <mesh
-              filename="${base_visual_cfg.geometry.mesh}"
-              scale="${(reflect_x if base_link_reflects else 1) * base_visual_cfg.geometry.scale.x} ${(reflect_y if base_link_reflects else 1) * base_visual_cfg.geometry.scale.y} ${(reflect_z if base_link_reflects else 1) * base_visual_cfg.geometry.scale.z}" />
-          </geometry>
-        </visual>
-      </xacro:if>
-      <xacro:if value="${base_link_name in collisions}">
-        <collision name="${base_link_full_name}_collision">
-          <xacro:property name="base_collision_cfg" value="${collisions[base_link_name]}" lazy_eval="false" />
-          <xacro:if value="${use_base_frame_shift}">
-            <xacro:openarm_emit_composed_origin first="${resolved_base_frame_shift}" second="${base_collision_cfg.origin}" reflect_x="${reflect_x if base_link_reflects else 1}" reflect_y="${reflect_y if base_link_reflects else 1}" reflect_z="${reflect_z if base_link_reflects else 1}" />
-          </xacro:if>
-          <xacro:unless value="${use_base_frame_shift}">
-            <xacro:openarm_emit_origin origin="${base_collision_cfg.origin}" reflect_x="${reflect_x if base_link_reflects else 1}" reflect_y="${reflect_y if base_link_reflects else 1}" reflect_z="${reflect_z if base_link_reflects else 1}" />
-          </xacro:unless>
-          <geometry>
-            <mesh
-              filename="${base_collision_cfg.geometry.mesh}"
-              scale="${(reflect_x if base_link_reflects else 1) * base_collision_cfg.geometry.scale.x} ${(reflect_y if base_link_reflects else 1) * base_collision_cfg.geometry.scale.y} ${(reflect_z if base_link_reflects else 1) * base_collision_cfg.geometry.scale.z}" />
-          </geometry>
-        </collision>
-      </xacro:if>
-      <xacro:if value="${base_link_name in inertials}">
-        <xacro:property name="base_inertial_cfg" value="${inertials[base_link_name]}" lazy_eval="false" />
-        <xacro:property name="base_inertia_terms" value="${base_inertial_cfg.inertia}" lazy_eval="false" />
-        <inertial>
-          <xacro:if value="${use_base_frame_shift}">
-            <xacro:openarm_emit_composed_origin first="${resolved_base_frame_shift}" second="${base_inertial_cfg.origin}" reflect_x="${reflect_x if base_link_reflects else 1}" reflect_y="${reflect_y if base_link_reflects else 1}" reflect_z="${reflect_z if base_link_reflects else 1}" />
-          </xacro:if>
-          <xacro:unless value="${use_base_frame_shift}">
-            <xacro:openarm_emit_origin origin="${base_inertial_cfg.origin}" reflect_x="${reflect_x if base_link_reflects else 1}" reflect_y="${reflect_y if base_link_reflects else 1}" reflect_z="${reflect_z if base_link_reflects else 1}" />
-          </xacro:unless>
-          <mass value="${base_inertial_cfg.mass}" />
-          <inertia
-            ixx="${base_inertia_terms.xx}"
-            ixy="${(reflect_x if base_link_reflects else 1) * (reflect_y if base_link_reflects else 1) * base_inertia_terms.xy}"
-            ixz="${(reflect_x if base_link_reflects else 1) * (reflect_z if base_link_reflects else 1) * base_inertia_terms.xz}"
-            iyy="${base_inertia_terms.yy}"
-            iyz="${(reflect_y if base_link_reflects else 1) * (reflect_z if base_link_reflects else 1) * base_inertia_terms.yz}"
-            izz="${base_inertia_terms.zz}" />
-        </inertial>
-      </xacro:if>
-    </link>
     <xacro:openarm_emit_link
-      link_name="${prefix}ee_link1"
+      link_name="${base_link_full_name}" source_name="${base_link_name}"
+      inertials="${inertials}" visuals="${visuals}" collisions="${collisions}"
+      reflect_x="${reflect_x if base_link_reflects else 1}"
+      reflect_y="${reflect_y if base_link_reflects else 1}"
+      reflect_z="${reflect_z if base_link_reflects else 1}"
+      frame_shift="${base_frame_shift}" />
+    <xacro:openarm_emit_link
+      link_name="${prefix}ee_${finger1_source}"
       source_name="${finger1_source}"
       inertials="${inertials}"
@@ -107,5 +58,5 @@
       reflect_z="${reflect_z if finger1_link_reflects else 1}" />
     <xacro:openarm_emit_link
-      link_name="${prefix}ee_link2"
+      link_name="${prefix}ee_${finger2_source}"
       source_name="${finger2_source}"
       inertials="${inertials}"
@@ -161,5 +112,5 @@
       value="${finger2_joint_limit_override if finger2_joint_limit_override != 'none' else (dict(lower=(-finger2_joint_limit_cfg['upper']), upper=(-finger2_joint_limit_cfg['lower']), effort=finger2_joint_limit_cfg['effort'], velocity=finger2_joint_limit_cfg['velocity']) if finger2_limit_should_mirror else finger2_joint_limit_cfg)}"
       lazy_eval="false" />
-    <joint name="${prefix}finger_joint1" type="revolute">
+    <joint name="${prefix}finger_joint1" type="${topology['joints'][finger1_joint_source]['type']}">
       <xacro:if value="${use_base_frame_shift}">
         <xacro:openarm_emit_composed_origin first="${resolved_base_frame_shift}" second="${finger1_joint_origin_cfg}" reflect_x="${reflect_x if finger1_joint_reflects else 1}" reflect_y="${reflect_y if finger1_joint_reflects else 1}" reflect_z="${reflect_z if finger1_joint_reflects else 1}" />
@@ -168,6 +119,7 @@
         <xacro:openarm_emit_origin origin="${finger1_joint_origin_cfg}" reflect_x="${reflect_x if finger1_joint_reflects else 1}" reflect_y="${reflect_y if finger1_joint_reflects else 1}" reflect_z="${reflect_z if finger1_joint_reflects else 1}" />
       </xacro:unless>
-      <parent link="${base_link_full_name}" />
-      <child link="${prefix}ee_link1" />
+      <parent link="${prefix}ee_${topology['joints'][finger1_joint_source]['parent']}" />
+      <child link="${prefix}ee_${finger1_source}" />
+      <xacro:if value="${topology['joints'][finger1_joint_source]['type'] != 'fixed'}">
       <axis xyz="${finger1_joint_axis_reflect_sign * finger1_joint_axis_cfg.x} ${finger1_joint_axis_reflect_sign * finger1_joint_axis_cfg.y} ${finger1_joint_axis_reflect_sign * finger1_joint_axis_cfg.z}" />
       <xacro:openarm_emit_limit limit="${finger1_joint_limit_effective}" />
@@ -178,6 +130,7 @@
           offset="${finger1_mimic_override['offset']}" />
       </xacro:if>
+          </xacro:if>
     </joint>
-    <joint name="${prefix}finger_joint2" type="revolute">
+    <joint name="${prefix}finger_joint2" type="${topology['joints'][finger2_joint_source]['type']}">
       <xacro:if value="${use_base_frame_shift}">
         <xacro:openarm_emit_composed_origin first="${resolved_base_frame_shift}" second="${finger2_joint_origin_cfg}" reflect_x="${reflect_x if finger2_joint_reflects else 1}" reflect_y="${reflect_y if finger2_joint_reflects else 1}" reflect_z="${reflect_z if finger2_joint_reflects else 1}" />
@@ -186,6 +139,7 @@
         <xacro:openarm_emit_origin origin="${finger2_joint_origin_cfg}" reflect_x="${reflect_x if finger2_joint_reflects else 1}" reflect_y="${reflect_y if finger2_joint_reflects else 1}" reflect_z="${reflect_z if finger2_joint_reflects else 1}" />
       </xacro:unless>
-      <parent link="${base_link_full_name}" />
-      <child link="${prefix}ee_link2" />
+      <parent link="${prefix}ee_${topology['joints'][finger2_joint_source]['parent']}" />
+      <child link="${prefix}ee_${finger2_source}" />
+      <xacro:if value="${topology['joints'][finger2_joint_source]['type'] != 'fixed'}">
       <axis xyz="${finger2_joint_axis_reflect_sign * finger2_joint_axis_cfg.x} ${finger2_joint_axis_reflect_sign * finger2_joint_axis_cfg.y} ${finger2_joint_axis_reflect_sign * finger2_joint_axis_cfg.z}" />
       <xacro:openarm_emit_limit limit="${finger2_joint_limit_effective}" />
@@ -196,4 +150,5 @@
           offset="${finger2_mimic_override['offset']}" />
       </xacro:if>
+          </xacro:if>
     </joint>
     <xacro:openarm_emit_reference_frames

File: assets/robot/openarm_v2.0/urdf/arm/openarm_arm.xacro (robot description, xacro)
@@ -15,9 +15,9 @@
   <xacro:include filename="$(find openarm_description)/assets/common/links.xacro" />
   <xacro:macro name="openarm_v20_emit_arm_chain"
-    params="index links prefix joint_origins joint_axes joint_limits inertials visuals collisions reflect_x:=1 reflect_y:=1 reflect_z:=1 component_reflects:=false reflect_include_links:=^ reflect_include_joints:=^ limit_override_joints:=^ tip_collapse_source_link:=none tip_collapse_child_link:=none base_frame_shift:=none">
-    <xacro:if value="${index &lt; len(links) - 1}">
-      <xacro:property name="joint_name" value="${'joint' + str(index + 1)}" />
-      <xacro:property name="parent_name" value="${links[index]}" />
-      <xacro:property name="child_name" value="${links[index + 1]}" />
+    params="index joint_names topology prefix joint_origins joint_axes joint_limits inertials visuals collisions reflect_x:=1 reflect_y:=1 reflect_z:=1 component_reflects:=false reflect_include_links:=^ reflect_include_joints:=^ limit_override_joints:=^ tip_collapse_source_link:=none tip_collapse_child_link:=none base_frame_shift:=none">
+    <xacro:if value="${index &lt; len(joint_names)}">
+      <xacro:property name="joint_name" value="${joint_names[index]}" />
+      <xacro:property name="parent_name" value="${topology['joints'][joint_name]['parent']}" />
+      <xacro:property name="child_name" value="${topology['joints'][joint_name]['child']}" />
       <xacro:property name="joint_limit_override" value="${limit_override_joints[joint_name] if joint_name in limit_override_joints else 'none'}" lazy_eval="false" />
       <xacro:property name="child_link_reflects" value="${component_reflects and child_name in reflect_include_links}" lazy_eval="false" />
@@ -26,5 +26,5 @@
       <xacro:property
         name="collapse_tip_child"
-        value="${tip_collapse_source_link != 'none' and child_name == tip_collapse_source_link and index == len(links) - 2}"
+        value="${tip_collapse_source_link != 'none' and child_name == tip_collapse_source_link}"
         lazy_eval="false" />
       <xacro:unless value="${collapse_tip_child}">
@@ -41,5 +41,5 @@
       <xacro:openarm_emit_joint
         joint_name="${prefix}${joint_name}"
-        joint_type="revolute"
+        joint_type="${topology['joints'][joint_name]['type']}"
         parent_link="${prefix}${parent_name}"
         child_link="${tip_collapse_child_link if collapse_tip_child else prefix + child_name}"
@@ -53,8 +53,9 @@
         limit_override="${joint_limit_override}"
         mirror_limit_sign="${joint_reflects}"
-        frame_shift="${base_frame_shift if index == 0 else 'none'}" />
+        frame_shift="${base_frame_shift if parent_name == topology['links'][0] else 'none'}" />
       <xacro:openarm_v20_emit_arm_chain
         index="${index + 1}"
-        links="${links}"
+        joint_names="${joint_names}"
+        topology="${topology}"
         prefix="${prefix}"
         joint_origins="${joint_origins}"
@@ -79,4 +80,5 @@
     params="prefix connected_to mount_origin topology joint_origins joint_axes joint_limits inertials visuals collisions reflect_x:=1 reflect_y:=1 reflect_z:=1 component_reflects:=false reflect_include_links:=^ reflect_include_joints:=^ limit_override_joints:=^ tip_collapse_source_link:=none tip_collapse_child_link:=none skip_mount_joint:=false base_frame_shift:=none">
     <xacro:property name="links" value="${topology['links']}" lazy_eval="false" />
+    <xacro:property name="joint_names" value="${list(topology['joints'].keys())}" lazy_eval="false" />
     <xacro:property name="base_link_name" value="${links[0]}" />
     <xacro:property name="resolved_base_frame_shift" value="${base_frame_shift if base_frame_shift != 'none' else 'none'}" lazy_eval="false" />
@@ -101,5 +103,6 @@
     <xacro:openarm_v20_emit_arm_chain
       index="0"
-      links="${links}"
+      joint_names="${joint_names}"
+        topology="${topology}"
       prefix="${prefix}"
       joint_origins="${joint_origins}"
