Commit message: Finalize shared model assembly, body assets and camera visuals
Move V1/V2 bodies into their own asset category and update the V2
open-cover mass properties. Complete the gripper camera visual and V1
material updates, fix oblique joint reflection and parent mount overrides,
and resolve body root aliases from topology.

Keep the batch URDF export helper local and outside the tracked changes.

File: assets/common/components.xacro (robot description, xacro)
@@ -66,7 +66,7 @@
           lazy_eval="false" />
       </xacro:if>
-      <xacro:if value="${source_type == 'accessory'}">
-        <xacro:property name="component_type" value="accessory" lazy_eval="false" />
-        <xacro:property name="component_cfg_root" value="${'$(find openarm_description)/assets/accessory/' + product + '/config'}" lazy_eval="false" />
+      <xacro:if value="${source_type in ['body', 'accessory']}">
+        <xacro:property name="component_type" value="${source_type}" lazy_eval="false" />
+        <xacro:property name="component_cfg_root" value="${'$(find openarm_description)/assets/' + source_type + '/' + product + '/config'}" lazy_eval="false" />
       </xacro:if>
       <xacro:property name="component_topology" value="${xacro.load_yaml(component_cfg_root + '/struct/topology.yaml')}" lazy_eval="false" />
@@ -75,8 +75,8 @@
       <xacro:openarm_validate_topology topology="${component_topology}" component="${component_name}" />
       <xacro:property name="component_reference_points" value="${xacro.load_yaml(component_cfg_root + '/struct/reference_points.yaml')}" lazy_eval="false" />
-      <xacro:if value="${component_type == 'accessory'}">
+      <xacro:if value="${component_type in ['body', 'accessory']}">
         <xacro:openarm_require
           condition="${len(component_topology['links']) == 1 and len(component_topology['joints']) == 0}"
-          message="${'Accessory `%s` must define one rigid link and no internal joints.' % component_name}" />
+          message="${'Component `%s` must define one rigid link and no internal joints.' % component_name}" />
       </xacro:if>
       <xacro:property name="component_joint_origins" value="${xacro.load_yaml(component_cfg_root + '/joint/joint_origins.yaml') if component_type not in ['body', 'accessory'] else empty_dict}" lazy_eval="false" />
@@ -87,5 +87,5 @@
       <xacro:property name="component_visuals" value="${xacro.load_yaml(component_cfg_root + '/link/visuals.yaml')}" lazy_eval="false" />
       <xacro:property name="component_collisions" value="${xacro.load_yaml(component_cfg_root + '/link/collisions.yaml')}" lazy_eval="false" />
-      <xacro:property name="component_link_name_map" value="${dict(body_link0=component_cfg['link_name']) if component_type == 'body' else empty_dict}" lazy_eval="false" />
+      <xacro:property name="component_link_name_map" value="${dict([(component_topology['links'][0], component_cfg['link_name'])]) if component_type == 'body' else empty_dict}" lazy_eval="false" />
       <xacro:property name="component_root_link_actual" value="${component_cfg['link_name'] if component_type == 'body' else (component_link_prefix + component_topology['links'][0])}" lazy_eval="false" />
       <xacro:property name="component_default_mount_parent" value="${component_cfg['link_name'] if component_type == 'body' else (component_link_prefix + component_topology['links'][-1])}" lazy_eval="false" />

File: assets/common/links.xacro (robot description, xacro)
@@ -93,8 +93,8 @@
         <xacro:property name="joint_axis_cfg" value="${axis_override if axis_override != 'none' else joint_axes[source_joint_name].axis}" lazy_eval="false" />
         <xacro:property
-          name="joint_axis_reflect_sign"
-          value="${-1 if ((reflect_x == -1 and joint_axis_cfg['x'] * joint_axis_cfg['x'] > 1e-18) or (reflect_y == -1 and joint_axis_cfg['y'] * joint_axis_cfg['y'] > 1e-18) or (reflect_z == -1 and joint_axis_cfg['z'] * joint_axis_cfg['z'] > 1e-18)) else 1}"
+          name="mirror_limit_for_axis"
+          value="${(reflect_x == -1 and joint_axis_cfg['x'] * joint_axis_cfg['x'] > 1e-18) or (reflect_y == -1 and joint_axis_cfg['y'] * joint_axis_cfg['y'] > 1e-18) or (reflect_z == -1 and joint_axis_cfg['z'] * joint_axis_cfg['z'] > 1e-18)}"
           lazy_eval="false" />
-        <axis xyz="${joint_axis_reflect_sign * joint_axis_cfg['x']} ${joint_axis_reflect_sign * joint_axis_cfg['y']} ${joint_axis_reflect_sign * joint_axis_cfg['z']}" />
+        <axis xyz="${reflect_x * joint_axis_cfg['x']} ${reflect_y * joint_axis_cfg['y']} ${reflect_z * joint_axis_cfg['z']}" />
       </xacro:if>
       <xacro:if value="${joint_type != 'fixed' and (limit_override != 'none' or source_joint_name in joint_limits)}">
@@ -102,5 +102,5 @@
         <xacro:property
           name="effective_mirror_limit_sign"
-          value="${mirror_limit_sign or joint_axis_reflect_sign == -1}"
+          value="${mirror_limit_sign or mirror_limit_for_axis}"
           lazy_eval="false" />
         <xacro:if value="${effective_mirror_limit_sign}">

File: assets/common/validation.xacro (robot description, xacro)
@@ -37,5 +37,5 @@
         message="${'Invalid robot preset: component `%s` attaches to disabled parent `%s`.' % (component_name, attach_to)}" />
       <xacro:openarm_require
-        condition="${robot_preset[attach_to]['type'] in ['robot', 'end_effector', 'sensor', 'accessory']}"
+        condition="${robot_preset[attach_to]['type'] in ['robot', 'body', 'end_effector', 'sensor', 'accessory']}"
         message="${'Invalid robot preset: component `%s` attaches to unsupported parent type `%s` on `%s`.' % (component_name, robot_preset[attach_to]['type'], attach_to)}" />
       <xacro:openarm_validate_component_lineage
@@ -61,5 +61,5 @@
       <xacro:property name="reflect_cfg" value="${component_cfg['reflect'] if 'reflect' in component_cfg else dict(x=1, y=1, z=1)}" lazy_eval="false" />
       <xacro:openarm_require
-        condition="${component_type in ['robot', 'end_effector', 'sensor', 'accessory']}"
+        condition="${component_type in ['robot', 'body', 'end_effector', 'sensor', 'accessory']}"
         message="${'Invalid robot preset: component `%s` has unsupported type `%s`.' % (component_name, component_type)}" />
       <xacro:openarm_require
@@ -74,6 +74,12 @@
           message="${'Invalid robot preset: robot component `%s` uses unsupported product `%s`.' % (component_name, component_cfg['product'])}" />
         <xacro:openarm_require
-          condition="${component_config in ['body', 'arm']}"
+          condition="${component_config == 'arm'}"
           message="${'Invalid robot preset: robot component `%s` has unsupported config `%s`.' % (component_name, component_config)}" />
+      </xacro:if>
+      <xacro:if value="${component_type == 'body'}">
+        <xacro:openarm_require condition="${component_cfg['product'] in ['v1.0', 'v2.0']}"
+          message="${'Unsupported body `%s`.' % component_cfg['product']}" />
+        <xacro:openarm_require condition="${component_config == None and 'link_name' in component_cfg}"
+          message="${'Body `%s` requires config: null and link_name.' % component_name}" />
       </xacro:if>
       <xacro:if value="${component_type == 'end_effector'}">

File: assets/robot/openarm_v1.0/urdf/example/v1.urdf (robot description, URDF)
Before this commit: robot openarm, 26 links, 25 joints
Links:
- link openarm_body_link0: geometry collision mesh filename=package://openarm_description/assets/body/v1.0/meshes/colli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 scale=0.001 0.001 0.001; visual mesh filename=package://openarm_description/assets/body/v1.0/meshes/visua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 scale=0.001 0.001 0.001

File: assets/robot/openarm_v1.0/urdf/openarm_v10.urdf.xacro (robot description, xacro)
@@ -43,5 +43,4 @@
   <xacro:property name="without_prefix" value="${'$(arg no_prefix)'.lower() in ['true', '1']}" />
   <xacro:property name="arm_count" value="${len([n for n in preset['robot']['components'] if preset[n]['enabled'] and preset[n]['type'] == 'robot' and preset[n]['config'] == 'arm'])}" />
-  <xacro:property name="body_mounts" value="${xacro.load_yaml(config_root + '/body/struct/reference_points.yaml')}" />
   <xacro:macro name="openarm_v1_entry_components" params="value index:=0 out_name">
     <xacro:property name="names" value="${value['robot']['components']}" />
@@ -50,5 +49,5 @@
       <xacro:property name="component" value="${value[name]}" lazy_eval="false" />
       <xacro:property name="connection" value="${component.get('connection', dict())}" lazy_eval="false" />
-      <xacro:if value="${without_prefix and component['type'] == 'robot' and component['config'] == 'body'}">
+      <xacro:if value="${without_prefix and component['type'] == 'body'}">
         <xacro:property name="component" value="${dict(component, link_name='body_link0')}" lazy_eval="false" />
       </xacro:if>
@@ -70,8 +69,24 @@
         <xacro:property name="rotation_arg" value="${'$(arg left_arm_base_rpy)' if side == 'left' else '$(arg right_arm_base_rpy)'}" />
         <xacro:if value="${position_arg != '' or rotation_arg != ''}">
-          <xacro:property name="base" value="${body_mounts[connection['parent_reference_point']]['origin'] if connection.get('parent_reference_point') else connection['origin']}" />
+          <xacro:property name="override_parent" value="${connection.get('parent')}" lazy_eval="false" />
+          <xacro:property name="offset" value="${connection.get('origin') or dict()}" lazy_eval="false" />
+          <xacro:property name="base" value="${dict(x=offset.get('x') or 0.0, y=offset.get('y') or 0.0, z=offset.get('z') or 0.0, roll=offset.get('roll') or 0.0, pitch=offset.get('pitch') or 0.0, yaw=offset.get('yaw') or 0.0)}" lazy_eval="false" />
+          <xacro:if value="${connection.get('parent_reference_point') not in [None, '']}">
+            <xacro:property name="mount_parent_cfg" value="${value[connection['attach_to']]}" lazy_eval="false" />
+            <xacro:openarm_load_component_descriptor component_name="${connection['attach_to']}" component_cfg="${mount_parent_cfg}" config_root="${config_root}" out_name="mount_parent_desc" />
+            <xacro:property name="mount_reference_name" value="${connection['parent_reference_point']}" lazy_eval="false" />
+            <xacro:property name="mount_reference" value="${mount_parent_desc['reference_points'][mount_reference_name]}" lazy_eval="false" />
+            <xacro:property name="reference_origin" value="${mount_reference['origin']}" lazy_eval="false" />
+            <xacro:property name="parent_reflection" value="${mount_parent_cfg.get('reflect', dict(x=1, y=1, z=1))}" lazy_eval="false" />
+            <xacro:if value="${mount_reference_name in parent_reflection.get('include', dict()).get('reference_points', list(mount_parent_desc['reference_points']))}">
+              <xacro:openarm_reflect_pose origin="${reference_origin}" reflect_x="${parent_reflection['x']}" reflect_y="${parent_reflection['y']}" reflect_z="${parent_reflection['z']}" out_name="reference_origin" />
+            </xacro:if>
+            <xacro:openarm_compose_pose first="${reference_origin}" second="${base}" out_name="base" />
+            <xacro:property name="reference_parent" value="${mount_parent_desc['link_name_map'].get(mount_reference['parent'], mount_parent_desc['link_prefix'] + mount_reference['parent'])}" lazy_eval="false" />
+            <xacro:property name="override_parent" value="${None if reference_parent == mount_parent_desc['default_mount_parent'] else reference_parent}" lazy_eval="false" />
+          </xacro:if>
           <xacro:property name="pos" value="${[float(v) for v in position_arg.split()] if position_arg else [base['x'], base['y'], base['z']]}" />
           <xacro:property name="rot" value="${[float(v) for v in rotation_arg.split()] if rotation_arg else [base['roll'], base['pitch'], base['yaw']]}" />
-          <xacro:property name="connection" value="${dict(connection, parent_reference_point=None, parent=None, origin=dict(x=pos[0], y=pos[1], z=pos[2], roll=rot[0], pitch=rot[1], yaw=rot[2]))}" lazy_eval="false" />
+          <xacro:property name="connection" value="${dict(connection, parent_reference_point=None, parent=override_parent, origin=dict(x=pos[0], y=pos[1], z=pos[2], roll=rot[0], pitch=rot[1], yaw=rot[2]))}" lazy_eval="false" />
         </xacro:if>
         <xacro:property name="prefix_arg" value="${'$(arg left_arm_prefix)' if side == 'left' else '$(arg right_arm_prefix)'}" />

File: assets/robot/openarm_v2.0/urdf/example/v2.urdf (robot description, URDF)
Before this commit: robot openarm_v20, 33 links, 32 joints
Links:
- link openarm_body_link0: mass 3.74 -> 3.734812201783; geometry collision mesh filename=package://openarm_description/assets/body/v2.0/meshes/colli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 scale=0.001 0.001 0.001; visual mesh filename=package://openarm_description/assets/body/v2.0/meshes/visua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 scale=1.0 1.0 1.0
