Commit message: Reuse shared mirroring while preserving V1 joint coordinates

File: assets/common/links.xacro (robot description, xacro)
@@ -78,13 +78,13 @@
     </link>
   </xacro:macro>
-  <xacro:macro name="openarm_emit_joint" params="joint_name joint_type parent_link child_link joint_origins joint_axes joint_limits reflect_x:=1 reflect_y:=1 reflect_z:=1 source_name:='' origin_override:=none axis_override:=none limit_override:=none mimic_override:=none mirror_limit_sign:=false frame_shift:=none">
+  <xacro:macro name="openarm_emit_joint" params="joint_name joint_type parent_link child_link joint_origins joint_axes joint_limits reflect_x:=1 reflect_y:=1 reflect_z:=1 source_name:='' origin_override:=none axis_override:=none limit_override:=none mimic_override:=none mirror_limit_sign:=false frame_shift:=none reflect_rotation:=${False}">
     <xacro:property name="source_joint_name" value="${source_name if source_name != '' else joint_name}" />
     <xacro:property name="joint_origin_cfg" value="${origin_override if origin_override != 'none' else joint_origins[source_joint_name].origin}" lazy_eval="false" />
     <joint name="${joint_name}" type="${joint_type}">
       <xacro:if value="${frame_shift != 'none'}">
-        <xacro:openarm_emit_composed_origin first="${frame_shift}" second="${joint_origin_cfg}" reflect_x="${reflect_x}" reflect_y="${reflect_y}" reflect_z="${reflect_z}" />
+        <xacro:openarm_emit_composed_origin first="${frame_shift}" second="${joint_origin_cfg}" reflect_x="${reflect_x}" reflect_y="${reflect_y}" reflect_z="${reflect_z}" reflect_rotation="${reflect_rotation}" />
       </xacro:if>
       <xacro:unless value="${frame_shift != 'none'}">
-        <xacro:openarm_emit_origin origin="${joint_origin_cfg}" reflect_x="${reflect_x}" reflect_y="${reflect_y}" reflect_z="${reflect_z}" />
+        <xacro:openarm_emit_origin origin="${joint_origin_cfg}" reflect_x="${reflect_x}" reflect_y="${reflect_y}" reflect_z="${reflect_z}" reflect_rotation="${reflect_rotation}" />
       </xacro:unless>
       <parent link="${parent_link}" />
@@ -94,7 +94,7 @@
         <xacro:property
           name="joint_axis_reflect_sign"
-          value="${-1 if ((reflect_x == -1 and joint_axis_cfg.x * joint_axis_cfg.x > 1e-18) or (reflect_y == -1 and joint_axis_cfg.y * joint_axis_cfg.y > 1e-18) or (reflect_z == -1 and joint_axis_cfg.z * joint_axis_cfg.z > 1e-18)) else 1}"
+          value="${-1 if ((reflect_x == -1 and joint_axis_cfg['x'] * joint_axis_cfg['x'] > 1e-18) or (reflect_y == -1 and joint_axis_cfg['y'] * joint_axis_cfg['y'] > 1e-18) or (reflect_z == -1 and joint_axis_cfg['z'] * joint_axis_cfg['z'] > 1e-18)) else 1}"
           lazy_eval="false" />
-        <axis xyz="${joint_axis_reflect_sign * joint_axis_cfg.x} ${joint_axis_reflect_sign * joint_axis_cfg.y} ${joint_axis_reflect_sign * joint_axis_cfg.z}" />
+        <axis xyz="${joint_axis_reflect_sign * joint_axis_cfg['x']} ${joint_axis_reflect_sign * joint_axis_cfg['y']} ${joint_axis_reflect_sign * joint_axis_cfg['z']}" />
       </xacro:if>
       <xacro:if value="${joint_type != 'fixed' and (limit_override != 'none' or source_joint_name in joint_limits)}">

File: assets/robot/openarm_v1.0/urdf/arm/openarm_arm.xacro (robot description, xacro)
@@ -16,4 +16,5 @@
   <xacro:macro name="openarm_arm" params="arm_type arm_prefix:='' no_prefix:=false description_pkg:='openarm_description' connected_to:='base' xyz:='0 0 0' rpy:='0 0 0' joint_limits inertials kinematics kinematics_link kinematics_offset:=none " >
     <xacro:property name="prefix" value="${'' if no_prefix else 'openarm' + '_' + arm_prefix}" />
+    <xacro:property name="mirror_rules" value="${xacro.load_yaml('$(find openarm_description)/assets/robot/openarm_v1.0/config/arm/mirroring.yaml')}" />
     <xacro:if value="${arm_prefix == '' or arm_prefix == 'right_'}">
       <xacro:property name="reflect" value="1" />
@@ -29,69 +30,43 @@
       </joint>
     </xacro:unless>
-    <xacro:link_with_sc no_prefix="${no_prefix}" name="link0" kinematics_link="${kinematics_link}" inertials="${inertials}" reflect="${reflect}"/>
-    <xacro:link_with_sc no_prefix="${no_prefix}" name="link1" kinematics_link="${kinematics_link}" inertials="${inertials}" reflect="${reflect}"/>
-    <joint name="${prefix}joint1" type="revolute">
-      <xacro:openarm-kinematics name="joint1" config="${kinematics}" reflect="${reflect}"/>
-      <parent link="${prefix}link0" />
-      <child link="${prefix}link1" />
-      <axis xyz="0 0 1" />
-      <xacro:openarm-limits name="joint1" config="${joint_limits}" offset="${-2.094396 if arm_prefix=='left_' else 0}"/>
-    </joint>
+    <xacro:link_with_sc no_prefix="${no_prefix}" name="link0" kinematics_link="${kinematics_link}" inertials="${inertials}" reflect="${reflect if 'link0' in mirror_rules.links else 1}"/>
+    <xacro:link_with_sc no_prefix="${no_prefix}" name="link1" kinematics_link="${kinematics_link}" inertials="${inertials}" reflect="${reflect if 'link1' in mirror_rules.links else 1}"/>
+    <xacro:openarm_joint_from_config
+      name="joint1" parent="link0" child="link1" axis="0 0 1" prefix="${prefix}"
+      kinematics="${kinematics}" joint_limits="${joint_limits}"
+     reflect="${reflect if 'joint1' in mirror_rules.joints else 1}" mirror_limits="${reflect == -1 and 'joint1' in mirror_rules.joints and arm_prefix == 'left_'}" />
     <!-- for bimanual offset -->
-    <xacro:link_with_sc no_prefix="${no_prefix}" name="link2" kinematics_link="${kinematics_link}" inertials="${inertials}" reflect="${reflect}"/>
-    <xacro:property name="limit_offset_joint2" value="0" />
-    <xacro:if value="${prefix.find('right_') != -1}">
-      <xacro:property name="limit_offset_joint2" value="${pi/2}" />
-    </xacro:if>
-    <xacro:if value="${prefix.find('left_') != -1}">
-      <xacro:property name="limit_offset_joint2" value="${-pi/2}" />
-    </xacro:if>
-    <joint name="${prefix}joint2" type="revolute">
-      <xacro:openarm-kinematics name="joint2" config="${kinematics}" offset="${kinematics_offset}" reflect="${reflect}"/>
-      <parent link="${prefix}link1" />
-      <child link="${prefix}link2" />
-      <axis xyz="-1 0 0" />
-      <xacro:openarm-limits name="joint2" config="${joint_limits}" reflect="${reflect}" offset="${limit_offset_joint2}"/>
-    </joint>
-    <xacro:link_with_sc no_prefix="${no_prefix}" name="link3" kinematics_link="${kinematics_link}" inertials="${inertials}"/>
-    <joint name="${prefix}joint3" type="revolute">
-      <xacro:openarm-kinematics name="joint3" config="${kinematics}" />
-      <parent link="${prefix}link2" />
-      <child link="${prefix}link3" />
-      <axis xyz="0 0 1" />
-      <xacro:openarm-limits name="joint3" config="${joint_limits}" />
-    </joint>
-    <xacro:link_with_sc no_prefix="${no_prefix}" name="link4" kinematics_link="${kinematics_link}" />
-    <joint name="${prefix}joint4" type="revolute">
-      <xacro:openarm-kinematics name="joint4" config="${kinematics}" />
-      <parent link="${prefix}link3" />
-      <child link="${prefix}link4" />
-      <axis xyz="0 1 0" />
-      <xacro:openarm-limits name="joint4" config="${joint_limits}" />
-    </joint>
-    <xacro:link_with_sc no_prefix="${no_prefix}" name="link5" kinematics_link="${kinematics_link}" inertials="${inertials}" reflect="${reflect}" />
-    <joint name="${prefix}joint5" type="revolute">
-      <xacro:openarm-kinematics name="joint5" config="${kinematics}" reflect="${reflect}"/>
-      <parent link="${prefix}link4" />
-      <child link="${prefix}link5" />
-      <axis xyz="0 0 1" />
-      <xacro:openarm-limits name="joint5" config="${joint_limits}" />
-    </joint>
-    <xacro:link_with_sc no_prefix="${no_prefix}" name="link6" kinematics_link="${kinematics_link}" inertials="${inertials}" reflect="${reflect}"/>
-    <joint name="${prefix}joint6" type="revolute">
-      <xacro:openarm-kinematics name="joint6" config="${kinematics}" />
-      <parent link="${prefix}link5" />
-      <child link="${prefix}link6" />
-      <axis xyz="1 0 0" />
-      <xacro:openarm-limits name="joint6" config="${joint_limits}" />
-    </joint>
-    <xacro:link_with_sc no_prefix="${no_prefix}" name="link7" kinematics_link="${kinematics_link}" inertials="${inertials}" reflect="${reflect}"/>
-    <joint name="${prefix}joint7" type="revolute">
-      <xacro:openarm-kinematics name="joint7" config="${kinematics}" />
-      <parent link="${prefix}link6"/>
-      <child link="${prefix}link7"/>
-      <axis xyz="0 ${reflect} 0"/>
-      <xacro:openarm-limits name="joint7" config="${joint_limits}" />
-    </joint>
+    <xacro:link_with_sc no_prefix="${no_prefix}" name="link2" kinematics_link="${kinematics_link}" inertials="${inertials}" reflect="${reflect if 'link2' in mirror_rules.links else 1}"/>
+    <xacro:property name="limit_offset_joint2" value="${pi/2 if ('right_' in prefix or 'left_' in prefix) else 0}" />
+    <xacro:openarm_joint_from_config
+      name="joint2" parent="link1" child="link2" axis="-1 0 0" prefix="${prefix}"
+      kinematics="${kinematics}" joint_limits="${joint_limits}"
+     reflect="${reflect if 'joint2' in mirror_rules.joints else 1}" mirror_limits="${reflect == -1 and 'joint2' in mirror_rules.joints}"
+      offset="${kinematics_offset}" limit_offset="${limit_offset_joint2}" />
+    <xacro:link_with_sc no_prefix="${no_prefix}" name="link3" kinematics_link="${kinematics_link}" inertials="${inertials}" reflect="${reflect if 'link3' in mirror_rules.links else 1}"/>
+    <xacro:openarm_joint_from_config
+      name="joint3" parent="link2" child="link3" axis="0 0 1" prefix="${prefix}"
+      kinematics="${kinematics}" joint_limits="${joint_limits}"
+     reflect="${reflect if 'joint3' in mirror_rules.joints else 1}" mirror_limits="${reflect == -1 and 'joint3' in mirror_rules.joints}" />
+    <xacro:link_with_sc no_prefix="${no_prefix}" name="link4" kinematics_link="${kinematics_link}" reflect="${reflect if 'link4' in mirror_rules.links else 1}"/>
+    <xacro:openarm_joint_from_config
+      name="joint4" parent="link3" child="link4" axis="0 1 0" prefix="${prefix}"
+      kinematics="${kinematics}" joint_limits="${joint_limits}"
+     reflect="${reflect if 'joint4' in mirror_rules.joints else 1}" mirror_limits="${reflect == -1 and 'joint4' in mirror_rules.joints}" />
+    <xacro:link_with_sc no_prefix="${no_prefix}" name="link5" kinematics_link="${kinematics_link}" inertials="${inertials}" reflect="${reflect if 'link5' in mirror_rules.links else 1}"/>
+    <xacro:openarm_joint_from_config
+      name="joint5" parent="link4" child="link5" axis="0 0 1" prefix="${prefix}"
+      kinematics="${kinematics}" joint_limits="${joint_limits}"
+     reflect="${reflect if 'joint5' in mirror_rules.joints else 1}" mirror_limits="${reflect == -1 and 'joint5' in mirror_rules.joints}" />
+    <xacro:link_with_sc no_prefix="${no_prefix}" name="link6" kinematics_link="${kinematics_link}" inertials="${inertials}" reflect="${reflect if 'link6' in mirror_rules.links else 1}"/>
+    <xacro:openarm_joint_from_config
+      name="joint6" parent="link5" child="link6" axis="1 0 0" prefix="${prefix}"
+      kinematics="${kinematics}" joint_limits="${joint_limits}"
+     reflect="${reflect if 'joint6' in mirror_rules.joints else 1}" mirror_limits="${reflect == -1 and 'joint6' in mirror_rules.joints}" />
+    <xacro:link_with_sc no_prefix="${no_prefix}" name="link7" kinematics_link="${kinematics_link}" inertials="${inertials}" reflect="${reflect if 'link7' in mirror_rules.links else 1}"/>
+    <xacro:openarm_joint_from_config
+      name="joint7" parent="link6" child="link7" axis="0 1 0" prefix="${prefix}"
+      kinematics="${kinematics}" joint_limits="${joint_limits}"
+     reflect="${reflect if 'joint7' in mirror_rules.joints else 1}" mirror_limits="${reflect == -1 and 'joint7' in mirror_rules.joints}" />
   </xacro:macro>
 </robot>

File: assets/robot/openarm_v1.0/urdf/arm/openarm_macro.xacro (robot description, xacro)
@@ -13,4 +13,5 @@
 -->
 <robot xmlns:xacro="http://www.ros.org/wiki/xacro">
+  <xacro:include filename="$(find openarm_description)/assets/common/links.xacro" />
   <xacro:macro name="openarm-inertials" params="name inertials:=^ reflect:=1">
     <xacro:unless value="${name in inertials}">
@@ -20,7 +21,5 @@
       <xacro:property name="I" value="${inertials[name]}" lazy_eval="false" />
       <inertial>
-        <origin
-          xyz="${I.origin.x} ${reflect * I.origin.y} ${I.origin.z}"
-          rpy="${I.origin.roll} ${I.origin.pitch} ${I.origin.yaw}" />
+        <xacro:openarm_emit_origin origin="${I.origin}" reflect_y="${reflect}" reflect_rotation="${True}" />
         <mass value="${I.mass}" />
         <xacro:if value="${'inertia' in I}">
@@ -37,5 +36,5 @@
     <link name="${prefix}${name}">
       <visual name="${prefix}${name}_visual">
-        <xacro:openarm-kinematics-link config="${kinematics_link}" name="${name}" />
+        <xacro:openarm-kinematics-link config="${kinematics_link}" name="${name}" reflect="${reflect}" />
         <geometry>
           <mesh filename="package://${description_pkg}/assets/robot/openarm_v1.0/mesh/arm/visual/${name}.dae" scale="0.001 ${0.001*reflect} 0.001" />
@@ -43,5 +42,5 @@
       </visual>
       <collision name="${prefix}${name}_collision">
-        <xacro:openarm-kinematics-link config="${kinematics_link}" name="${name}" />
+        <xacro:openarm-kinematics-link config="${kinematics_link}" name="${name}" reflect="${reflect}" />
         <geometry>
           <mesh filename="package://openarm_description/assets/robot/openarm_v1.0/mesh/arm/collision/${name}_symp.stl" scale="0.001 ${0.001*reflect} 0.001" />
@@ -128,8 +127,23 @@
     </xacro:unless>
   </xacro:macro>
-  <xacro:macro name="openarm-kinematics-link" params="config name">
+  <xacro:macro name="openarm-kinematics-link" params="config name reflect:=1">
     <xacro:property name="kinematics_link" value="${config[name]['kinematic']}" lazy_eval="false" />
-    <origin rpy="${kinematics_link.roll} ${kinematics_link.pitch} ${kinematics_link.yaw}"
-            xyz="${kinematics_link.x} ${kinematics_link.y} ${kinematics_link.z}" />
+    <xacro:openarm_emit_origin origin="${kinematics_link}" reflect_y="${reflect}" reflect_rotation="${True}" />
+  </xacro:macro>
+  <xacro:macro name="openarm_joint_from_config"
+    params="name parent child axis prefix kinematics joint_limits reflect:=1 offset:=none limit_offset:=0 mirror_limits:=${False}">
+    <xacro:property name="origin_cfg" value="${kinematics[name]['kinematic']}" />
+    <xacro:property name="offset_cfg" value="${offset[name]['kinematic_offset'] if offset != 'none' else dict(x=0, y=0, z=0, roll=0, pitch=0, yaw=0)}" />
+    <xacro:property name="right_origin" value="${dict([(key, origin_cfg[key] + offset_cfg[key]) for key in ['x', 'y', 'z', 'roll', 'pitch', 'yaw']])}" />
+    <xacro:property name="axis_values" value="${[float(value) for value in axis.split()]}" />
+    <xacro:property name="limit" value="${joint_limits[name]['limit']}" />
+    <xacro:openarm_emit_joint
+      joint_name="${prefix}${name}" joint_type="revolute"
+      parent_link="${prefix}${parent}" child_link="${prefix}${child}"
+      joint_origins="${dict()}" joint_axes="${dict()}" joint_limits="${dict()}"
+      origin_override="${right_origin}"
+      axis_override="${dict(x=axis_values[0], y=axis_values[1], z=axis_values[2])}"
+      limit_override="${dict(lower=limit.lower + limit_offset, upper=limit.upper + limit_offset, effort=limit.effort, velocity=limit.velocity)}"
+      reflect_y="${reflect}" reflect_rotation="${True}" mirror_limit_sign="${mirror_limits}" />
   </xacro:macro>
 </robot>

File: assets/robot/openarm_v1.0/urdf/example/v1.urdf (robot description, URDF)
Before this commit: robot openarm, 26 links, 25 joints
Joints:
- joint openarm_left_joint1: axis 0 0 1 -> 0.0 0.0 1.0; limit lower=-3.490659 upper=1.3962629999999998 effort=40 velocity=16.754666 -> lower=-3.490659 upper=1.396263 effort=40 velocity=16.754666; origin xyz=0.0 0.0 0.0625 rpy=0 0 0 -> xyz=0.0 -0.0 0.0625 rpy=0 0 0
- joint openarm_left_joint2: axis -1 0 0 -> -1.0 0.0 0.0; origin xyz=-0.0301 0.0 0.06 rpy=-1.57079632679 0 0 -> xyz=-0.0301 -0.0 0.06 rpy=-1.57079632679 0 0
- joint openarm_left_joint3: axis 0 0 1 -> 0.0 0.0 1.0; origin xyz=0.0301 0.0 0.06625 rpy=0 0 0 -> xyz=0.0301 -0.0 0.06625 rpy=0 0 0
- joint openarm_left_joint4: axis 0 1 0 -> 0.0 1.0 0.0; origin xyz=-0.0 0.0315 0.15375 rpy=0 0 0 -> xyz=0.0 0.0315 0.15375 rpy=0 0 0
- joint openarm_left_joint5: axis 0 0 1 -> 0.0 0.0 1.0
- joint openarm_left_joint6: axis 1 0 0 -> 1.0 0.0 0.0; origin xyz=0.0375 0.0 0.1205 rpy=0 0 0 -> xyz=0.0375 -0.0 0.1205 rpy=0 0 0
- joint openarm_left_joint7: axis 0 -1 0 -> -0.0 -1.0 -0.0; origin xyz=-0.0375 0.0 0.0 rpy=0 0 0 -> xyz=-0.0375 -0.0 0.0 rpy=0 0 0
- joint openarm_right_joint1: axis 0 0 1 -> 0.0 0.0 1.0
- joint openarm_right_joint2: axis -1 0 0 -> -1.0 0.0 0.0
- joint openarm_right_joint3: axis 0 0 1 -> 0.0 0.0 1.0
- joint openarm_right_joint4: axis 0 1 0 -> 0.0 1.0 0.0; origin xyz=-0.0 0.0315 0.15375 rpy=0 0 0 -> xyz=0.0 0.0315 0.15375 rpy=0 0 0
- joint openarm_right_joint5: axis 0 0 1 -> 0.0 0.0 1.0
- joint openarm_right_joint6: axis 1 0 0 -> 1.0 0.0 0.0
- joint openarm_right_joint7: axis 0 1 0 -> 0.0 1.0 0.0

Commit message: Support component-wise joint-axis and origin reflection

File: assets/common/links.xacro (robot description, xacro)
@@ -78,13 +78,13 @@
     </link>
   </xacro:macro>
-  <xacro:macro name="openarm_emit_joint" params="joint_name joint_type parent_link child_link joint_origins joint_axes joint_limits reflect_x:=1 reflect_y:=1 reflect_z:=1 source_name:='' origin_override:=none axis_override:=none limit_override:=none mimic_override:=none mirror_limit_sign:=false frame_shift:=none">
+  <xacro:macro name="openarm_emit_joint" params="joint_name joint_type parent_link child_link joint_origins joint_axes joint_limits reflect_x:=1 reflect_y:=1 reflect_z:=1 source_name:='' origin_override:=none axis_override:=none limit_override:=none mimic_override:=none mirror_limit_sign:=false frame_shift:=none reflect_rotation:=${False}">
     <xacro:property name="source_joint_name" value="${source_name if source_name != '' else joint_name}" />
     <xacro:property name="joint_origin_cfg" value="${origin_override if origin_override != 'none' else joint_origins[source_joint_name].origin}" lazy_eval="false" />
     <joint name="${joint_name}" type="${joint_type}">
       <xacro:if value="${frame_shift != 'none'}">
-        <xacro:openarm_emit_composed_origin first="${frame_shift}" second="${joint_origin_cfg}" reflect_x="${reflect_x}" reflect_y="${reflect_y}" reflect_z="${reflect_z}" />
+        <xacro:openarm_emit_composed_origin first="${frame_shift}" second="${joint_origin_cfg}" reflect_x="${reflect_x}" reflect_y="${reflect_y}" reflect_z="${reflect_z}" reflect_rotation="${reflect_rotation}" />
       </xacro:if>
       <xacro:unless value="${frame_shift != 'none'}">
-        <xacro:openarm_emit_origin origin="${joint_origin_cfg}" reflect_x="${reflect_x}" reflect_y="${reflect_y}" reflect_z="${reflect_z}" />
+        <xacro:openarm_emit_origin origin="${joint_origin_cfg}" reflect_x="${reflect_x}" reflect_y="${reflect_y}" reflect_z="${reflect_z}" reflect_rotation="${reflect_rotation}" />
       </xacro:unless>
       <parent link="${parent_link}" />
@@ -93,8 +93,8 @@
         <xacro:property name="joint_axis_cfg" value="${axis_override if axis_override != 'none' else joint_axes[source_joint_name].axis}" lazy_eval="false" />
         <xacro:property
-          name="joint_axis_reflect_sign"
-          value="${-1 if ((reflect_x == -1 and joint_axis_cfg.x * joint_axis_cfg.x > 1e-18) or (reflect_y == -1 and joint_axis_cfg.y * joint_axis_cfg.y > 1e-18) or (reflect_z == -1 and joint_axis_cfg.z * joint_axis_cfg.z > 1e-18)) else 1}"
+          name="mirror_limit_for_axis"
+          value="${(reflect_x == -1 and joint_axis_cfg['x'] * joint_axis_cfg['x'] > 1e-18) or (reflect_y == -1 and joint_axis_cfg['y'] * joint_axis_cfg['y'] > 1e-18) or (reflect_z == -1 and joint_axis_cfg['z'] * joint_axis_cfg['z'] > 1e-18)}"
           lazy_eval="false" />
-        <axis xyz="${joint_axis_reflect_sign * joint_axis_cfg.x} ${joint_axis_reflect_sign * joint_axis_cfg.y} ${joint_axis_reflect_sign * joint_axis_cfg.z}" />
+        <axis xyz="${reflect_x * joint_axis_cfg['x']} ${reflect_y * joint_axis_cfg['y']} ${reflect_z * joint_axis_cfg['z']}" />
       </xacro:if>
       <xacro:if value="${joint_type != 'fixed' and (limit_override != 'none' or source_joint_name in joint_limits)}">
@@ -102,5 +102,5 @@
         <xacro:property
           name="effective_mirror_limit_sign"
-          value="${mirror_limit_sign or joint_axis_reflect_sign == -1}"
+          value="${mirror_limit_sign or mirror_limit_for_axis}"
           lazy_eval="false" />
         <xacro:if value="${effective_mirror_limit_sign}">
