Commit message: Reframe V1 arm links while preserving motor coordinates

File: assets/robot/openarm_v1.0/urdf/arm/openarm_arm.xacro (robot description, xacro)
@@ -35,5 +35,5 @@
       <parent link="${prefix}link0" />
       <child link="${prefix}link1" />
-      <axis xyz="0 0 1" />
+      <axis xyz="0 ${-reflect} 0" />
       <xacro:openarm-limits name="joint1" config="${joint_limits}" offset="${-2.094396 if arm_prefix=='left_' else 0}"/>
     </joint>
@@ -59,5 +59,5 @@
       <parent link="${prefix}link2" />
       <child link="${prefix}link3" />
-      <axis xyz="0 0 1" />
+      <axis xyz="0 0 -1" />
       <xacro:openarm-limits name="joint3" config="${joint_limits}" />
     </joint>
@@ -67,5 +67,5 @@
       <parent link="${prefix}link3" />
       <child link="${prefix}link4" />
-      <axis xyz="0 1 0" />
+      <axis xyz="0 -1 0" />
       <xacro:openarm-limits name="joint4" config="${joint_limits}" />
     </joint>
@@ -75,5 +75,5 @@
       <parent link="${prefix}link4" />
       <child link="${prefix}link5" />
-      <axis xyz="0 0 1" />
+      <axis xyz="0 0 -1" />
       <xacro:openarm-limits name="joint5" config="${joint_limits}" />
     </joint>
@@ -91,5 +91,5 @@
       <parent link="${prefix}link6"/>
       <child link="${prefix}link7"/>
-      <axis xyz="0 ${reflect} 0"/>
+      <axis xyz="0 ${-reflect} 0"/>
       <xacro:openarm-limits name="joint7" config="${joint_limits}" />
     </joint>

File: assets/robot/openarm_v1.0/urdf/arm/openarm_macro.xacro (robot description, xacro)
@@ -37,5 +37,5 @@
     <link name="${prefix}${name}">
       <visual name="${prefix}${name}_visual">
-        <xacro:openarm-kinematics-link config="${kinematics_link}" name="${name}" />
+        <xacro:openarm-kinematics-link config="${kinematics_link}" name="${name}" reflect="${reflect}" />
         <geometry>
           <mesh filename="package://${description_pkg}/assets/robot/openarm_v1.0/mesh/arm/visual/${name}.dae" scale="0.001 ${0.001*reflect} 0.001" />
@@ -43,5 +43,5 @@
       </visual>
       <collision name="${prefix}${name}_collision">
-        <xacro:openarm-kinematics-link config="${kinematics_link}" name="${name}" />
+        <xacro:openarm-kinematics-link config="${kinematics_link}" name="${name}" reflect="${reflect}" />
         <geometry>
           <mesh filename="package://openarm_description/assets/robot/openarm_v1.0/mesh/arm/collision/${name}_symp.stl" scale="0.001 ${0.001*reflect} 0.001" />
@@ -119,17 +119,17 @@
       <xacro:property name="offset" value="${offset[name]['kinematic_offset']}" lazy_eval="false" />
       <origin
-        xyz="${kinematics.x + offset.x} ${kinematics.y + offset.y} ${kinematics.z + offset.z}"
+        xyz="${kinematics.x + offset.x} ${reflect*(kinematics.y + offset.y)} ${kinematics.z + offset.z}"
         rpy="${reflect*(kinematics.roll + offset.roll)} ${reflect*(kinematics.pitch + offset.pitch)} ${reflect*(kinematics.yaw + offset.yaw)}" />
     </xacro:if>
     <xacro:unless value="${offset != 'none'}">
       <origin
-        xyz="${kinematics.x} ${kinematics.y} ${kinematics.z}"
+        xyz="${kinematics.x} ${reflect*kinematics.y} ${kinematics.z}"
         rpy="${reflect*kinematics.roll} ${reflect*kinematics.pitch} ${reflect*kinematics.yaw}" />
     </xacro:unless>
   </xacro:macro>
-  <xacro:macro name="openarm-kinematics-link" params="config name">
+  <xacro:macro name="openarm-kinematics-link" params="config name reflect:=1">
     <xacro:property name="kinematics_link" value="${config[name]['kinematic']}" lazy_eval="false" />
-    <origin rpy="${kinematics_link.roll} ${kinematics_link.pitch} ${kinematics_link.yaw}"
-            xyz="${kinematics_link.x} ${kinematics_link.y} ${kinematics_link.z}" />
+    <origin rpy="${reflect*kinematics_link.roll} ${kinematics_link.pitch} ${reflect*kinematics_link.yaw}"
+            xyz="${kinematics_link.x} ${reflect*kinematics_link.y} ${kinematics_link.z}" />
   </xacro:macro>
 </robot>

File: assets/robot/openarm_v1.0/urdf/ee/ee_dispatcher.xacro (robot description, xacro)
@@ -21,4 +21,6 @@
         arm_prefix="${arm_prefix}"
         ee_type="${ee_type}"
+        xyz_ee="${xyz_ee}"
+        rpy_ee="${rpy_ee}"
         ee_kinematics="${ee_kinematics}"
         ee_kinematics_link="${ee_kinematics_link}"

File: assets/robot/openarm_v1.0/urdf/ee/parallel_link/openarm_parallel_gripper.xacro (robot description, xacro)
@@ -13,4 +13,5 @@
 -->
 <robot xmlns:xacro="http://www.ros.org/wiki/xacro" name="parallel_gripper">
+  <xacro:include filename="$(find openarm_description)/assets/common/transforms.xacro" />
   <!-- tcp_xyz: offset from hand to hand_tcp (metres). -->
   <xacro:macro name="openarm_parallel_gripper" params="connected_to:='' arm_type arm_prefix:='' ee_type ee_inertials ee_kinematics ee_kinematics_link ee_joints_limits rpy_ee:='0 0 0' xyz_ee:='0 0 0' tcp_xyz:='0 0 0.09' tcp_rpy:='0 0 0' description_pkg:=openarm_description no_prefix:=false mesh_root:=''">
@@ -34,5 +35,9 @@
     </link>
     <joint name="${ee_prefix}hand_joint" type="fixed">
-      <xacro:openarm-ee-kinematics config="${ee_kinematics}" name="hand" />
+      <xacro:property name="mount_xyz" value="${[float(v) for v in xyz_ee.split()]}" />
+      <xacro:property name="mount_rpy" value="${[float(v) for v in rpy_ee.split()]}" />
+      <xacro:openarm_emit_composed_origin
+        first="${dict(x=mount_xyz[0], y=mount_xyz[1], z=mount_xyz[2], roll=mount_rpy[0], pitch=mount_rpy[1], yaw=mount_rpy[2])}"
+        second="${ee_kinematics['hand']['kinematic']}" />
       <parent link="${connected_to}" />
       <child link="${ee_prefix}hand" />

File: assets/robot/openarm_v1.0/urdf/example/v1.urdf (robot description, URDF)
Before this commit: robot openarm, 26 links, 25 joints
Joints:
- joint openarm_left_hand_joint: origin xyz=0.0 0.0 0.1001 rpy=0 0 0 -> xyz=0.0 -1.2258714459465006e-17 -0.1001 rpy=3.141592653589793 -0.0 0.0
- joint openarm_left_joint1: axis 0 0 1 -> 0 1 0; origin xyz=0.0 0.0 0.0625 rpy=0 0 0 -> xyz=0 0.0625 0 rpy=0 0 0
- joint openarm_left_joint2: origin xyz=-0.0301 0.0 0.06 rpy=-1.57079632679 0 0 -> xyz=0.0 0.06 0.0 rpy=4.8965276278067904e-12 0 0
- joint openarm_left_joint3: axis 0 0 1 -> 0 0 -1; origin xyz=0.0301 0.0 0.06625 rpy=0 0 0 -> xyz=0 0 -0.06625 rpy=0 0 0
- joint openarm_left_joint4: axis 0 1 0 -> 0 -1 0; origin xyz=-0.0 0.0315 0.15375 rpy=0 0 0 -> xyz=0 0 -0.15375 rpy=0 0 0
- joint openarm_left_joint5: axis 0 0 1 -> 0 0 -1; origin xyz=0.0 -0.0315 0.0955 rpy=0 0 0 -> xyz=0 0 -0.0955 rpy=0 0 0
- joint openarm_left_joint6: origin xyz=0.0375 0.0 0.1205 rpy=0 0 0 -> xyz=0 0 -0.1205 rpy=0 0 0
- joint openarm_left_joint7: axis 0 -1 0 -> 0 1 0; origin xyz=-0.0375 0.0 0.0 rpy=0 0 0 -> xyz=0 0 0 rpy=0 0 0
- joint openarm_left_openarm_body_link0_joint: origin xyz=0.0 0.030 0.697 rpy=-1.5708 0 0 -> xyz=0.0 0.030 0.697 rpy=-3.673205103416066e-06 0 0
- joint openarm_right_hand_joint: origin xyz=0.0 0.0 0.1001 rpy=0 0 0 -> xyz=0.0 -1.2258714459465006e-17 -0.1001 rpy=3.141592653589793 -0.0 0.0
- joint openarm_right_joint1: axis 0 0 1 -> 0 -1 0; origin xyz=0.0 0.0 0.0625 rpy=0 0 0 -> xyz=0 -0.0625 0 rpy=0 0 0
- joint openarm_right_joint2: origin xyz=-0.0301 0.0 0.06 rpy=1.57079632679 0 0 -> xyz=0.0 -0.06 0.0 rpy=-4.8965276278067904e-12 0 0
- joint openarm_right_joint3: axis 0 0 1 -> 0 0 -1; origin xyz=0.0301 0.0 0.06625 rpy=0 0 0 -> xyz=0 0 -0.06625 rpy=0 0 0
- joint openarm_right_joint4: axis 0 1 0 -> 0 -1 0; origin xyz=-0.0 0.0315 0.15375 rpy=0 0 0 -> xyz=0 0 -0.15375 rpy=0 0 0
- joint openarm_right_joint5: axis 0 0 1 -> 0 0 -1; origin xyz=0.0 -0.0315 0.0955 rpy=0 0 0 -> xyz=0 0 -0.0955 rpy=0 0 0
- joint openarm_right_joint6: origin xyz=0.0375 0.0 0.1205 rpy=0 0 0 -> xyz=0 0 -0.1205 rpy=0 0 0
- joint openarm_right_joint7: axis 0 1 0 -> 0 -1 0; origin xyz=-0.0375 0.0 0.0 rpy=0 0 0 -> xyz=0 0 0 rpy=0 0 0
- joint openarm_right_openarm_body_link0_joint: origin xyz=0.0 -0.030 0.697 rpy=1.5708 0 0 -> xyz=0.0 -0.030 0.697 rpy=3.673205103416066e-06 0 0

File: assets/robot/openarm_v1.0/urdf/openarm_v10.urdf.xacro (robot description, xacro)
@@ -30,7 +30,7 @@
   <xacro:arg name="bimanual" default="true" />
   <xacro:arg name="right_arm_base_xyz" default="0.0 -0.030 0.697" />
-  <xacro:arg name="right_arm_base_rpy" default="1.5708 0 0" />
+  <xacro:arg name="right_arm_base_rpy" default="3.673205103416066e-06 0 0" />
   <xacro:arg name="left_arm_base_xyz" default="0.0 0.030 0.697" />
-  <xacro:arg name="left_arm_base_rpy" default="-1.5708 0 0" />
+  <xacro:arg name="left_arm_base_rpy" default="-3.673205103416066e-06 0 0" />
   <xacro:arg name="can_fd" default="true" />
   <xacro:property name="accepted_arm_types" value="${('v10', 'v1.0', 'v1_0', 'openarm_v10', 'openarm_v1.0', 'openarm_v1_0')}" />

File: assets/robot/openarm_v1.0/urdf/robot/openarm_robot.xacro (robot description, xacro)
@@ -111,4 +111,5 @@
             arm_prefix="left_"
             ee_type="${ee_type}"
+            rpy_ee="${pi} 0 0"
             ee_kinematics="${ee_kinematics}"
             ee_kinematics_link="${ee_kinematics_link}"
@@ -121,4 +122,5 @@
             arm_prefix="right_"
             ee_type="${ee_type}"
+            rpy_ee="${pi} 0 0"
             ee_kinematics="${ee_kinematics}"
             ee_kinematics_link="${ee_kinematics_link}"
@@ -142,15 +144,16 @@
     </xacro:if>
     <xacro:if value="${not bimanual}">
+        <link name="world" />
         <xacro:openarm_arm
             arm_type="${arm_type}"
             arm_prefix="${arm_prefix_modified}"
             no_prefix="${no_prefix}"
-            xyz="${xyz}"
-            rpy="${rpy}"
+            xyz="0 0 0"
+            rpy="${-pi/2 if arm_prefix_modified in ['', 'right_'] else pi/2} 0 0"
             joint_limits="${joint_limits}"
             kinematics="${kinematics}"
             kinematics_link="${kinematics_link}"
             inertials="${inertials}"
-            connected_to=""
+            connected_to="world"
         />
         <xacro:openarm_ee
@@ -159,4 +162,5 @@
             no_prefix="${no_prefix}"
             ee_type="${ee_type}"
+            rpy_ee="${pi} 0 0"
             ee_kinematics="${ee_kinematics}"
             ee_kinematics_link="${ee_kinematics_link}"

Commit message: Revert "Reframe V1 arm links while preserving motor coordinates"
This reverts commit 274794ef0faa6b28cbc728bdf9e08ab9e3ee65b9.

File: assets/robot/openarm_v1.0/urdf/arm/openarm_arm.xacro (robot description, xacro)
@@ -35,5 +35,5 @@
       <parent link="${prefix}link0" />
       <child link="${prefix}link1" />
-      <axis xyz="0 ${-reflect} 0" />
+      <axis xyz="0 0 1" />
       <xacro:openarm-limits name="joint1" config="${joint_limits}" offset="${-2.094396 if arm_prefix=='left_' else 0}"/>
     </joint>
@@ -59,5 +59,5 @@
       <parent link="${prefix}link2" />
       <child link="${prefix}link3" />
-      <axis xyz="0 0 -1" />
+      <axis xyz="0 0 1" />
       <xacro:openarm-limits name="joint3" config="${joint_limits}" />
     </joint>
@@ -67,5 +67,5 @@
       <parent link="${prefix}link3" />
       <child link="${prefix}link4" />
-      <axis xyz="0 -1 0" />
+      <axis xyz="0 1 0" />
       <xacro:openarm-limits name="joint4" config="${joint_limits}" />
     </joint>
@@ -75,5 +75,5 @@
       <parent link="${prefix}link4" />
       <child link="${prefix}link5" />
-      <axis xyz="0 0 -1" />
+      <axis xyz="0 0 1" />
       <xacro:openarm-limits name="joint5" config="${joint_limits}" />
     </joint>
@@ -91,5 +91,5 @@
       <parent link="${prefix}link6"/>
       <child link="${prefix}link7"/>
-      <axis xyz="0 ${-reflect} 0"/>
+      <axis xyz="0 ${reflect} 0"/>
       <xacro:openarm-limits name="joint7" config="${joint_limits}" />
     </joint>

File: assets/robot/openarm_v1.0/urdf/arm/openarm_macro.xacro (robot description, xacro)
@@ -37,5 +37,5 @@
     <link name="${prefix}${name}">
       <visual name="${prefix}${name}_visual">
-        <xacro:openarm-kinematics-link config="${kinematics_link}" name="${name}" reflect="${reflect}" />
+        <xacro:openarm-kinematics-link config="${kinematics_link}" name="${name}" />
         <geometry>
           <mesh filename="package://${description_pkg}/assets/robot/openarm_v1.0/mesh/arm/visual/${name}.dae" scale="0.001 ${0.001*reflect} 0.001" />
@@ -43,5 +43,5 @@
       </visual>
       <collision name="${prefix}${name}_collision">
-        <xacro:openarm-kinematics-link config="${kinematics_link}" name="${name}" reflect="${reflect}" />
+        <xacro:openarm-kinematics-link config="${kinematics_link}" name="${name}" />
         <geometry>
           <mesh filename="package://openarm_description/assets/robot/openarm_v1.0/mesh/arm/collision/${name}_symp.stl" scale="0.001 ${0.001*reflect} 0.001" />
@@ -119,17 +119,17 @@
       <xacro:property name="offset" value="${offset[name]['kinematic_offset']}" lazy_eval="false" />
       <origin
-        xyz="${kinematics.x + offset.x} ${reflect*(kinematics.y + offset.y)} ${kinematics.z + offset.z}"
+        xyz="${kinematics.x + offset.x} ${kinematics.y + offset.y} ${kinematics.z + offset.z}"
         rpy="${reflect*(kinematics.roll + offset.roll)} ${reflect*(kinematics.pitch + offset.pitch)} ${reflect*(kinematics.yaw + offset.yaw)}" />
     </xacro:if>
     <xacro:unless value="${offset != 'none'}">
       <origin
-        xyz="${kinematics.x} ${reflect*kinematics.y} ${kinematics.z}"
+        xyz="${kinematics.x} ${kinematics.y} ${kinematics.z}"
         rpy="${reflect*kinematics.roll} ${reflect*kinematics.pitch} ${reflect*kinematics.yaw}" />
     </xacro:unless>
   </xacro:macro>
-  <xacro:macro name="openarm-kinematics-link" params="config name reflect:=1">
+  <xacro:macro name="openarm-kinematics-link" params="config name">
     <xacro:property name="kinematics_link" value="${config[name]['kinematic']}" lazy_eval="false" />
-    <origin rpy="${reflect*kinematics_link.roll} ${kinematics_link.pitch} ${reflect*kinematics_link.yaw}"
-            xyz="${kinematics_link.x} ${reflect*kinematics_link.y} ${kinematics_link.z}" />
+    <origin rpy="${kinematics_link.roll} ${kinematics_link.pitch} ${kinematics_link.yaw}"
+            xyz="${kinematics_link.x} ${kinematics_link.y} ${kinematics_link.z}" />
   </xacro:macro>
 </robot>

File: assets/robot/openarm_v1.0/urdf/ee/ee_dispatcher.xacro (robot description, xacro)
@@ -21,6 +21,4 @@
         arm_prefix="${arm_prefix}"
         ee_type="${ee_type}"
-        xyz_ee="${xyz_ee}"
-        rpy_ee="${rpy_ee}"
         ee_kinematics="${ee_kinematics}"
         ee_kinematics_link="${ee_kinematics_link}"

File: assets/robot/openarm_v1.0/urdf/ee/parallel_link/openarm_parallel_gripper.xacro (robot description, xacro)
@@ -13,5 +13,4 @@
 -->
 <robot xmlns:xacro="http://www.ros.org/wiki/xacro" name="parallel_gripper">
-  <xacro:include filename="$(find openarm_description)/assets/common/transforms.xacro" />
   <!-- tcp_xyz: offset from hand to hand_tcp (metres). -->
   <xacro:macro name="openarm_parallel_gripper" params="connected_to:='' arm_type arm_prefix:='' ee_type ee_inertials ee_kinematics ee_kinematics_link ee_joints_limits rpy_ee:='0 0 0' xyz_ee:='0 0 0' tcp_xyz:='0 0 0.09' tcp_rpy:='0 0 0' description_pkg:=openarm_description no_prefix:=false mesh_root:=''">
@@ -35,9 +34,5 @@
     </link>
     <joint name="${ee_prefix}hand_joint" type="fixed">
-      <xacro:property name="mount_xyz" value="${[float(v) for v in xyz_ee.split()]}" />
-      <xacro:property name="mount_rpy" value="${[float(v) for v in rpy_ee.split()]}" />
-      <xacro:openarm_emit_composed_origin
-        first="${dict(x=mount_xyz[0], y=mount_xyz[1], z=mount_xyz[2], roll=mount_rpy[0], pitch=mount_rpy[1], yaw=mount_rpy[2])}"
-        second="${ee_kinematics['hand']['kinematic']}" />
+      <xacro:openarm-ee-kinematics config="${ee_kinematics}" name="hand" />
       <parent link="${connected_to}" />
       <child link="${ee_prefix}hand" />

File: assets/robot/openarm_v1.0/urdf/example/v1.urdf (robot description, URDF)
Before this commit: robot openarm, 26 links, 25 joints
Joints:
- joint openarm_left_hand_joint: origin xyz=0.0 -1.2258714459465006e-17 -0.1001 rpy=3.141592653589793 -0.0 0.0 -> xyz=0.0 0.0 0.1001 rpy=0 0 0
- joint openarm_left_joint1: axis 0 1 0 -> 0 0 1; origin xyz=0 0.0625 0 rpy=0 0 0 -> xyz=0.0 0.0 0.0625 rpy=0 0 0
- joint openarm_left_joint2: origin xyz=0.0 0.06 0.0 rpy=4.8965276278067904e-12 0 0 -> xyz=-0.0301 0.0 0.06 rpy=-1.57079632679 0 0
- joint openarm_left_joint3: axis 0 0 -1 -> 0 0 1; origin xyz=0 0 -0.06625 rpy=0 0 0 -> xyz=0.0301 0.0 0.06625 rpy=0 0 0
- joint openarm_left_joint4: axis 0 -1 0 -> 0 1 0; origin xyz=0 0 -0.15375 rpy=0 0 0 -> xyz=-0.0 0.0315 0.15375 rpy=0 0 0
- joint openarm_left_joint5: axis 0 0 -1 -> 0 0 1; origin xyz=0 0 -0.0955 rpy=0 0 0 -> xyz=0.0 -0.0315 0.0955 rpy=0 0 0
- joint openarm_left_joint6: origin xyz=0 0 -0.1205 rpy=0 0 0 -> xyz=0.0375 0.0 0.1205 rpy=0 0 0
- joint openarm_left_joint7: axis 0 1 0 -> 0 -1 0; origin xyz=0 0 0 rpy=0 0 0 -> xyz=-0.0375 0.0 0.0 rpy=0 0 0
- joint openarm_left_openarm_body_link0_joint: origin xyz=0.0 0.030 0.697 rpy=-3.673205103416066e-06 0 0 -> xyz=0.0 0.030 0.697 rpy=-1.5708 0 0
- joint openarm_right_hand_joint: origin xyz=0.0 -1.2258714459465006e-17 -0.1001 rpy=3.141592653589793 -0.0 0.0 -> xyz=0.0 0.0 0.1001 rpy=0 0 0
- joint openarm_right_joint1: axis 0 -1 0 -> 0 0 1; origin xyz=0 -0.0625 0 rpy=0 0 0 -> xyz=0.0 0.0 0.0625 rpy=0 0 0
- joint openarm_right_joint2: origin xyz=0.0 -0.06 0.0 rpy=-4.8965276278067904e-12 0 0 -> xyz=-0.0301 0.0 0.06 rpy=1.57079632679 0 0
- joint openarm_right_joint3: axis 0 0 -1 -> 0 0 1; origin xyz=0 0 -0.06625 rpy=0 0 0 -> xyz=0.0301 0.0 0.06625 rpy=0 0 0
- joint openarm_right_joint4: axis 0 -1 0 -> 0 1 0; origin xyz=0 0 -0.15375 rpy=0 0 0 -> xyz=-0.0 0.0315 0.15375 rpy=0 0 0
- joint openarm_right_joint5: axis 0 0 -1 -> 0 0 1; origin xyz=0 0 -0.0955 rpy=0 0 0 -> xyz=0.0 -0.0315 0.0955 rpy=0 0 0
- joint openarm_right_joint6: origin xyz=0 0 -0.1205 rpy=0 0 0 -> xyz=0.0375 0.0 0.1205 rpy=0 0 0
- joint openarm_right_joint7: axis 0 -1 0 -> 0 1 0; origin xyz=0 0 0 rpy=0 0 0 -> xyz=-0.0375 0.0 0.0 rpy=0 0 0
- joint openarm_right_openarm_body_link0_joint: origin xyz=0.0 -0.030 0.697 rpy=3.673205103416066e-06 0 0 -> xyz=0.0 -0.030 0.697 rpy=1.5708 0 0

File: assets/robot/openarm_v1.0/urdf/openarm_v10.urdf.xacro (robot description, xacro)
@@ -30,7 +30,7 @@
   <xacro:arg name="bimanual" default="true" />
   <xacro:arg name="right_arm_base_xyz" default="0.0 -0.030 0.697" />
-  <xacro:arg name="right_arm_base_rpy" default="3.673205103416066e-06 0 0" />
+  <xacro:arg name="right_arm_base_rpy" default="1.5708 0 0" />
   <xacro:arg name="left_arm_base_xyz" default="0.0 0.030 0.697" />
-  <xacro:arg name="left_arm_base_rpy" default="-3.673205103416066e-06 0 0" />
+  <xacro:arg name="left_arm_base_rpy" default="-1.5708 0 0" />
   <xacro:arg name="can_fd" default="true" />
   <xacro:property name="accepted_arm_types" value="${('v10', 'v1.0', 'v1_0', 'openarm_v10', 'openarm_v1.0', 'openarm_v1_0')}" />

File: assets/robot/openarm_v1.0/urdf/robot/openarm_robot.xacro (robot description, xacro)
@@ -111,5 +111,4 @@
             arm_prefix="left_"
             ee_type="${ee_type}"
-            rpy_ee="${pi} 0 0"
             ee_kinematics="${ee_kinematics}"
             ee_kinematics_link="${ee_kinematics_link}"
@@ -122,5 +121,4 @@
             arm_prefix="right_"
             ee_type="${ee_type}"
-            rpy_ee="${pi} 0 0"
             ee_kinematics="${ee_kinematics}"
             ee_kinematics_link="${ee_kinematics_link}"
@@ -144,16 +142,15 @@
     </xacro:if>
     <xacro:if value="${not bimanual}">
-        <link name="world" />
         <xacro:openarm_arm
             arm_type="${arm_type}"
             arm_prefix="${arm_prefix_modified}"
             no_prefix="${no_prefix}"
-            xyz="0 0 0"
-            rpy="${-pi/2 if arm_prefix_modified in ['', 'right_'] else pi/2} 0 0"
+            xyz="${xyz}"
+            rpy="${rpy}"
             joint_limits="${joint_limits}"
             kinematics="${kinematics}"
             kinematics_link="${kinematics_link}"
             inertials="${inertials}"
-            connected_to="world"
+            connected_to=""
         />
         <xacro:openarm_ee
@@ -162,5 +159,4 @@
             no_prefix="${no_prefix}"
             ee_type="${ee_type}"
-            rpy_ee="${pi} 0 0"
             ee_kinematics="${ee_kinematics}"
             ee_kinematics_link="${ee_kinematics_link}"
