Commit message: feat: add modular V2 camera assembly and updated visuals

File: assets/robot/openarm_v2.0/urdf/example/v2.urdf (robot description, URDF)
Before this commit: robot openarm_v20, 22 links, 21 joints
Links:
- added link openarm_body_link0_camera_mount_point
- added link openarm_left_camera_view_frame
- added link openarm_right_camera_view_frame
- link openarm_body_link0: geometry collision mesh filename=package://openarm_description/assets/robot/openarm_v2.0/mes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 scale=0.001 0.001 0.001; visual mesh filename=package://openarm_description/assets/robot/openarm_v2.0/mes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 scale=1.0 1.0 1.0
Joints:
- added joint openarm_body_link0_camera_mount_point_joint: type fixed, parent openarm_body_link0, child openarm_body_link0_camera_mount_point, origin xyz=0.03 0.0 0.743 rpy=0.0 0.0 0.0
- added joint openarm_left_camera_view_frame_joint: type fixed, parent openarm_left_ee_base_link, child openarm_left_camera_view_frame, origin xyz=0.021835300000000002 0.024136 -0.086895 rpy=-2.1009 1.1424 -2.1431
- added joint openarm_right_camera_view_frame_joint: type fixed, parent openarm_right_ee_base_link, child openarm_right_camera_view_frame, origin xyz=0.021835300000000002 -0.024136 -0.086895 rpy=2.1009 1.1424 2.1431

File: assets/robot/openarm_v2.0/urdf/utils/openarm_v20_ee.xacro (robot description, xacro)
@@ -210,4 +210,13 @@
         frame_shift="${resolved_base_frame_shift if use_base_frame_shift else 'none'}" />
     </xacro:if>
+    <xacro:openarm_v20_emit_reference_frames
+      reference_points="${ee_reference_points}"
+      prefix="${prefix}" link_prefix="${prefix + 'ee_'}"
+      base_link_name="${base_link_name}"
+      reflect_x="${reflect_x if component_reflects else 1}"
+      reflect_y="${reflect_y if component_reflects else 1}"
+      reflect_z="${reflect_z if component_reflects else 1}"
+      reflect_include_reference_points="${reflect_include_reference_points}"
+      frame_shift="${resolved_base_frame_shift if use_base_frame_shift else 'none'}" />
   </xacro:macro>
 </robot>

File: assets/robot/openarm_v2.0/urdf/utils/openarm_v20_robot.xacro (robot description, xacro)
@@ -95,10 +95,19 @@
           lazy_eval="false" />
       </xacro:if>
+      <xacro:if value="${source_type == 'accessory'}">
+        <xacro:property name="component_type" value="accessory" lazy_eval="false" />
+        <xacro:property name="component_cfg_root" value="${'$(find openarm_description)/assets/accessory/' + product + '/config'}" lazy_eval="false" />
+      </xacro:if>
       <xacro:property name="component_link_prefix" value="${component_prefix + ('ee_' if component_type == 'end_effector' else '')}" lazy_eval="false" />
       <xacro:property name="component_topology" value="${xacro.load_yaml(component_cfg_root + '/struct/topology.yaml')}" lazy_eval="false" />
       <xacro:property name="component_reference_points" value="${xacro.load_yaml(component_cfg_root + '/struct/reference_points.yaml')}" lazy_eval="false" />
-      <xacro:property name="component_joint_origins" value="${xacro.load_yaml(component_cfg_root + '/joint/joint_origins.yaml') if component_type != 'body' else empty_dict}" lazy_eval="false" />
-      <xacro:property name="component_joint_axes" value="${xacro.load_yaml(component_cfg_root + '/joint/joint_axes.yaml') if component_type != 'body' else empty_dict}" lazy_eval="false" />
-      <xacro:property name="component_joint_limits" value="${xacro.load_yaml(component_cfg_root + '/joint/joint_limits.yaml') if component_type != 'body' else empty_dict}" lazy_eval="false" />
+      <xacro:if value="${component_type == 'accessory'}">
+        <xacro:openarm_v20_require
+          condition="${len(component_topology['links']) == 1 and len(component_topology['joints']) == 0}"
+          message="${'Accessory `%s` must define one rigid link and no internal joints.' % component_name}" />
+      </xacro:if>
+      <xacro:property name="component_joint_origins" value="${xacro.load_yaml(component_cfg_root + '/joint/joint_origins.yaml') if component_type not in ['body', 'accessory'] else empty_dict}" lazy_eval="false" />
+      <xacro:property name="component_joint_axes" value="${xacro.load_yaml(component_cfg_root + '/joint/joint_axes.yaml') if component_type not in ['body', 'accessory'] else empty_dict}" lazy_eval="false" />
+      <xacro:property name="component_joint_limits" value="${xacro.load_yaml(component_cfg_root + '/joint/joint_limits.yaml') if component_type not in ['body', 'accessory'] else empty_dict}" lazy_eval="false" />
       <xacro:property name="component_joint_mimics" value="${xacro.load_yaml(component_cfg_root + '/joint/joint_mimics.yaml') if component_type == 'end_effector' else empty_dict}" lazy_eval="false" />
       <xacro:property name="component_inertials" value="${xacro.load_yaml(component_cfg_root + '/inertials/' + component_cfg['inertials'] + '.yaml')}" lazy_eval="false" />
@@ -156,5 +165,5 @@
         message="${'Invalid robot preset: component `%s` attaches to disabled parent `%s`.' % (component_name, attach_to)}" />
       <xacro:openarm_v20_require
-        condition="${robot_preset[attach_to]['type'] in ['robot', 'end_effector', 'sensor']}"
+        condition="${robot_preset[attach_to]['type'] in ['robot', 'end_effector', 'sensor', 'accessory']}"
         message="${'Invalid robot preset: component `%s` attaches to unsupported parent type `%s` on `%s`.' % (component_name, robot_preset[attach_to]['type'], attach_to)}" />
       <xacro:openarm_v20_validate_component_lineage
@@ -181,5 +190,5 @@
       <xacro:property name="reflect_cfg" value="${component_cfg['reflect'] if 'reflect' in component_cfg else dict(x=1, y=1, z=1)}" lazy_eval="false" />
       <xacro:openarm_v20_require
-        condition="${component_type in ['robot', 'end_effector', 'sensor']}"
+        condition="${component_type in ['robot', 'end_effector', 'sensor', 'accessory']}"
         message="${'Invalid robot preset: component `%s` has unsupported type `%s`.' % (component_name, component_type)}" />
       <xacro:openarm_v20_require
@@ -306,4 +315,9 @@
                      yaw=parent_ref['origin']['yaw'])}"
         lazy_eval="false" />
+      <xacro:if value="${parent_ref.get('emit', False)}">
+        <xacro:property name="reference_prefix" value="${parent_desc['root_link_actual'] + '_' if parent_desc['component_type'] == 'body' else parent_desc['prefix']}" lazy_eval="false" />
+        <xacro:property name="resolved_connected_to" value="${reference_prefix + parent_ref_name}" lazy_eval="false" />
+        <xacro:property name="resolved_mount_origin" value="${zero_origin}" lazy_eval="false" />
+      </xacro:if>
     </xacro:if>
     <xacro:if value="${has_parent_override}">
@@ -386,5 +400,5 @@
     params="component_desc component_runtime emit_grasp_frame:=false">
     <xacro:property name="component_type" value="${component_runtime['component_type']}" lazy_eval="false" />
-    <xacro:if value="${component_type == 'body'}">
+    <xacro:if value="${component_type in ['body', 'accessory']}">
       <xacro:openarm_v20_body
         link_name="${component_desc['root_link_actual']}"
@@ -460,4 +474,17 @@
         prefix="${component_desc['prefix']}" />
     </xacro:if>
+    <xacro:unless value="${component_type == 'end_effector'}">
+      <xacro:openarm_v20_emit_reference_frames
+        reference_points="${component_desc['reference_points']}"
+        prefix="${component_desc['root_link_actual'] + '_' if component_type == 'body' else component_desc['prefix']}"
+        link_prefix="${component_desc['link_prefix']}"
+        link_name_map="${component_desc['link_name_map']}"
+        base_link_name="${component_desc['topology']['links'][0]}"
+        reflect_x="${component_runtime['reflect_x']}"
+        reflect_y="${component_runtime['reflect_y']}"
+        reflect_z="${component_runtime['reflect_z']}"
+        reflect_include_reference_points="${component_runtime['reflect_include_reference_points']}"
+        frame_shift="${component_runtime['base_frame_shift']}" />
+    </xacro:unless>
   </xacro:macro>
   <!-- Per-component orchestration: descriptor -> runtime resolution -> emission -> child recursion. -->

File: assets/robot/openarm_v2.0/urdf/utils/openarm_v20_utils.xacro (robot description, xacro)
@@ -13,12 +13,12 @@
 -->
 <robot xmlns:xacro="http://www.ros.org/wiki/xacro">
-  <!-- Emit one origin while optionally mirroring translation along selected axes. -->
-  <xacro:macro name="openarm_v20_emit_origin" params="origin reflect_x:=1 reflect_y:=1 reflect_z:=1 reflect_position:=true">
+  <!-- Emit one origin with optional translation and rotation reflection. -->
+  <xacro:macro name="openarm_v20_emit_origin" params="origin reflect_x:=1 reflect_y:=1 reflect_z:=1 reflect_position:=true reflect_rotation:=${False}">
     <origin
       xyz="${(reflect_x * origin['x']) if reflect_position else origin['x']} ${(reflect_y * origin['y']) if reflect_position else origin['y']} ${(reflect_z * origin['z']) if reflect_position else origin['z']}"
-      rpy="${origin['roll']} ${origin['pitch']} ${origin['yaw']}" />
+      rpy="${reflect_y * reflect_z * origin['roll'] if reflect_rotation else origin['roll']} ${reflect_x * reflect_z * origin['pitch'] if reflect_rotation else origin['pitch']} ${reflect_x * reflect_y * origin['yaw'] if reflect_rotation else origin['yaw']}" />
   </xacro:macro>
   <!-- Compose two poses in xacro so mount transforms can be absorbed into geometry or joints. -->
-  <xacro:macro name="openarm_v20_emit_composed_origin" params="first second reflect_x:=1 reflect_y:=1 reflect_z:=1 reflect_position:=true">
+  <xacro:macro name="openarm_v20_emit_composed_origin" params="first second reflect_x:=1 reflect_y:=1 reflect_z:=1 reflect_position:=true reflect_rotation:=${False}">
     <xacro:property name="a_r" value="${first['roll']}" />
     <xacro:property name="a_p" value="${first['pitch']}" />
@@ -73,5 +73,5 @@
     <origin
       xyz="${(reflect_x * tx) if reflect_position else tx} ${(reflect_y * ty) if reflect_position else ty} ${(reflect_z * tz) if reflect_position else tz}"
-      rpy="${rr} ${rp} ${ry}" />
+      rpy="${reflect_y * reflect_z * rr if reflect_rotation else rr} ${reflect_x * reflect_z * rp if reflect_rotation else rp} ${reflect_x * reflect_y * ry if reflect_rotation else ry}" />
   </xacro:macro>
   <xacro:macro name="openarm_v20_emit_limit" params="limit">
@@ -145,8 +145,8 @@
     <joint name="${link_name}_joint" type="fixed">
       <xacro:if value="${frame_shift != 'none'}">
-        <xacro:openarm_v20_emit_composed_origin first="${frame_shift}" second="${origin}" reflect_x="${reflect_x}" reflect_y="${reflect_y}" reflect_z="${reflect_z}" />
+        <xacro:openarm_v20_emit_composed_origin first="${frame_shift}" second="${origin}" reflect_x="${reflect_x}" reflect_y="${reflect_y}" reflect_z="${reflect_z}" reflect_rotation="${True}" />
       </xacro:if>
       <xacro:unless value="${frame_shift != 'none'}">
-        <xacro:openarm_v20_emit_origin origin="${origin}" reflect_x="${reflect_x}" reflect_y="${reflect_y}" reflect_z="${reflect_z}" />
+        <xacro:openarm_v20_emit_origin origin="${origin}" reflect_x="${reflect_x}" reflect_y="${reflect_y}" reflect_z="${reflect_z}" reflect_rotation="${True}" />
       </xacro:unless>
       <parent link="${parent_link}" />
@@ -200,3 +200,29 @@
     </joint>
   </xacro:macro>
+  <xacro:macro name="openarm_v20_emit_reference_frames"
+    params="reference_points prefix link_prefix link_name_map:=${dict()} base_link_name:='' reflect_x:=1 reflect_y:=1 reflect_z:=1 reflect_include_reference_points:=^ frame_shift:=none index:=0">
+    <xacro:property name="reference_names" value="${list(reference_points.keys())}" lazy_eval="false" />
+    <xacro:if value="${index &lt; len(reference_names)}">
+      <xacro:property name="reference_name" value="${reference_names[index]}" lazy_eval="false" />
+      <xacro:property name="reference" value="${reference_points[reference_name]}" lazy_eval="false" />
+      <xacro:if value="${reference.get('emit', False)}">
+        <xacro:property name="reference_parent" value="${reference['parent']}" lazy_eval="false" />
+        <xacro:property name="reference_reflects" value="${reference_name in reflect_include_reference_points}" lazy_eval="false" />
+        <xacro:openarm_v20_emit_reference_link
+          link_name="${prefix + reference_name}"
+          parent_link="${link_name_map[reference_parent] if reference_parent in link_name_map else link_prefix + reference_parent}"
+          origin="${reference['origin']}"
+          reflect_x="${reflect_x if reference_reflects else 1}"
+          reflect_y="${reflect_y if reference_reflects else 1}"
+          reflect_z="${reflect_z if reference_reflects else 1}"
+          frame_shift="${frame_shift if reference_parent == base_link_name else 'none'}" />
+      </xacro:if>
+      <xacro:openarm_v20_emit_reference_frames
+        reference_points="${reference_points}" prefix="${prefix}" link_prefix="${link_prefix}"
+        link_name_map="${link_name_map}" base_link_name="${base_link_name}"
+        reflect_x="${reflect_x}" reflect_y="${reflect_y}" reflect_z="${reflect_z}"
+        reflect_include_reference_points="${reflect_include_reference_points}"
+        frame_shift="${frame_shift}" index="${index + 1}" />
+    </xacro:if>
+  </xacro:macro>
 </robot>

Commit message: Make the camera assembly the default V2 bimanual preset

File: assets/robot/openarm_v2.0/urdf/example/v2.urdf (robot description, URDF)
Before this commit: robot openarm_v20, 25 links, 24 joints
Links:
- added link openarm_body_zed_camera_center; collision mesh filename=package://zed_description/meshes/zedm.stl; visual mesh filename=package://zed_description/meshes/zedm.stl
- added link openarm_body_zed_camera_link
- added link openarm_body_zed_left_camera_frame
- added link openarm_body_zed_left_camera_frame_optical
- added link openarm_body_zed_mount_base_link, mass 0.13704; visual mesh filename=package://openarm_description/assets/accessory/zed_mount/me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 scale=1 1 1
- added link openarm_body_zed_mount_camera_mount_point
- added link openarm_body_zed_right_camera_frame
- added link openarm_body_zed_right_camera_frame_optical
Joints:
- added joint openarm_body_zed_camera_center_joint: type fixed, parent openarm_body_zed_camera_link, child openarm_body_zed_camera_center, origin xyz=0 0 0.01325 rpy=0 0.0 0
- added joint openarm_body_zed_left_camera_joint: type fixed, parent openarm_body_zed_camera_center, child openarm_body_zed_left_camera_frame, origin xyz=0.0 0.0315 0 rpy=0 0 0
- added joint openarm_body_zed_left_camera_optical_joint: type fixed, parent openarm_body_zed_left_camera_frame, child openarm_body_zed_left_camera_frame_optical, origin xyz=0 0 0 rpy=-1.5707963267948966 0.0 -1.5707963267948966
- added joint openarm_body_zed_mount_base_link_mount_joint: type fixed, parent openarm_body_link0_camera_mount_point, child openarm_body_zed_mount_base_link, origin xyz=0.0 0.0 0.0 rpy=0.0 0.0 0.0
- added joint openarm_body_zed_mount_camera_mount_point_joint: type fixed, parent openarm_body_zed_mount_base_link, child openarm_body_zed_mount_camera_mount_point, origin xyz=0.0263085336684006 0.00869000000000031 0.065829226007701 rpy=0 1.08210413623648 0
- added joint openarm_body_zed_mount_joint: type fixed, parent openarm_body_zed_mount_camera_mount_point, child openarm_body_zed_camera_link, origin xyz=0.00119247 -0.007723415 8.746e-05 rpy=0.0 0.0 0.0
- added joint openarm_body_zed_right_camera_joint: type fixed, parent openarm_body_zed_camera_center, child openarm_body_zed_right_camera_frame, origin xyz=0.0 -0.0315 0 rpy=0 0 0
- added joint openarm_body_zed_right_camera_optical_joint: type fixed, parent openarm_body_zed_right_camera_frame, child openarm_body_zed_right_camera_frame_optical, origin xyz=0 0 0 rpy=-1.5707963267948966 0.0 -1.5707963267948966
- joint openarm_left_base_link_mount_joint: origin xyz=0.0 0.03 0.697 rpy=0.0 0.0 0.0 -> xyz=0.0 0.03 0.697 rpy=0.0 -0.0 0.0
- joint openarm_right_base_link_mount_joint: origin xyz=0.0 -0.03 0.697 rpy=0.0 0.0 0.0 -> xyz=0.0 -0.03 0.697 rpy=0.0 -0.0 0.0

Commit message: Update the V2 open-top body visual and measured inertia

File: assets/robot/openarm_v2.0/urdf/example/v2.urdf (robot description, URDF)
Before this commit: robot openarm_v20, 22 links, 21 joints
Links:
- link openarm_body_link0: mass 3.74 -> 3.734812201783; geometry collision mesh filename=package://openarm_description/assets/robot/openarm_v2.0/mes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 scale=0.001 0.001 0.001; visual mesh filename=package://openarm_description/assets/robot/openarm_v2.0/mes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 scale=1.0 1.0 1.0
