Commit message: Add V2 gripper camera visuals and mounting reference frames (#100)
The V2 gripper model lacks the camera geometry and viewing reference
from the CAD assembly. Add the B0495 camera visual to `ee_base_link` and
a massless `camera_view_frame` to the full robot and standalone gripper.

- Reflect reference-frame position and orientation together for the left
side.
- Compose `connection.origin` relative to the selected mounting
reference. Toggling `emit` changes the frame output while preserving the
mounted component's pose.
- Carry the reference poses through arm-tip folding, generate the grasp
frame once, and regenerate the V2 example URDF.

### Compatibility

`connection.origin` was an absolute override of the mounting reference's
pose. It's now an offset relative to the mounting reference. All bundled
presets use `origin: null`, so their generated URDFs don't change except
the new `camera_view_frame`. Custom presets that set `connection.origin`
with `parent_reference_point` need to be updated.

### RViz comparison

| Before | After |
| --- | --- |
|
![Before](https://github.com/user-attachments/assets/4552563f-6318-4849-b53a-413bd2f21b25)
|
![After](https://github.com/user-attachments/assets/7817bcc4-43a2-478d-91aa-756bf0b80340)
|

Gripper base visual; colored axes show the new `camera_view_frame`.
Separate RViz captures use identical placement and camera settings.

Validation: eight tests cover mirrored frames, standalone generation,
folding, reference emission, grasp frame emission and mounting offsets,
including the generated component and its composed world pose, and check
`camera_view_frame` against the camera parts in the visual mesh. CI runs
them with `test/run.sh`. All five V2 presets and both standalone
grippers expand and pass `check_urdf`; the updated DAE loads
successfully.

---------

Co-authored-by: Sutou Kouhei <kou@clear-code.com>
Co-authored-by: Claude Opus 5.5 <noreply@anthropic.com>

File: assets/robot/openarm_v2.0/urdf/example/v2.urdf (robot description, URDF)
Before this commit: robot openarm_v20, 22 links, 21 joints
Links:
- added link openarm_left_camera_view_frame
- added link openarm_right_camera_view_frame
Joints:
- added joint openarm_left_camera_view_frame_joint: type fixed, parent openarm_left_ee_base_link, child openarm_left_camera_view_frame, origin xyz=0.021835300000000002 0.024136 -0.086895 rpy=-2.1009 1.1424 -2.1431
- added joint openarm_right_camera_view_frame_joint: type fixed, parent openarm_right_ee_base_link, child openarm_right_camera_view_frame, origin xyz=0.021835300000000002 -0.024136 -0.086895 rpy=2.1009 1.1424 2.1431
- joint openarm_left_base_link_mount_joint: origin xyz=0.0 0.03 0.697 rpy=0.0 0.0 0.0 -> xyz=0.0 0.03 0.697 rpy=0.0 -0.0 0.0
- joint openarm_right_base_link_mount_joint: origin xyz=0.0 -0.03 0.697 rpy=0.0 0.0 0.0 -> xyz=0.0 -0.03 0.697 rpy=0.0 -0.0 0.0
