Commit message: Move the pinch-gripper macro into its asset directory

File: assets/component_loader.xacro (robot description, xacro)
@@ -17,5 +17,5 @@
   <xacro:include filename="$(find openarm_description)/assets/common/validation.xacro" />
   <xacro:include filename="$(find openarm_description)/assets/robot/openarm_v2.0/urdf/utils/openarm_v20_arm.xacro" />
-  <xacro:include filename="$(find openarm_description)/assets/robot/openarm_v2.0/urdf/utils/openarm_v20_ee.xacro" />
+  <xacro:include filename="$(find openarm_description)/assets/end_effector/pinch_gripper/urdf/pinch_gripper_macro.xacro" />
   <xacro:include filename="$(find openarm_description)/assets/robot/openarm_v2.0/urdf/utils/openarm_v20_sensor.xacro" />
   <xacro:macro name="openarm_load_component_descriptor"
@@ -164,5 +164,5 @@
     </xacro:if>
     <xacro:if value="${component_type == 'end_effector'}">
-      <xacro:openarm_v20_ee
+      <xacro:openarm_pinch_gripper
         prefix="${component_desc['prefix']}"
         connected_to="${component_runtime['resolved_connected_to']}"

File: assets/end_effector/pinch_gripper/urdf/pinch_gripper_macro.xacro (robot description, xacro)
@@ -17,5 +17,5 @@
   <!-- Current EE implementation targets the two-finger gripper topology. -->
   <xacro:include filename="$(find openarm_description)/assets/common/validation.xacro" />
-  <xacro:macro name="openarm_v20_ee"
+  <xacro:macro name="openarm_pinch_gripper"
     params="prefix connected_to mount_origin:=none topology joint_origins joint_axes joint_limits joint_mimics inertials visuals collisions reflect_x:=1 reflect_y:=1 reflect_z:=1 component_reflects:=false reflect_include_links:=^ reflect_include_joints:=^ reflect_include_reference_points:=^ limit_override_joints:=^ ee_reference_points:=^ emit_grasp_frame:=false grasp_reference_point:=grasp_frame skip_mount_joint:=false base_frame_shift:=none">
     <xacro:property name="base_link_name" value="${topology['links'][0]}" />

File: assets/end_effector/pinch_gripper/urdf/pinch_gripper_standalone.urdf.xacro (robot description, xacro)
@@ -15,5 +15,5 @@
   <xacro:include filename="$(find openarm_description)/assets/common/links.xacro" />
   <xacro:include filename="$(find openarm_description)/assets/common/reference_frames.xacro" />
-  <xacro:include filename="$(find openarm_description)/assets/robot/openarm_v2.0/urdf/utils/openarm_v20_ee.xacro" />
+  <xacro:include filename="$(find openarm_description)/assets/end_effector/pinch_gripper/urdf/pinch_gripper_macro.xacro" />
   <xacro:arg name="ee_config_dir" default="$(find openarm_description)/assets/end_effector/pinch_gripper/config" />
   <xacro:arg name="ee_inertials_name" default="nominal" />
@@ -34,5 +34,5 @@
   <xacro:property name="ee_topology" value="${xacro.load_yaml('$(arg ee_config_dir)/struct/topology.yaml')}" lazy_eval="false" />
   <xacro:property name="ee_reference_points" value="${xacro.load_yaml('$(arg ee_config_dir)/struct/reference_points.yaml')}" lazy_eval="false" />
-  <xacro:openarm_v20_ee
+  <xacro:openarm_pinch_gripper
     prefix=""
     connected_to="world"
